File: ShiroFOC/Manual_Layout_P2/MCUclockSWD.kicad_sch (KiCad schematic)
At the start: 25 parts, among them J1001 ARM Cortex SWD 10-pin, SW301 RESET, U4 STSPIN32G4, Y301 24MHz 7pF

Commit message: Backup before 2nd encoder support
Parts:
- C301, C303, C305, C307, C310: footprint Capacitor_SMD:C_0603_1608Metric -> Capacitor_SMD:C_0402_1005Metric; Procurement Select to specification: 100nF; C_0603_1608Metric -> 0402; preserve Value/tolerance requirements; exact part not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
- C308, C309: footprint Capacitor_SMD:C_0603_1608Metric -> Capacitor_SMD:C_0402_1005Metric; Procurement Select to specification: 10pF C0G; C_0603_1608Metric -> 0402; preserve Value/tolerance requirements; exact part not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
- R301, R302: footprint Resistor_SMD:R_0603_1608Metric -> Resistor_SMD:R_0402_1005Metric; Procurement Select to specification: 0R; R_0603_1608Metric -> 0402; preserve Value/tolerance requirements; exact part not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
- R303: footprint Resistor_SMD:R_0603_1608Metric -> Resistor_SMD:R_0402_1005Metric; Procurement Select to specification: 100k; R_0603_1608Metric -> 0402; preserve Value/tolerance requirements; exact part not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
- R304: footprint Resistor_SMD:R_0603_1608Metric -> Resistor_SMD:R_0402_1005Metric; Procurement 2.2k 1%, 0603; low-current active-low status LED -> 0402; preserve Value/tolerance requirements; exact part not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
- TP1021: value SPARE_GPIO_1 -> STATUS_LED_N
