File: ShiroFOC/Manual_Layout_P3/ShiroFOC_Manual.kicad_sch (KiCad schematic)
At the start: 4 parts

Commit message: progress
Parts:
- H1, H2, H3, H4: value M3 NPTH -> M2 PTH; footprint MountingHole:MountingHole_3.2mm_M3 -> MountingHole:MountingHole_2.2mm_M2_Pad_Via
Other:
- note added: "4 x M2 / 2.2 mm PTH + vias"
- note added: "Review each page before PCB update. Downloads/checklist: downloads/FOOTPRINT_CAD_CHECKLIST.md H1-H4: M2 plated clearance holes with perimeter vias. Existing manual PCB has not been synchronized with this schematic."
- note removed: "4 x M3 / 3.2 mm NPTH"
- note removed: "Review each page before PCB update. Downloads/checklist: downloads/FOOTPRINT_CAD_CHECKLIST.md H1-H4: M3 clearance holes. Existing manual PCB has not been synchronized with this schematic."
Changed lines of the file:
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@@
 		)
 	)
-	(text "4 x M3 / 3.2 mm NPTH"
+	(text "4 x M2 / 2.2 mm PTH + vias"
 		(exclude_from_sim no)
 		(at 104.14 135.89 0)
@@
 		)
 	)
-	(text "Review each page before PCB update. Downloads/checklist: downloads/FOOTPRINT_CAD_CHECKLIST.md\nH1-H4: M3 clearance holes. Existing manual PCB has not been synchronized with this schematic."
+	(text "Review each page before PCB update. Downloads/checklist: downloads/FOOTPRINT_CAD_CHECKLIST.md\nH1-H4: M2 plated clearance holes with perimeter vias. Existing manual PCB has not been synchronized with this schematic."
 		(exclude_from_sim no)
 		(at 15.24 281.94 0)
@@
 			)
 		)
-		(property "Value" "M3 NPTH"
+		(property "Value" "M2 PTH"
 			(at 111.76 167.64 0)
 			(effects
@@
 			)
 		)
-		(property "Footprint" "MountingHole:MountingHole_3.2mm_M3"
+		(property "Footprint" "MountingHole:MountingHole_2.2mm_M2_Pad_Via"
 			(at 111.76 163.83 0)
 			(effects
@@
 			)
 		)
-		(property "Value" "M3 NPTH"
+		(property "Value" "M2 PTH"
 			(at 147.32 151.13 0)
 			(effects
@@
 			)
 		)
-		(property "Footprint" "MountingHole:MountingHole_3.2mm_M3"
+		(property "Footprint" "MountingHole:MountingHole_2.2mm_M2_Pad_Via"
 			(at 147.32 147.32 0)
 			(effects
@@
 			)
 		)
-		(property "Value" "M3 NPTH"
+		(property "Value" "M2 PTH"
 			(at 147.32 167.64 0)
 			(effects
@@
 			)
 		)
-		(property "Footprint" "MountingHole:MountingHole_3.2mm_M3"
+		(property "Footprint" "MountingHole:MountingHole_2.2mm_M2_Pad_Via"
 			(at 147.32 163.83 0)
 			(effects
@@
 			)
 		)
-		(property "Value" "M3 NPTH"
+		(property "Value" "M2 PTH"
 			(at 111.76 151.13 0)
 			(effects
@@
 			)
 		)
-		(property "Footprint" "MountingHole:MountingHole_3.2mm_M3"
+		(property "Footprint" "MountingHole:MountingHole_2.2mm_M2_Pad_Via"
 			(at 111.76 147.32 0)
 			(effects
