File: ShiroFOC/Manual_Layout_P3/02_Auxiliary_Power.kicad_sch (KiCad schematic)
At the start: 39 parts, among them U201 LMR36510FADDAR, U203 TPS2121RUXR, U204 TLV75533PDYDR, U205 MPM3620AGQV-Z

Commit message: CAN layout
Parts:
- C201: symbol Manual:COMP_C201 -> ShiroFOCLib:COMP_C201
- C202: symbol Manual:COMP_C202 -> ShiroFOCLib:COMP_C202
- C203: symbol Manual:COMP_C203 -> ShiroFOCLib:COMP_C203
- C204: symbol Manual:COMP_C204 -> ShiroFOCLib:COMP_C204
- C205, C214, C215, C218, C219: symbol Manual:COMP_C205 -> ShiroFOCLib:COMP_C205
- C206: symbol Manual:COMP_C206 -> ShiroFOCLib:COMP_C206
- C209: symbol Manual:COMP_C209 -> ShiroFOCLib:COMP_C209
- C210: symbol Manual:COMP_C210 -> ShiroFOCLib:COMP_C210
- C211: symbol Manual:COMP_C211 -> ShiroFOCLib:COMP_C211
- C212: symbol Manual:COMP_C212 -> ShiroFOCLib:COMP_C212
- C213: symbol Manual:COMP_C213 -> ShiroFOCLib:COMP_C213
- L201: footprint Manual:WE_LHMI_7050_74437349470 -> ShiroFOCLib:WE_LHMI_7050_74437349470; symbol Manual:COMP_L201 -> ShiroFOCLib:COMP_L201
- R201: symbol Manual:COMP_R201 -> ShiroFOCLib:COMP_R201
- R202, R216, R217, R218, R219: symbol Manual:COMP_R202 -> ShiroFOCLib:COMP_R202
- R206: symbol Manual:COMP_R206 -> ShiroFOCLib:COMP_R206
- R207: symbol Manual:COMP_R207 -> ShiroFOCLib:COMP_R207
- R208: symbol Manual:COMP_R208 -> ShiroFOCLib:COMP_R208
- R209: symbol Manual:COMP_R209 -> ShiroFOCLib:COMP_R209
- R210: symbol Manual:COMP_R210 -> ShiroFOCLib:COMP_R210
- R211: symbol Manual:COMP_R211 -> ShiroFOCLib:COMP_R211
- R212: symbol Manual:COMP_R212 -> ShiroFOCLib:COMP_R212
- R213: symbol Manual:COMP_R213 -> ShiroFOCLib:COMP_R213
- R214: symbol Manual:COMP_R214 -> ShiroFOCLib:COMP_R214
- R215: symbol Manual:COMP_R215 -> ShiroFOCLib:COMP_R215
- TP1005: symbol Manual:COMP_TP1005 -> ShiroFOCLib:COMP_TP1005
- TP1006: symbol Manual:COMP_TP1006 -> ShiroFOCLib:COMP_TP1006
- TP201: symbol Manual:COMP_TP201 -> ShiroFOCLib:COMP_TP201
- U201: footprint Manual:LMR36510_DDA -> ShiroFOCLib:LMR36510_DDA; symbol Manual:COMP_U201 -> ShiroFOCLib:COMP_U201
- U203: footprint Manual:TPS2121_RUX -> ShiroFOCLib:TPS2121_RUX; symbol Manual:COMP_U203 -> ShiroFOCLib:COMP_U203
- U204: footprint Manual:TLV75533_DYD_GND -> ShiroFOCLib:TLV75533_DYD_GND; symbol Manual:COMP_U204 -> ShiroFOCLib:COMP_U204
- U205: footprint Manual:IC18_MPM3620AGQV-Z_MNP -> ShiroFOCLib:IC18_MPM3620AGQV-Z_MNP; symbol Manual:MPM3620AGQV-Z -> ShiroFOCLib:MPM3620AGQV-Z

Commit message: progress
Parts:
- added D201: LTST-C19HE1WT, LED_SMD:LED_LiteOn_LTST-C19HE1WT, symbol ShiroFOCLib:LTST_C19HE1WT
- added Q201: CSD17483F4, ShiroFOCLib:CSD17483F4_YJC0003A, symbol ShiroFOCLib:CSD17483F4
- added R220: 10k, Resistor_SMD:R_0402_1005Metric, symbol ShiroFOCLib:COMP_R215
- added R221: 33k, Resistor_SMD:R_0402_1005Metric, symbol ShiroFOCLib:COMP_R215
Connections:
- net 3V3: no longer R215.1
- net 5V_SYS: now also R215.1, D201.4 (A)
- net GND: now also Q201.2 (S), R220.2
- net PWR_SOURCE_STATUS: now also Q201.1 (G)
- new net: D201.2 (GK), R221.1
- new net: Q201.3 (D), R221.2
- new net: D201.3 (BK), R220.1
- no-connect marks 4 -> 5
Other:
- note added: "BLUE = USB selected; CYAN = motor/battery selected. Red unused. R215 pulls ST up to 3V3; no MCU needed. 10k blue / 33k green: subdued starting values."
- note added: "POWER SOURCE INDICATOR"

Commit message: progress + p4
Parts:
- R206: value 15.0k 1% -> 10.0k 1%
- R208: value 10.0k 1% -> 15.0k 1%
Other:
- note added: "AUXILIARY POWER - BATTERY HAS PRIORITY"
- note added: "At 5 V: PR1 = 1.689 V; CP2 = 1.269 V."
- note added: "At nominal 5 V, battery has priority. Coarse OV = 5.63 V typical."
- note added: "BATTERY-PRIORITY POWER MUX"
- note removed: "AUXILIARY POWER - USB HAS PRIORITY"
- note removed: "At 5 V: PR1 = 1.269 V; CP2 = 1.689 V."
- note removed: "USB wins the priority comparison. Coarse OV = 5.63 V typical."
- note removed: "USB-PRIORITY POWER MUX"
Changed lines of the file:
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@@
 		)
 	)
-	(text "At 5 V: PR1 = 1.269 V; CP2 = 1.689 V."
+	(text "At 5 V: PR1 = 1.689 V; CP2 = 1.269 V."
 		(exclude_from_sim no)
 		(at 25.4 246.38 0)
@@
 		)
 	)
-	(text "AUXILIARY POWER - USB HAS PRIORITY"
+	(text "AUXILIARY POWER - BATTERY HAS PRIORITY"
 		(exclude_from_sim no)
 		(at 17.78 22.86 0)
@@
 		)
 	)
-	(text "USB-PRIORITY POWER MUX"
+	(text "BATTERY-PRIORITY POWER MUX"
 		(exclude_from_sim no)
 		(at 25.4 142.24 0)
@@
 		)
 	)
-	(text "USB wins the priority comparison. Coarse OV = 5.63 V typical."
+	(text "At nominal 5 V, battery has priority. Coarse OV = 5.63 V typical."
 		(exclude_from_sim no)
 		(at 25.4 252.73 0)
@@
 			)
 		)
-		(property "Value" "10.0k 1%"
+		(property "Value" "15.0k 1%"
 			(at 267.97 177.8 0)
 			(effects
@@
 			)
 		)
-		(property "Value" "15.0k 1%"
+		(property "Value" "10.0k 1%"
 			(at 143.51 177.8 0)
 			(effects
