File: ShiroFOC/Manual_Layout_P3/ShiroFOC_Manual.kicad_pcb (KiCad board)
At the start: 4 copper layers, 80 x 80 mm, 259 parts, among them J1 MOTOR U/V/W, J1001 TC2030-NL SWD, J101 AMASS XT60PW-M, J201 USB-C service, J501 BRAKE RESISTOR, J502 BRAKE NTC, J601 EXT ENCODER / HALL, J801 CAN 1, J802 CAN 2, Q501 CSD19531Q5A 100V, SW301 RESET, U1 CSD88599Q5DC, U2 CSD88599Q5DC, U201 LMR36510FADDAR, U202 USBLC6-2SC6, U203 TPS2121RUXR, U204 TLV75533PDYDR, U205 MPM3620AGQV-Z, U3 CSD88599Q5DC, U4 STSPIN32G4, U501 UCC27517ADBVR, U502 TLV3012BIDBVR, U601 AS5047P-ATSM, U602 TMUX1574PW, U603 74LVC3G17, U604 TPS2553DBVR, U701 BMI323, U801 TCAN3413DR, U901 CP2102N-A02-GQFN20, Y301 24MHz 7pF

Commit message: pcb layout blocks
Parts:
- removed D504: B5100C 100V 5A, Diode_SMD:D_SMC
- removed R507, R508: 150k 0.1% 200V, Resistor_SMD:R_1206_3216Metric
- C201, C205, C206, C208, C209, C210, C211, C212, C213, C214, C215, C218, C219, C301, C302, C303, C307, L201, R206, R207, R208, R209, R210, R211, R212, R213, R214, R215, U201, U203, U204, U205: moved to B.Cu
- C311, C312, C313, C501, C502, C503, C504, C901, C902, C903, C904, D501, R504, R505, R901, R902, R904, R905, TH701, TH702, TH703: moved to F.Cu
- R506: value 150k 0.1% 200V -> 470k 1% 75V; footprint Resistor_SMD:R_1206_3216Metric -> Resistor_SMD:R_0603_1608Metric; moved to F.Cu
- R509: value 12.7k 0.1% -> 13.3k 1%; moved to F.Cu
- R510: value 1M 0.1% -> 1M 1%; moved to F.Cu
- moved R506 275.8 mm to (-1.25, 156.3), turned to 0 degrees
- moved C503 266.3 mm to (3.95, 151.6), turned to 180 degrees
- moved R510 265.9 mm to (-1.25, 154.6), turned to -90 degrees
- moved C504 264.2 mm to (1.00, 154.6), turned to 90 degrees
- moved D501 263.4 mm to (9.18, 145.2), turned to -90 degrees
- moved R509 263.1 mm to (-0.25, 154.6)
- moved R504 259.8 mm to (8.95, 142.3), turned to 0 degrees
- moved C502 258.8 mm to (11.5, 147.5)
- moved R217 258.1 mm to (20.4, 91.0), turned to 180 degrees
- moved C501 257.2 mm to (12.1, 148.8)
- moved R216 254.7 mm to (20.4, 90.0)
- moved R505 253.5 mm to (14.1, 146.9), turned to -90 degrees
- moved R202 231.9 mm to (23.7, 71.3), turned to 180 degrees
- moved R201 229.7 mm to (25.6, 71.3), turned to 180 degrees
- moved C202 229.0 mm to (17.3, 75.6), turned to -90 degrees
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Connections:
- R506 pad 2: Net-(R506-Pad2) -> Net-(U502-IN+)
- U4 pad 10: NTC_PHASE_C -> NTC_BRAKE
- U4 pad 11: NTC_BRAKE -> NTC_PHASE_B
- U4 pad 13: VBUS_SENSE -> NTC_PHASE_C
- U4 pad 9: NTC_PHASE_B -> VBUS_SENSE
Routing:
- net VM: track 133.1 -> 0.50 mm
- net GND: track 127.5 -> 55.2 mm, vias 1 -> 7
- net /Current / temperature/NTC_C_RAW: track 0.00 -> 45.7 mm, vias 0 -> 2
- net /Current / temperature/NTC_A_RAW: track 0.00 -> 39.6 mm, vias 0 -> 2
- net USB_UART_RX: track 0.00 -> 39.5 mm, vias 0 -> 2
- net /USB service/UART_BRIDGE_RX: track 0.00 -> 39.0 mm, vias 0 -> 2
- net /Current / temperature/NTC_B_RAW: track 0.00 -> 37.0 mm, vias 0 -> 3
- net 5V_USB_RAW: track 0.00 -> 28.7 mm
- net I2C2_SDA: track 15.1 -> 0.00 mm, vias 2 -> 0
- net PHASE_U: track 9.36 -> 0.00 mm
- net AS5047P_CS_N: track 9.31 -> 0.00 mm, vias 1 -> 0
- net GLS1: track 29.9 -> 38.6 mm
- net PHASE_W: track 8.65 -> 0.00 mm
- net PHASE_V: track 8.65 -> 0.00 mm
- net /USB service/USB_DM: track 0.00 -> 7.71 mm
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
Commit message: STSPIN solder paste updated
Parts:
- removed C414, C424, C434: 47pF C0G, Capacitor_SMD:C_0603_1608Metric
- removed R104: 270k 0.1% 100V, Resistor_SMD:R_1206_3216Metric
- removed TP1005: 5V_SYS, TestPoint:TestPoint_Pad_D1.0mm
- removed TP1006: 3V3, TestPoint:TestPoint_Pad_D1.0mm
- removed TP1008: SWDIO, TestPoint:TestPoint_Pad_D1.0mm
- removed TP1009: SWCLK, TestPoint:TestPoint_Pad_D1.0mm
- removed TP101: VM, TestPoint:TestPoint_Pad_D1.5mm
- removed TP1010: ENC_SPI_CLK, TestPoint:TestPoint_Pad_D1.0mm
- removed TP1011: SPI3_MISO, TestPoint:TestPoint_Pad_D1.0mm
- removed TP1012: ENC_SPI_MOSI, TestPoint:TestPoint_Pad_D1.0mm
- removed TP1013: FDCAN1_TX, TestPoint:TestPoint_Pad_D1.0mm
- removed TP1014: FDCAN1_RX, TestPoint:TestPoint_Pad_D1.0mm
- removed TP1015: FEEDBACK_A_H1, TestPoint:TestPoint_Pad_D1.0mm
- removed TP1016: FEEDBACK_B_H2, TestPoint:TestPoint_Pad_D1.0mm
- removed TP1018: OPO_U1, TestPoint:TestPoint_Pad_D1.0mm
- removed TP1019: OPO_V1, TestPoint:TestPoint_Pad_D1.0mm
- removed TP102: GND, TestPoint:TestPoint_Pad_D1.5mm
- removed TP1020: OPO_W1, TestPoint:TestPoint_Pad_D1.0mm
- removed TP1021: STATUS_LED_N, TestPoint:TestPoint_Pad_D1.0mm
- removed TP1022: CAN_STB, TestPoint:TestPoint_Pad_D1.0mm
- removed TP1023: EXT_SENSOR_FAULT_N, TestPoint:TestPoint_Pad_D1.0mm
- removed TP1024: I2C2_SDA, TestPoint:TestPoint_Pad_D1.0mm
- removed TP103: VBUS_SENSE, TestPoint:TestPoint_Pad_D1.5mm
- removed TP201: PWR_SOURCE_STATUS, TestPoint:TestPoint_Pad_D1.5mm
- removed TP202: 5V_USB, TestPoint:TestPoint_Pad_D1.5mm
- removed TP301: VCC, TestPoint:TestPoint_Pad_D1.5mm
- removed TP302: SCREF, TestPoint:TestPoint_Pad_D1.5mm
- removed TP303: NRST, TestPoint:TestPoint_Pad_D1.5mm
- removed TP501: BRAKE_GATE, TestPoint:TestPoint_Pad_D1.5mm
- removed TP502: BRAKE_SWITCH, TestPoint:TestPoint_Pad_D1.5mm
- removed TP701: NTC_PHASE_A, TestPoint:TestPoint_Pad_D1.0mm
- removed TP702: NTC_PHASE_B, TestPoint:TestPoint_Pad_D1.0mm
- removed TP703: NTC_PHASE_C, TestPoint:TestPoint_Pad_D1.0mm
- removed TP901: USB_UART_TX, TestPoint:TestPoint_Pad_D1.0mm
- removed TP902: USB_UART_RX, TestPoint:TestPoint_Pad_D1.0mm
- R103: value 270k 0.1% 100V -> 560k 0.1% 75V; footprint Resistor_SMD:R_1206_3216Metric -> Resistor_SMD:R_0603_1608Metric
- R105: value 27k 0.1% -> 28k 0.1%
- moved R218 243.6 mm to (27.0, 88.3)
- moved R219 243.6 mm to (27.0, 90.3)
- moved C108 170.2 mm to (114.0, 114.5), turned to 180 degrees
- moved R701 60.2 mm to (162.6, 106.2)
- moved R702 59.6 mm to (157.8, 106.1)
- moved R703 59.6 mm to (160.4, 106.1)
- moved R712 42.4 mm to (160.6, 108.3)
- moved R711 42.1 mm to (159.6, 108.3), turned to -90 degrees
- moved C505 39.9 mm to (159.6, 110.0)
- moved C711 39.9 mm to (159.6, 111.9)
- moved C712 39.9 mm to (159.6, 110.9)
- moved C713 39.8 mm to (159.6, 112.8)
- moved J1 8.00 mm to (149.6, 100.0)
- moved R2 8.00 mm to (145.1, 103.6)
- moved TH702 8.00 mm to (144.7, 109.6)
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Connections:
- R105 pad 1: Net-(R104-Pad2) -> Net-(R103-Pad2)
- R106 pad 1: Net-(R104-Pad2) -> Net-(R103-Pad2)
Routing:
- net SHUNT_U_SENSE_P: track 57.9 -> 0.00 mm
- net SHUNT_U_SENSE_N: track 54.4 -> 0.00 mm
- net /Current / temperature/NTC_C_RAW: track 45.7 -> 0.00 mm
- net /Current / temperature/NTC_A_RAW: track 39.6 -> 0.00 mm, vias 2 -> 1
- net USB_UART_RX: track 39.5 -> 0.98 mm
- net /USB service/UART_BRIDGE_RX: track 39.0 -> 2.17 mm, vias 2 -> 1
- net SHUNT_V_SENSE_P: track 34.2 -> 0.00 mm
- net SHUNT_V_SENSE_N: track 32.8 -> 0.01 mm
- net /Current / temperature/NTC_B_RAW: track 37.0 -> 9.62 mm, vias 3 -> 2
- net GLS1: track 38.6 -> 13.7 mm, vias 2 -> 1
- net GLS2: track 24.1 -> 8.94 mm, vias 2 -> 1
- net HS_RETURN_U: track 35.2 -> 20.8 mm
- net SHUNT_W_SENSE_N: track 14.0 -> 0.00 mm
- net SHUNT_W_SENSE_P: track 14.0 -> 0.00 mm
- net GHS1: track 31.0 -> 17.4 mm, vias 2 -> 1
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
Commit message: usb and pwr mux
Parts:
- removed C207: 4.7nF 2kV, Capacitor_SMD:C_1206_3216Metric
- removed R205: 0R, Resistor_SMD:R_0402_1005Metric
- added C110: 10uF, Capacitor_SMD:C_1210_3225Metric, B.Cu at (10.4, -46.9)
- added C111: 10uF, Capacitor_SMD:C_1210_3225Metric, B.Cu at (15.6, -46.9)
- added C112: 10uF, Capacitor_SMD:C_1210_3225Metric, B.Cu at (5.18, -43.3)
- added C113: 10uF, Capacitor_SMD:C_1210_3225Metric, B.Cu at (10.4, -43.3)
- added C114: 10uF, Capacitor_SMD:C_1210_3225Metric, B.Cu at (15.6, -43.3)
- added C115: 10uF, Capacitor_SMD:C_1210_3225Metric, B.Cu at (5.18, -39.7)
- added C116: 10uF, Capacitor_SMD:C_1210_3225Metric, B.Cu at (10.4, -39.7)
- added C117: 10uF, Capacitor_SMD:C_1210_3225Metric, B.Cu at (15.6, -39.7)
- added C118: 10uF, Capacitor_SMD:C_1210_3225Metric, B.Cu at (5.18, -36.1)
- added C119: 10uF, Capacitor_SMD:C_1210_3225Metric, B.Cu at (14.6, -36.2)
- added C120: 10uF, Capacitor_SMD:C_1210_3225Metric, B.Cu at (9.94, -36.2)
- added C121: 10uF, Capacitor_SMD:C_1210_3225Metric, F.Cu at (-34.5, -69.6)
- added C122: 10uF, Capacitor_SMD:C_1210_3225Metric, F.Cu at (-29.4, -69.6)
- added C123: 10uF, Capacitor_SMD:C_1210_3225Metric, F.Cu at (-24.1, -69.6)
- added C124: 10uF, Capacitor_SMD:C_1210_3225Metric, F.Cu at (-18.9, -69.6)
- added C125: 10uF DNP, Capacitor_SMD:C_1210_3225Metric, F.Cu at (-27.5, -83.5)
- added C126: 10uF DNP, Capacitor_SMD:C_1210_3225Metric, F.Cu at (-22.3, -83.5)
- added C127: 10uF, Capacitor_SMD:C_1210_3225Metric, B.Cu at (48.4, -47.0)
- added C128: 10uF, Capacitor_SMD:C_1210_3225Metric, B.Cu at (53.6, -47.0)
- added C129: 10uF, Capacitor_SMD:C_1210_3225Metric, B.Cu at (43.2, -47.0)
- added C130: 10uF, Capacitor_SMD:C_1210_3225Metric, F.Cu at (24.1, -54.2)
- added C131: 10uF, Capacitor_SMD:C_1210_3225Metric, F.Cu at (29.3, -54.2)
- added C132: 10uF, Capacitor_SMD:C_1210_3225Metric, F.Cu at (8.47, -54.2)
- added C133: 10uF, Capacitor_SMD:C_1210_3225Metric, F.Cu at (18.9, -57.8)
- added C134: 10uF, Capacitor_SMD:C_1210_3225Metric, F.Cu at (34.5, -54.2)
- added C135: 10uF, Capacitor_SMD:C_1210_3225Metric, B.Cu at (48.4, -36.2)
- added C136: 10uF, Capacitor_SMD:C_1210_3225Metric, B.Cu at (53.6, -36.2)
- added C137: 10uF, Capacitor_SMD:C_1210_3225Metric, F.Cu at (24.1, -57.8)
- added C138: 10uF, Capacitor_SMD:C_1210_3225Metric, F.Cu at (8.47, -61.4)
- added C139: 10uF, Capacitor_SMD:C_1210_3225Metric, F.Cu at (13.7, -61.4)
- added C140: 10uF, Capacitor_SMD:C_1210_3225Metric, F.Cu at (18.9, -61.4)
- added C141: 10uF, Capacitor_SMD:C_1210_3225Metric, F.Cu at (24.1, -61.4)
- added C142: 10uF DNP, Capacitor_SMD:C_1210_3225Metric, F.Cu at (29.3, -61.4)
- added C143: 10uF DNP, Capacitor_SMD:C_1210_3225Metric, F.Cu at (34.5, -61.4)
- added C144: 10uF, Capacitor_SMD:C_1210_3225Metric, B.Cu at (53.6, -32.6)
- added C145: 10uF, Capacitor_SMD:C_1210_3225Metric, F.Cu at (29.3, -57.8)
- added C146: 10uF, Capacitor_SMD:C_1210_3225Metric, B.Cu at (19.9, 51.1)
- added C147: 10uF, Capacitor_SMD:C_1210_3225Metric, F.Cu at (3.27, -54.2)
- added C148: 10uF, Capacitor_SMD:C_1210_3225Metric, F.Cu at (34.5, -57.8)
- added C149: 10uF, Capacitor_SMD:C_1210_3225Metric, F.Cu at (13.7, -57.8)
- added C150: 10uF, Capacitor_SMD:C_1210_3225Metric, F.Cu at (8.47, -57.8)
- added C151: 10uF, Capacitor_SMD:C_1210_3225Metric, F.Cu at (3.27, -57.8)
- added C152: 10uF, Capacitor_SMD:C_1210_3225Metric, B.Cu at (44.1, 54.9)
- added C153: 10uF, Capacitor_SMD:C_1210_3225Metric, F.Cu at (-1.93, -57.8)
- added C154: 10uF, Capacitor_SMD:C_1210_3225Metric, F.Cu at (3.27, -61.4)
- added C155: 10uF, Capacitor_SMD:C_1210_3225Metric, F.Cu at (3.27, -65.0)
- added C156: 10uF, Capacitor_SMD:C_1210_3225Metric, F.Cu at (13.7, -68.6)
- added C157: 10uF, Capacitor_SMD:C_1210_3225Metric, F.Cu at (18.9, -68.6)
- added C158: 10uF, Capacitor_SMD:C_1210_3225Metric, F.Cu at (24.1, -68.6)
- added C159: 10uF DNP, Capacitor_SMD:C_1210_3225Metric, F.Cu at (29.3, -68.6)
- added C160: 10uF DNP, Capacitor_SMD:C_1210_3225Metric, F.Cu at (8.47, -68.6)
- added C413: TUNE DNP, Capacitor_SMD:C_1206_3216Metric, F.Cu at (50.3, -10.4)
- added C414: 47pF C0G, Capacitor_SMD:C_0603_1608Metric, B.Cu at (-16.3, 29.1)
- added C423: TUNE DNP, Capacitor_SMD:C_1206_3216Metric, F.Cu at (52.0, 6.29)
- added C424: 47pF C0G, Capacitor_SMD:C_0603_1608Metric, B.Cu at (-14.8, 29.2)
- added C433: TUNE DNP, Capacitor_SMD:C_1206_3216Metric, F.Cu at (52.4, 34.5)
- added C434: 47pF C0G, Capacitor_SMD:C_0603_1608Metric, B.Cu at (-13.3, 29.2)
- added R415: TUNE DNP, Resistor_SMD:R_1206_3216Metric, F.Cu at (55.0, -10.4)
- added R425: TUNE DNP, Resistor_SMD:R_1206_3216Metric, F.Cu at (56.7, 6.04)
- added R435: TUNE DNP, Resistor_SMD:R_1206_3216Metric, F.Cu at (57.1, 34.5)
- added TP1005: 5V_SYS, TestPoint:TestPoint_Pad_D1.0mm, F.Cu at (89.6, 27.5)
- added TP1006: 3V3, TestPoint:TestPoint_Pad_D1.0mm, F.Cu at (89.6, 30.6)
- added TP1008: SWDIO, TestPoint:TestPoint_Pad_D1.0mm, F.Cu at (81.0, 5.23)
- added TP1009: SWCLK, TestPoint:TestPoint_Pad_D1.0mm, F.Cu at (81.0, 8.28)
- added TP101: VM, TestPoint:TestPoint_Pad_D1.5mm, F.Cu at (-64.4, -27.5)
- added TP1010: ENC_SPI_CLK, TestPoint:TestPoint_Pad_D1.0mm, F.Cu at (105.8, 16.4)
- added TP1011: SPI3_MISO, TestPoint:TestPoint_Pad_D1.0mm, F.Cu at (105.8, 19.4)
- added TP1012: ENC_SPI_MOSI, TestPoint:TestPoint_Pad_D1.0mm, F.Cu at (105.8, 22.5)
- added TP1013: FDCAN1_TX, TestPoint:TestPoint_Pad_D1.0mm, F.Cu at (100.8, 16.4)
- added TP1014: FDCAN1_RX, TestPoint:TestPoint_Pad_D1.0mm, F.Cu at (100.8, 19.4)
- added TP1015: FEEDBACK_A_H1, TestPoint:TestPoint_Pad_D1.0mm, F.Cu at (81.0, 22.5)
- added TP1016: FEEDBACK_B_H2, TestPoint:TestPoint_Pad_D1.0mm, F.Cu at (81.0, 25.5)
- added TP1018: OPO_U1, TestPoint:TestPoint_Pad_D1.0mm, F.Cu at (95.7, 16.4)
- added TP1019: OPO_V1, TestPoint:TestPoint_Pad_D1.0mm, F.Cu at (95.7, 19.4)
- added TP102: GND, TestPoint:TestPoint_Pad_D1.5mm, F.Cu at (-61.6, -27.5)
- added TP1020: OPO_W1, TestPoint:TestPoint_Pad_D1.0mm, F.Cu at (95.7, 22.5)
- added TP1021: STATUS_LED_N, TestPoint:TestPoint_Pad_D1.0mm, F.Cu at (81.0, 11.3)
- added TP1022: CAN_STB, TestPoint:TestPoint_Pad_D1.0mm, F.Cu at (100.8, 22.5)
- added TP1023: EXT_SENSOR_FAULT_N, TestPoint:TestPoint_Pad_D1.0mm, F.Cu at (81.0, 14.4)
- added TP1024: I2C2_SDA, TestPoint:TestPoint_Pad_D1.0mm, F.Cu at (81.0, 17.4)
- added TP103: VBUS_SENSE, TestPoint:TestPoint_Pad_D1.5mm, F.Cu at (81.2, 30.8)
- added TP104: VM BULK, TestPoint:TestPoint_Pad_D3.0mm, F.Cu at (-64.4, -31.0)
- added TP105: GND BULK, TestPoint:TestPoint_Pad_D3.0mm, F.Cu at (-59.9, -31.0)
- added TP201: PWR_SOURCE_STATUS, TestPoint:TestPoint_Pad_D1.5mm, F.Cu at (92.9, 27.8)
- added TP202: 5V_USB, TestPoint:TestPoint_Pad_D1.5mm, F.Cu at (104.0, 27.8)
- added TP301: VCC, TestPoint:TestPoint_Pad_D1.5mm, F.Cu at (106.5, 5.48)
- added TP302: SCREF, TestPoint:TestPoint_Pad_D1.5mm, F.Cu at (106.5, 9.03)
- added TP303: NRST, TestPoint:TestPoint_Pad_D1.5mm, F.Cu at (84.3, 5.48)
- added TP411: GL, TestPoint:TestPoint_Pad_D1.0mm, F.Cu at (89.6, 5.23)
- added TP412: SOURCE, TestPoint:TestPoint_Pad_D1.0mm, F.Cu at (89.6, 8.28)
- added TP413: PHASE, TestPoint:TestPoint_Pad_D1.0mm, F.Cu at (89.6, 11.3)
- added TP414: SCOPE GND, TestPoint:TestPoint_Pad_D1.0mm, F.Cu at (89.6, 16.4)
- added TP421: GL, TestPoint:TestPoint_Pad_D1.0mm, F.Cu at (92.7, 5.23)
- added TP422: SOURCE, TestPoint:TestPoint_Pad_D1.0mm, F.Cu at (92.7, 8.28)
- added TP423: PHASE, TestPoint:TestPoint_Pad_D1.0mm, F.Cu at (92.7, 11.3)
- added TP424: SCOPE GND, TestPoint:TestPoint_Pad_D1.0mm, F.Cu at (89.6, 19.4)
- added TP431: GL, TestPoint:TestPoint_Pad_D1.0mm, F.Cu at (95.7, 5.23)
- added TP432: SOURCE, TestPoint:TestPoint_Pad_D1.0mm, F.Cu at (95.7, 8.28)
- added TP433: PHASE, TestPoint:TestPoint_Pad_D1.0mm, F.Cu at (95.7, 11.3)
- added TP434: SCOPE GND, TestPoint:TestPoint_Pad_D1.0mm, F.Cu at (89.6, 22.5)
- added TP501: BRAKE_GATE, TestPoint:TestPoint_Pad_D1.5mm, F.Cu at (101.0, 5.48)
- added TP502: BRAKE_SWITCH, TestPoint:TestPoint_Pad_D1.5mm, F.Cu at (101.0, 9.03)
- added TP701: NTC_PHASE_A, TestPoint:TestPoint_Pad_D1.0mm, F.Cu at (92.7, 16.4)
- added TP702: NTC_PHASE_B, TestPoint:TestPoint_Pad_D1.0mm, F.Cu at (92.7, 19.4)
- added TP703: NTC_PHASE_C, TestPoint:TestPoint_Pad_D1.0mm, F.Cu at (92.7, 22.5)
- added TP901: USB_UART_TX, TestPoint:TestPoint_Pad_D1.0mm, F.Cu at (100.8, 27.5)
- added TP902: USB_UART_RX, TestPoint:TestPoint_Pad_D1.0mm, F.Cu at (100.8, 30.6)
- C101, C102, C103: value 680uF 63V -> 10uF; footprint Manual:Panasonic_EEVFK_K16_18x16.5 -> Capacitor_SMD:C_1210_3225Metric; moved to B.Cu
- C108, C201, C202, C203, C204, C205, C206, C303, L201, R201, R202, R210, R211, R309, R310, R311, R312, R419, R429, R439, U201: moved to F.Cu
- J1: footprint Connector_Wire:SolderWire-6sqmm_1x03_P14mm_D3.5mm_OD7mm -> Connector_AMASS:AMASS_MR30PW-M_1x03_P3.50mm_Horizontal
- JP601, R103, R105, R106: moved to B.Cu
- moved D101 335.7 mm to (-66.4, -35.0)
- moved J502 332.3 mm to (-73.9, 2.22)
- moved C107 327.6 mm to (-57.5, -43.6)
- moved R102 326.4 mm to (-55.4, -29.0)
- moved R617 287.6 mm to (13.8, 53.9)
- moved R616 286.7 mm to (14.6, 52.5)
- moved R615 286.6 mm to (14.6, 51.1)
- moved C603 285.3 mm to (14.1, 62.1), turned to 0 degrees
- moved R512 281.7 mm to (-2.33, 52.7)
- moved R305 273.8 mm to (16.1, 54.0)
- moved D505 259.4 mm to (1.97, 51.7)
- moved R511 258.4 mm to (-5.03, 52.7)
- moved R306 256.6 mm to (21.1, 54.0)
- moved C606 234.6 mm to (22.1, 54.1), turned to 90 degrees
- moved C607 233.6 mm to (41.9, 50.5), turned to 90 degrees
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Connections:
- net Net-(R1-POWER+) renamed /Three-phase bridge/LS_SOURCE_V
- net Net-(R3-POWER+) renamed /Three-phase bridge/LS_SOURCE_U
- net Net-(R5-POWER+) renamed /Three-phase bridge/LS_SOURCE_W
- J201 pad A4: 5V_USB_RAW -> 5V_USB
- J201 pad A9: 5V_USB_RAW -> 5V_USB
- J201 pad B4: 5V_USB_RAW -> 5V_USB
- J201 pad B9: 5V_USB_RAW -> 5V_USB
- J201 pad S1: /USB service/USB_SHIELD -> GND
- R904 pad 1: 5V_USB_RAW -> 5V_USB
- U202 pad 5: 5V_USB_RAW -> 5V_USB
Routing:
- net GND: track 55.2 -> 24.6 mm, vias 7 -> 6
- net 5V_USB_RAW: track 28.7 -> 0.00 mm
- net USB_UART_RX: track 0.98 -> 26.3 mm
- net SHUNT_U_SENSE_P: track 0.00 -> 25.0 mm
- net SHUNT_U_SENSE_N: track 0.00 -> 24.7 mm
- net /USB service/UART_BRIDGE_RX: track 2.17 -> 25.8 mm, vias 1 -> 2
- net 5V_USB: track 0.00 -> 20.8 mm, vias 0 -> 2
- net SHUNT_W_SENSE_P: track 0.00 -> 18.5 mm
- net SHUNT_V_SENSE_P: track 0.00 -> 12.7 mm
- net GLS3: track 7.42 -> 18.8 mm, vias 1 -> 3
- net SHUNT_V_SENSE_N: track 0.01 -> 10.9 mm
- net /Current / temperature/NTC_B_RAW: track 9.62 -> 0.00 mm, vias 2 -> 0
- net GLS2: track 8.94 -> 16.2 mm, vias 1 -> 2
- net I2C2_SCL: track 8.67 -> 2.13 mm, vias 2 -> 0
- net SHUNT_W_SENSE_N: track 0.00 -> 6.32 mm
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- added copper zone on In1.Cu, net GND
- added copper zone on In4.Cu, net GND
Other:
- board size 80 x 80 mm -> 65 x 65 mm
- copper layers 4 -> 6
- board text added: "10 V AUXILIARY POWER"
- board text added: "5 V / POWER MUX / 3.3 V"
- board text added: "50 x 50 mm"
- board text added: "60 x 60 mm"
- board text added: "70 x 70 mm"
- board text added: "80 x 80 mm"
- board text added: "BRAKE CHOPPER"
- board text added: "BRAKE NTC"
- board text added: "BRIDGE ROUTING - FIXED"
- board text added: "CAN INTERFACE"
- board text added: "DC INPUT"
- board text added: "DC LINK / BULK CAPACITORS"
- board text added: "DC LINK PROTECTION / DAMPING"
- board text added: "ENCODER - CENTRED AS5047"
- board text added: "EXTERNAL ENCODER / HALL"
- board text added: "F.Cu: HIGH POWER | In1.Cu: SIGNALS + LV POWER | In2.Cu: GND | B.Cu: SIGNALS + GND"
- board text added: "FEEDBACK MUX / BUS SENSE"
- board text added: "HALF-BRIDGES / SHUNTS - FIXED"
- board text added: "IMU"
- board text added: "MCU + ANALOG - FIXED"
- board text added: "MCU / OP-AMP R + C - FIXED"
- board text added: "P3 PLACEMENT | NO NEW ROUTING | NO TEST POINTS"
- board text added: "RESET / STATUS"
- board text added: "SWD"
- board text added: "TEMPERATURE / ADC FILTERS"
- board text added: "USB / UART"
- board text added: "User.1: FRONT AREAS | User.2: BACK AREAS | Non-copper placement guides"
- board text removed: "${REFERENCE}"
- board text removed: "P3 CORE SHIFT REVIEW | MCU + SUPPORT: 7 mm DOWN"
- board text removed: "U601: exact board centre, B.Cu | Other component placement awaits review"
- board text removed: "p4 / p5 / p7 | MOVED AS ONE BLOCK"
- board text removed: "p9 | CENTRED ENCODER (BACK)"

Commit message: power section updated
Parts:
- C210: moved to F.Cu
- R210, R211: moved to B.Cu
- moved C201 56.5 mm to (-18.5, 0.79), turned to -90 degrees
- moved C202 53.1 mm to (-21.2, 1.40), turned to -90 degrees
- moved J101 50.2 mm to (-15.6, -7.51)
- moved U201 41.5 mm to (-26.4, 1.09), turned to 180 degrees
- moved C218 38.2 mm to (-23.7, 11.3), turned to 180 degrees
- moved C214 36.6 mm to (-20.7, 1.56)
- moved C215 36.6 mm to (-20.7, 4.81)
- moved U205 36.6 mm to (-19.2, 9.33)
- moved R217 36.6 mm to (-16.1, 8.91)
- moved R216 36.6 mm to (-16.1, 7.93), turned to 180 degrees
- moved C213 36.6 mm to (-22.2, 26.3), turned to 90 degrees
- moved C219 36.2 mm to (-23.6, 8.07), turned to 180 degrees
- moved C212 35.0 mm to (-20.0, 22.8)
- moved U204 34.9 mm to (-19.7, 25.6), turned to -90 degrees
- moved R202 33.9 mm to (-31.0, -2.17)
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Routing:
- net 5V_BAT: track 3.11 -> 7.46 mm
- net Net-(U203-OV2): track 2.22 -> 5.50 mm
- net /5 V / 3.3 V power/10V_GOOD: track 0.00 -> 2.94 mm
- net /USB service/USB_DP_CONN: track 5.26 -> 2.92 mm
- net 5V_USB: track 20.8 -> 18.5 mm
- net /USB service/USB_DM_CONN: track 5.18 -> 2.92 mm
- net Net-(U201-VCC): track 0.00 -> 2.17 mm
- net Net-(U203-OV1): track 3.40 -> 5.34 mm, vias 1 -> 0
- net /USB service/USB_CC2: track 1.93 -> 0.00 mm
- net Net-(U201-BOOT): track 0.00 -> 1.92 mm
- net Net-(U201-SW): track 0.00 -> 1.90 mm
- net GND: track 24.6 -> 26.1 mm
- net /USB service/USB_DM: track 6.28 -> 5.75 mm
- net VCC: vias 0 -> 1
- net USB_UART_RX: vias 2 -> 1
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
Commit message: CAN layout
Parts:
- removed C101, C102, C103, C110, C111, C112, C113, C114, C115, C116, C117, C118, C119, C120, C121, C122, C123, C124, C127, C128, C129, C130, C131, C132, C133, C134, C135, C136, C137, C138, C139, C140, C141, C144, C145, C147, C148, C149, C150, C151, C153, C154, C155, C156, C157, C158: 10uF, Capacitor_SMD:C_1210_3225Metric
- removed C104: 4.7uF 100V X7R, Capacitor_SMD:C_1210_3225Metric
- removed C105: 100nF 100V X7R, Capacitor_SMD:C_0402_1005Metric
- removed C106: 10nF 100V C0G, Capacitor_SMD:C_0402_1005Metric
- removed C125, C126, C142, C143, C159, C160: 10uF DNP, Capacitor_SMD:C_1210_3225Metric
- removed C414, C424, C434: 47pF C0G, Capacitor_SMD:C_0603_1608Metric
- removed JP801: TERM ENABLE, Jumper:SolderJumper-2_P1.3mm_Open_Pad1.0x1.5mm
- removed R101: 470k 0.25W, Resistor_SMD:R_1206_3216Metric
- removed TP1005: 5V_SYS, TestPoint:TestPoint_Pad_D1.0mm
- removed TP1006: 3V3, TestPoint:TestPoint_Pad_D1.0mm
- removed TP1008: SWDIO, TestPoint:TestPoint_Pad_D1.0mm
- removed TP1009: SWCLK, TestPoint:TestPoint_Pad_D1.0mm
- removed TP1010: ENC_SPI_CLK, TestPoint:TestPoint_Pad_D1.0mm
- removed TP1011: SPI3_MISO, TestPoint:TestPoint_Pad_D1.0mm
- removed TP1012: ENC_SPI_MOSI, TestPoint:TestPoint_Pad_D1.0mm
- removed TP1013: FDCAN1_TX, TestPoint:TestPoint_Pad_D1.0mm
- removed TP1014: FDCAN1_RX, TestPoint:TestPoint_Pad_D1.0mm
- removed TP1015: FEEDBACK_A_H1, TestPoint:TestPoint_Pad_D1.0mm
- removed TP1016: FEEDBACK_B_H2, TestPoint:TestPoint_Pad_D1.0mm
- removed TP1018: OPO_U1, TestPoint:TestPoint_Pad_D1.0mm
- removed TP1019: OPO_V1, TestPoint:TestPoint_Pad_D1.0mm
- removed TP1020: OPO_W1, TestPoint:TestPoint_Pad_D1.0mm
- removed TP1021: STATUS_LED_N, TestPoint:TestPoint_Pad_D1.0mm
- removed TP1022: CAN_STB, TestPoint:TestPoint_Pad_D1.0mm
- removed TP1023: EXT_SENSOR_FAULT_N, TestPoint:TestPoint_Pad_D1.0mm
- removed TP1024: I2C2_SDA, TestPoint:TestPoint_Pad_D1.0mm
- removed TP103: VBUS_SENSE, TestPoint:TestPoint_Pad_D1.5mm
- removed TP201: PWR_SOURCE_STATUS, TestPoint:TestPoint_Pad_D1.5mm
- removed TP202: 5V_USB, TestPoint:TestPoint_Pad_D1.5mm
- removed TP301: VCC, TestPoint:TestPoint_Pad_D1.5mm
- removed TP302: SCREF, TestPoint:TestPoint_Pad_D1.5mm
- removed TP303: NRST, TestPoint:TestPoint_Pad_D1.5mm
- removed TP411, TP421, TP431: GL, TestPoint:TestPoint_Pad_D1.0mm
- removed TP412, TP422, TP432: SOURCE, TestPoint:TestPoint_Pad_D1.0mm
- removed TP413, TP423, TP433: PHASE, TestPoint:TestPoint_Pad_D1.0mm
- removed TP414, TP424, TP434: SCOPE GND, TestPoint:TestPoint_Pad_D1.0mm
- removed TP501: BRAKE_GATE, TestPoint:TestPoint_Pad_D1.5mm
- removed TP502: BRAKE_SWITCH, TestPoint:TestPoint_Pad_D1.5mm
- removed TP701: NTC_PHASE_A, TestPoint:TestPoint_Pad_D1.0mm
- removed TP702: NTC_PHASE_B, TestPoint:TestPoint_Pad_D1.0mm
- removed TP703: NTC_PHASE_C, TestPoint:TestPoint_Pad_D1.0mm
- removed TP901: USB_UART_TX, TestPoint:TestPoint_Pad_D1.0mm
- removed TP902: USB_UART_RX, TestPoint:TestPoint_Pad_D1.0mm
- added Q301: BSS138AKM-Q, Package_TO_SOT_SMD:SOT-883, F.Cu at (-12.4, 26.4)
- added Q801: CSD17483F4, ShiroFOCLib:CSD17483F4_YJC0003A, B.Cu at (-12.9, 25.2)
- added Q802: CSD87502Q2, ShiroFOCLib:CSD87502Q2_DLV0006A, B.Cu at (-15.1, 27.6)
- added R315: 10k, Resistor_SMD:R_0402_1005Metric, F.Cu at (-7.28, 24.9)
- added R806: 10k, Resistor_SMD:R_0402_1005Metric, B.Cu at (-14.3, 25.2)
- C604, C801, C802, D801, R605, R606, R607, R801, R802, R805, U603: moved to B.Cu
- D301: value RED -> LTST-C19HE1WT; footprint LED_SMD:LED_0603_1608Metric -> LED_SMD:LED_LiteOn_LTST-C19HE1WT
- D601: value TPD3E001DRLR 3-line ESD -> TPD3E001DRYR; footprint Manual:TPD3E001_DRL5 -> ShiroFOCLib:TPD3E001_DRY6; moved to B.Cu
- L201: footprint Manual:WE_LHMI_7050_74437349470 -> ShiroFOCLib:WE_LHMI_7050_74437349470
- Q501: footprint Manual:CSD19531Q5A_Q5A_DQJ0008A -> ShiroFOCLib:CSD19531Q5A_Q5A_DQJ0008A
- R1, R3, R5: footprint Manual:R_Shunt_LR2512D_0m5_3W_Kelvin -> ShiroFOCLib:R_Shunt_LR2512D_0m5_3W_Kelvin
- R304: value 2.2k -> 15k
- R803: value 0R CANH link -> 4.7k; moved to B.Cu
- R804: value 0R CANL link -> 100k; moved to B.Cu
- U1, U2, U3: footprint Manual:DMM0022A -> ShiroFOCLib:DMM0022A
- U201: footprint Manual:LMR36510_DDA -> ShiroFOCLib:LMR36510_DDA
- U202: footprint Manual:USBLC6_SOT23_6 -> ShiroFOCLib:USBLC6_SOT23_6
- U203: footprint Manual:TPS2121_RUX -> ShiroFOCLib:TPS2121_RUX
- U204: footprint Manual:TLV75533_DYD_GND -> ShiroFOCLib:TLV75533_DYD_GND
- U205: footprint Manual:IC18_MPM3620AGQV-Z_MNP -> ShiroFOCLib:IC18_MPM3620AGQV-Z_MNP
- U4: footprint Manual:QFN_IN32G4_STM -> ShiroFOCLib:QFN_IN32G4_STM
- U501: footprint Manual:UCC27517A_DBV5 -> ShiroFOCLib:UCC27517A_DBV5
- U601: footprint Manual:AS5047P_TSSOP14 -> ShiroFOCLib:AS5047P_TSSOP14
- U602: footprint Manual:TMUX1574_PW16 -> ShiroFOCLib:TMUX1574_PW16
- U701: footprint Manual:BMI323_LGA14 -> ShiroFOCLib:BMI323_LGA14
- U801: value TCAN3413DR -> TCAN3413DRBR; footprint Package_SO:SOIC-8_3.9x4.9mm_P1.27mm -> ShiroFOCLib:TCAN3413_DRB8; moved to B.Cu
- moved SW301 123.6 mm to (-60.4, 47.6)
- moved J501 106.8 mm to (29.6, -15.2)
- moved J601 44.4 mm to (1.80, 29.2)
- moved D301 40.7 mm to (-9.21, 24.8), turned to 90 degrees
- moved R304 38.7 mm to (-11.6, 25.3)
- moved J802 34.7 mm to (-8.99, 29.2)
- moved J801 34.0 mm to (-18.5, 29.1)
- moved R802 33.0 mm to (-13.0, 27.3), turned to 90 degrees
- moved D601 32.2 mm to (1.18, 29.8), turned to -90 degrees
- moved R804 31.9 mm to (-11.6, 25.5)
- moved U602 31.9 mm to (10.6, 27.9)
- moved R803 31.4 mm to (-12.1, 24.1), turned to 180 degrees
- moved C604 30.8 mm to (-0.38, 30.2)
- moved R607 27.1 mm to (3.21, 28.9)
- moved U603 26.5 mm to (5.44, 29.1), turned to 90 degrees
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Connections:
- D301 pad 1: /MCU / clock / SWD/STATUS_LED_N -> Net-(D301-RK)
- D301 pad 2: Net-(D301-A) -> unconnected-(D301-GK-Pad2)
- D601 pad 5: /External feedback/FB_ESD_RAIL -> unconnected-(D601-NC-Pad5)
- D801 pad 1: /CAN interface/CANH_BUS -> /CAN interface/CANL_BUS
- D801 pad 2: /CAN interface/CANL_BUS -> /CAN interface/CANH_BUS
- J601 pad 3: Net-(D601-IO1) -> Net-(D601-IO3)
- J601 pad 5: Net-(D601-IO3) -> Net-(D601-IO1)
- J801 pad 2: /CAN interface/CANL_BUS -> /CAN interface/CANH_BUS
- J801 pad 3: /CAN interface/CANH_BUS -> /CAN interface/CANL_BUS
- J802 pad 2: /CAN interface/CANL_BUS -> /CAN interface/CANH_BUS
- J802 pad 3: /CAN interface/CANH_BUS -> /CAN interface/CANL_BUS
- R304 pad 1: 3V3 -> Net-(Q301-D)
- R304 pad 2: Net-(D301-A) -> Net-(D301-RK)
- R605 pad 1: Net-(D601-IO1) -> Net-(D601-IO3)
- R607 pad 1: Net-(D601-IO3) -> Net-(D601-IO1)
- R802 pad 2: /CAN interface/CAN_TERM_MID -> Net-(Q802A-D1)
- R803 pad 1: /CAN interface/CANH_INT -> CAN_TERM_DISABLE
- R803 pad 2: /CAN interface/CANH_BUS -> Net-(Q801-G)
- R804 pad 1: /CAN interface/CANL_INT -> Net-(Q801-G)
- R804 pad 2: /CAN interface/CANL_BUS -> GND
- U4 pad 5: /MCU / clock / SWD/STATUS_LED_N -> CAN_TERM_DISABLE
- U801 pad 6: /CAN interface/CANL_INT -> /CAN interface/CANL_BUS
- U801 pad 7: /CAN interface/CANH_INT -> /CAN interface/CANH_BUS
Routing:
- net /CAN interface/CANL_BUS: track 0.00 -> 25.8 mm, vias 0 -> 3
- net /CAN interface/CANH_BUS: track 0.00 -> 22.4 mm, vias 0 -> 1
- net /CAN interface/CAN_SHIELD: track 0.00 -> 11.5 mm
- net CAN_TERM_GATE: track 0.00 -> 9.59 mm, vias 0 -> 1
- net Net-(D601-IO1): track 0.00 -> 7.91 mm, vias 0 -> 1
- net Net-(D601-IO2): track 0.00 -> 7.56 mm, vias 0 -> 2
- net 3V3: track 1.47 -> 8.96 mm
- net GND: track 26.1 -> 31.0 mm, vias 6 -> 7
- net Net-(D601-IO3): track 0.00 -> 4.86 mm, vias 0 -> 1
- net Net-(R605-Pad2): track 0.00 -> 3.54 mm
- net Net-(Q802A-S1): track 0.00 -> 2.67 mm, vias 0 -> 2
- net Net-(Q802A-D1): track 0.00 -> 2.46 mm
- net Net-(R606-Pad2): track 0.00 -> 2.42 mm
- net Net-(R607-Pad2): track 0.00 -> 2.36 mm
- net Net-(Q801-G): track 0.00 -> 1.95 mm
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
Commit message: progress
Parts:
- removed C146, C152: 10uF, Capacitor_SMD:C_1210_3225Metric
- added D201: LTST-C19HE1WT, LED_SMD:LED_LiteOn_LTST-C19HE1WT, F.Cu at (-15.5, -17.2)
- added Q201: CSD17483F4, ShiroFOCLib:CSD17483F4_YJC0003A, B.Cu at (-14.9, -17.6)
- added R220: 10k, Resistor_SMD:R_0402_1005Metric, F.Cu at (-16.0, -18.8)
- added R221: 33k, Resistor_SMD:R_0402_1005Metric, B.Cu at (-16.2, -17.1)
- C203, C204, C210, C308, C309, C901, C902, C903, C904, J601, R201, R202, R203, R204, R309, R901, R902, R904, R905, U202, U901: moved to B.Cu
- C604, D601, JP601, R206, R208, R210, R212, R214, R215, R605, R606, R607, U602, U603: moved to F.Cu
- H1, H2, H3, H4: value M3 NPTH -> M2 PTH; footprint MountingHole:MountingHole_3.2mm_M3 -> MountingHole:MountingHole_2.2mm_M2_Pad_Via
- J1: value MOTOR U/V/W -> MR60PW-M; footprint Connector_AMASS:AMASS_MR30PW-M_1x03_P3.50mm_Horizontal -> ShiroFOCLib:AMASS_MR60PW-M_1x03_P5.50mm_Horizontal
- Q301: value BSS138AKM-Q -> CSD17483F4; footprint Package_TO_SOT_SMD:SOT-883 -> ShiroFOCLib:CSD17483F4_YJC0003A
- moved SW301 144.6 mm to (57.5, -36.1)
- moved C701 91.4 mm to (-72.4, 34.9)
- moved C702 91.4 mm to (-72.4, 33.1)
- moved R303 91.4 mm to (-69.6, 29.4)
- moved R308 91.4 mm to (-69.6, 36.4)
- moved R611 91.4 mm to (-63.0, 30.3)
- moved R713 91.4 mm to (-70.7, 43.8)
- moved R715 91.4 mm to (-70.5, 33.5)
- moved U701 91.4 mm to (-70.3, 33.7)
- moved Q501 76.9 mm to (13.2, -52.7), turned to 180 degrees
- moved D501 69.1 mm to (8.66, -53.1), turned to 90 degrees
- moved R504 67.0 mm to (8.88, -50.2), turned to 180 degrees
- moved R604 59.7 mm to (3.13, 30.3), turned to 90 degrees
- moved R503 56.3 mm to (6.44, -50.0)
- moved C503 51.5 mm to (-11.6, -40.2)
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Connections:
- R215 pad 1: 3V3 -> 5V_SYS
Routing:
- net USB_UART_RX: track 26.3 -> 1.39 mm, vias 1 -> 2
- net /USB service/UART_BRIDGE_RX: track 25.8 -> 4.90 mm, vias 1 -> 2
- net VCC: track 0.00 -> 19.3 mm, vias 2 -> 4
- net Net-(U602A-S3B): track 0.00 -> 13.0 mm
- net 3V3: track 8.96 -> 20.3 mm, vias 1 -> 5
- net /5 V / 3.3 V power/10V_GOOD: track 2.94 -> 12.7 mm, vias 1 -> 2
- net /USB service/CP2102_VBUS_SENSE: track 0.00 -> 9.01 mm, vias 0 -> 2
- net 5V_BAT: track 7.46 -> 0.00 mm, vias 1 -> 0
- net GND: track 31.0 -> 25.4 mm, vias 7 -> 9
- net Net-(U203-OV2): track 5.50 -> 1.13 mm
- net /USB service/USB_CC2: track 0.00 -> 4.16 mm, vias 0 -> 1
- net Net-(U203-OV1): track 5.34 -> 1.33 mm
- net Net-(U4A-PF1): track 0.48 -> 4.35 mm, vias 0 -> 1
- net VM: track 0.00 -> 3.68 mm
- net 5V_SYS: track 0.00 -> 3.65 mm
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Other:
- board size 65 x 65 mm -> 45 x 45 mm
- board text added: "55 x 55 mm"
