File: ShiroFOC/Manual_Layout_P3/ShiroFOC_Manual.kicad_pcb (KiCad board)
At the start: 6 copper layers, 45 x 45 mm, 228 parts, among them J1 MR60PW-M, J1001 TC2030-NL SWD, J101 AMASS XT60PW-M, J201 USB-C service, J501 BRAKE RESISTOR, J502 BRAKE NTC, J601 EXT ENCODER / HALL, J801 CAN 1, J802 CAN 2, Q201 CSD17483F4, Q301 CSD17483F4, Q501 CSD19531Q5A 100V, Q801 CSD17483F4, Q802 CSD87502Q2, SW301 RESET, U1 CSD88599Q5DC, U2 CSD88599Q5DC, U201 LMR36510FADDAR, U202 USBLC6-2SC6, U203 TPS2121RUXR, U204 TLV75533PDYDR, U205 MPM3620AGQV-Z, U3 CSD88599Q5DC, U4 STSPIN32G4, U501 UCC27517ADBVR, U502 TLV3012BIDBVR, U601 AS5047P-ATSM, U602 TMUX1574PW, U603 74LVC3G17, U604 TPS2553DBVR, U701 BMI323, U801 TCAN3413DRBR, U901 CP2102N-A02-GQFN20, Y301 24MHz 7pF

Commit message: progress + p4
Parts:
- removed D503: BAT54H, Diode_SMD:D_SOD-123F
- removed D505: BAT54S, Package_TO_SOT_SMD:SOT-23
- removed JP601: SENSOR SUPPLY, Jumper:SolderJumper-3_P1.3mm_Open_Pad1.0x1.5mm
- removed R608, R609, R610: 4.7k DNP, Resistor_SMD:R_0402_1005Metric
- removed TP101: VM, TestPoint:TestPoint_Pad_D1.5mm
- removed TP102: GND, TestPoint:TestPoint_Pad_D1.5mm
- removed TP104: VM BULK, TestPoint:TestPoint_Pad_D3.0mm
- removed TP105: GND BULK, TestPoint:TestPoint_Pad_D3.0mm
- added C101: 10uF, Capacitor_SMD:C_1210_3225Metric, F.Cu at (67.9, -11.3)
- added C102: 10uF, Capacitor_SMD:C_1210_3225Metric, F.Cu at (67.9, -7.01)
- added C103: 10uF, Capacitor_SMD:C_1210_3225Metric, F.Cu at (67.9, -2.76)
- added C104: 4.7uF 100V X7R, Capacitor_SMD:C_1210_3225Metric, F.Cu at (67.9, 1.49)
- added C105: 100nF 100V X7R, Capacitor_SMD:C_0402_1005Metric, F.Cu at (71.6, 24.9)
- added C106: 10nF 100V C0G, Capacitor_SMD:C_0402_1005Metric, F.Cu at (71.6, 26.9)
- added C110: 10uF, Capacitor_SMD:C_1210_3225Metric, F.Cu at (67.9, 5.74)
- added C111: 10uF, Capacitor_SMD:C_1210_3225Metric, F.Cu at (67.9, 9.99)
- added C112: 10uF, Capacitor_SMD:C_1210_3225Metric, F.Cu at (67.9, 14.2)
- added C113: 10uF, Capacitor_SMD:C_1210_3225Metric, F.Cu at (67.9, 18.5)
- added C114: 10uF, Capacitor_SMD:C_1210_3225Metric, F.Cu at (73.6, -11.3)
- added C115: 10uF, Capacitor_SMD:C_1210_3225Metric, F.Cu at (73.6, -7.01)
- added C116: 10uF, Capacitor_SMD:C_1210_3225Metric, F.Cu at (73.6, -2.76)
- added C117: 10uF, Capacitor_SMD:C_1210_3225Metric, F.Cu at (73.6, 1.49)
- added C118: 10uF, Capacitor_SMD:C_1210_3225Metric, F.Cu at (73.6, 5.74)
- added C119: 10uF, Capacitor_SMD:C_1210_3225Metric, F.Cu at (73.6, 9.99)
- added C120: 10uF, Capacitor_SMD:C_1210_3225Metric, F.Cu at (73.6, 14.2)
- added C121: 10uF, Capacitor_SMD:C_1210_3225Metric, F.Cu at (73.6, 18.5)
- added C122: 10uF, Capacitor_SMD:C_1210_3225Metric, F.Cu at (79.2, -11.3)
- added C123: 10uF, Capacitor_SMD:C_1210_3225Metric, F.Cu at (79.2, -7.01)
- added C124: 10uF, Capacitor_SMD:C_1210_3225Metric, F.Cu at (79.2, -2.76)
- added C125: 10uF DNP, Capacitor_SMD:C_1210_3225Metric, F.Cu at (79.2, 1.49)
- added C126: 10uF DNP, Capacitor_SMD:C_1210_3225Metric, F.Cu at (79.2, 5.74)
- added C127: 10uF, Capacitor_SMD:C_1210_3225Metric, F.Cu at (79.2, 9.99)
- added C128: 10uF, Capacitor_SMD:C_1210_3225Metric, F.Cu at (79.2, 14.2)
- added C129: 10uF, Capacitor_SMD:C_1210_3225Metric, F.Cu at (79.2, 18.5)
- added C130: 10uF, Capacitor_SMD:C_1210_3225Metric, F.Cu at (84.9, -11.3)
- added C131: 10uF, Capacitor_SMD:C_1210_3225Metric, F.Cu at (84.9, -7.01)
- added C132: 10uF, Capacitor_SMD:C_1210_3225Metric, F.Cu at (84.9, -2.76)
- added C133: 10uF, Capacitor_SMD:C_1210_3225Metric, F.Cu at (84.9, 1.49)
- added C134: 10uF, Capacitor_SMD:C_1210_3225Metric, F.Cu at (84.9, 5.74)
- added C135: 10uF, Capacitor_SMD:C_1210_3225Metric, F.Cu at (84.9, 9.99)
- added C136: 10uF, Capacitor_SMD:C_1210_3225Metric, F.Cu at (84.9, 14.2)
- added C137: 10uF, Capacitor_SMD:C_1210_3225Metric, F.Cu at (84.9, 18.5)
- added C138: 10uF, Capacitor_SMD:C_1210_3225Metric, F.Cu at (90.5, -11.3)
- added C139: 10uF, Capacitor_SMD:C_1210_3225Metric, F.Cu at (90.5, -7.01)
- added C140: 10uF, Capacitor_SMD:C_1210_3225Metric, F.Cu at (90.5, -2.76)
- added C141: 10uF, Capacitor_SMD:C_1210_3225Metric, F.Cu at (90.5, 1.49)
- added C142: 10uF DNP, Capacitor_SMD:C_1210_3225Metric, F.Cu at (90.5, 5.74)
- added C143: 10uF DNP, Capacitor_SMD:C_1210_3225Metric, F.Cu at (90.5, 9.99)
- added C144: 10uF, Capacitor_SMD:C_1210_3225Metric, F.Cu at (90.5, 14.2)
- added C145: 10uF, Capacitor_SMD:C_1210_3225Metric, F.Cu at (90.5, 18.5)
- added C146: 10uF, Capacitor_SMD:C_1210_3225Metric, F.Cu at (96.2, -11.3)
- added C147: 10uF, Capacitor_SMD:C_1210_3225Metric, F.Cu at (96.2, -7.01)
- added C148: 10uF, Capacitor_SMD:C_1210_3225Metric, F.Cu at (96.2, -2.76)
- added C149: 10uF, Capacitor_SMD:C_1210_3225Metric, F.Cu at (96.2, 1.49)
- added C150: 10uF, Capacitor_SMD:C_1210_3225Metric, F.Cu at (96.2, 5.74)
- added C151: 10uF, Capacitor_SMD:C_1210_3225Metric, F.Cu at (96.2, 9.99)
- added C152: 10uF, Capacitor_SMD:C_1210_3225Metric, F.Cu at (96.2, 14.2)
- added C153: 10uF, Capacitor_SMD:C_1210_3225Metric, F.Cu at (96.2, 18.5)
- added C154: 10uF, Capacitor_SMD:C_1210_3225Metric, F.Cu at (101.8, -11.3)
- added C155: 10uF, Capacitor_SMD:C_1210_3225Metric, F.Cu at (101.8, -7.01)
- added C156: 10uF, Capacitor_SMD:C_1210_3225Metric, F.Cu at (101.8, -2.76)
- added C157: 10uF, Capacitor_SMD:C_1210_3225Metric, F.Cu at (101.8, 1.49)
- added C158: 10uF, Capacitor_SMD:C_1210_3225Metric, F.Cu at (101.8, 5.74)
- added C159: 10uF DNP, Capacitor_SMD:C_1210_3225Metric, F.Cu at (101.8, 9.99)
- added C160: 10uF DNP, Capacitor_SMD:C_1210_3225Metric, F.Cu at (101.8, 14.2)
- added C506: 4.7uF, Capacitor_SMD:C_0603_1608Metric, F.Cu at (1.59, 38.2)
- added R101: 470k 0.25W, Resistor_SMD:R_1206_3216Metric, F.Cu at (72.9, 22.3)
- added R618: 49.9k 1%, Resistor_SMD:R_0402_1005Metric, F.Cu at (-9.70, 34.4)
- added U503: 74AHCT1G125W5-7, Package_TO_SOT_SMD:SOT-23-5, F.Cu at (-5.26, 31.0)
- C210, J601: moved to F.Cu
- C504: footprint Capacitor_SMD:C_0603_1608Metric -> Capacitor_SMD:C_0402_1005Metric
- C505: value 100nF 16V -> 100nF
- C604, R501, R502, R503, R504, R505, R506, R510, R604, R605, R606, R607, U501, U602, U603: moved to B.Cu
- C606: value 4.7uF 16V X7R -> 4.7uF
- D502: value BAT54H -> BAT54CM; footprint Diode_SMD:D_SOD-123F -> Package_TO_SOT_SMD:SOT-883; moved to B.Cu
- J1: value MR60PW-M -> Motor phases - solder wires; footprint ShiroFOCLib:AMASS_MR60PW-M_1x03_P5.50mm_Horizontal -> ShiroFOCLib:WireSolder_Phase_1x03_P6.35mm_D2.90mm_Pad4.10mm
- J101: value AMASS XT60PW-M -> DC input - solder wires; footprint Connector_AMASS:AMASS_XT60PW-M_1x02_P7.20mm_Horizontal -> ShiroFOCLib:WireSolder_DC_1x02_P6.35mm_D2.70mm_Pad4.10mm
- J501: footprint Connector_Wire:SolderWire-2sqmm_1x02_P7.8mm_D2mm_OD3.9mm -> Connector_Wire:SolderWire-0.75sqmm_1x02_P4.8mm_D1.25mm_OD2.3mm
- J502: value BRAKE NTC -> 5V PWM FAN; footprint Connector_JST:JST_GH_SM02B-GHS-TB_1x02-1MP_P1.25mm_Horizontal -> Connector_JST:JST_GH_SM04B-GHS-TB_1x04-1MP_P1.25mm_Horizontal; moved to F.Cu
- Q501: value CSD19531Q5A 100V -> ISZ080N10NM6 100V; footprint ShiroFOCLib:CSD19531Q5A_Q5A_DQJ0008A -> ShiroFOCLib:ISZ080N10NM6_TSDSON8_FL
- R206: value 15.0k 1% -> 10.0k 1%
- R208: value 10.0k 1% -> 15.0k 1%
- R511: value 10k 1% -> 100R
- R512: value 4.7k 1% -> 100k
- U502: value TLV3012BIDBVR -> TLV3012BIDCKR; footprint Package_TO_SOT_SMD:SOT-23-6 -> Package_TO_SOT_SMD:SOT-363_SC-70-6; moved to B.Cu
- moved J502 88.2 mm to (-1.56, 19.3), turned to 0 degrees
- moved R611 71.8 mm to (1.11, -2.01)
- moved R713 55.9 mm to (-15.3, 36.3), turned to 180 degrees
- moved R105 52.5 mm to (-0.10, 19.1), turned to 180 degrees
- moved R106 52.1 mm to (1.35, 19.9), turned to -90 degrees
- moved R103 50.0 mm to (-0.66, 20.4), turned to 0 degrees
- moved R617 46.0 mm to (-14.2, 17.4), turned to 90 degrees
- moved R616 44.4 mm to (-15.6, 19.9), turned to 180 degrees
- moved R615 42.0 mm to (-15.6, 21.8), turned to 180 degrees
- moved C501 40.6 mm to (11.2, -10.5), turned to 180 degrees
- moved D501 39.8 mm to (10.7, -13.4), turned to 180 degrees
- moved C502 39.6 mm to (11.2, -11.7), turned to 180 degrees
- moved R505 37.8 mm to (10.1, -10.3), turned to 0 degrees
- moved R504 37.5 mm to (12.9, -13.0), turned to -90 degrees
- moved U501 37.1 mm to (10.7, -12.9), turned to 90 degrees
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Connections:
- net EXT_SENSOR_FAULT_N renamed EXT_POWER_FAULT_N
- C505 pad 1: NTC_BRAKE -> EXT_VCC
- C606 pad 1: /External feedback/EXT_SUPPLY_SELECTED -> 5V_SYS
- C607 pad 1: /External feedback/EXT_VCC -> EXT_VCC
- D502 pad 1: /Brake chopper/BRAKE_PWM_DRV -> Net-(D502-A1)
- D502 pad 2: Net-(D502-A) -> /Brake chopper/BRAKE_OV_CMD
- D601 pad 5: unconnected-(D601-NC-Pad5) -> Net-(D601-IO2)
- J501 pad 1: VM -> Net-(J501-Pad1)
- J501 pad 2: Net-(J501-Pad2) -> VM
- J502 pad 1: /Brake chopper/BRAKE_NTC_RAW -> GND
- J502 pad 2: GND -> EXT_VCC
- J502 pad MP: (no net) -> GND
- J601 pad 1: /External feedback/EXT_VCC -> EXT_VCC
- J601 pad 6: unconnected-(J601-Pad6) -> GND
- J601 pad MP: (no net) -> GND
- J801 pad MP: (no net) -> GND
- J802 pad MP: (no net) -> GND
- Q501 pad 5: Net-(J501-Pad2) -> Net-(J501-Pad1)
- Q501 pad 6: Net-(J501-Pad2) -> Net-(J501-Pad1)
- Q501 pad 7: Net-(J501-Pad2) -> Net-(J501-Pad1)
- Q501 pad 8: Net-(J501-Pad2) -> Net-(J501-Pad1)
- R502 pad 2: Net-(D502-A) -> Net-(D502-A1)
- R511 pad 1: 3V3 -> FAN_PWM
- R511 pad 2: /Brake chopper/BRAKE_NTC_RAW -> Net-(U503-A)
- R512 pad 1: /Brake chopper/BRAKE_NTC_RAW -> Net-(U503-A)
- R512 pad 2: NTC_BRAKE -> GND
- U4 pad 10: NTC_BRAKE -> FAN_PWM
- U604 pad 1: /External feedback/EXT_SUPPLY_SELECTED -> 5V_SYS
- U604 pad 3: /External feedback/EXT_SUPPLY_SELECTED -> 5V_SYS
- U604 pad 5: /External feedback/EXT_SUPPLY_SELECTED -> Net-(U604-ILIM)
- U604 pad 6: /External feedback/EXT_VCC -> EXT_VCC
Routing:
- net VM: track 3.68 -> 18.1 mm
- net GHS1: track 16.9 -> 2.48 mm
- net GND: track 25.4 -> 19.4 mm, vias 9 -> 12
- net Net-(U502-IN+): track 5.88 -> 0.00 mm, vias 0 -> 1
- net 5V_USB: track 22.0 -> 17.1 mm
- net Net-(D601-IO3): track 7.17 -> 11.7 mm, vias 1 -> 2
- net /Brake chopper/BRAKE_OV_CMD: track 4.44 -> 0.00 mm
- net Net-(U602A-S2B): track 3.05 -> 0.00 mm
- net Net-(D601-IO2): track 6.01 -> 8.59 mm, vias 1 -> 2
- net Net-(U602A-S1B): track 2.53 -> 0.00 mm
- net (no net): track 0.00 -> 2.16 mm
- net I2C2_SCL: track 2.13 -> 0.00 mm
- net Net-(U602A-S3B): track 13.0 -> 11.5 mm, vias 0 -> 2
- net NTC_BRAKE: track 1.40 -> 0.00 mm, vias 1 -> 0
- net NTC_PHASE_C: track 1.38 -> 0.00 mm, vias 1 -> 0
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