File: ShiroFOC/Manual_Layout_P3/04_Gate_Driver.kicad_sch (KiCad schematic)
At the start: 13 parts, among them U4 STSPIN32G4

Commit message: CAN layout
Parts:
- C311: symbol Manual:COMP_C311 -> ShiroFOCLib:COMP_C311
- C312: symbol Manual:COMP_C312 -> ShiroFOCLib:COMP_C312
- C313: symbol Manual:COMP_C313 -> ShiroFOCLib:COMP_C313
- C314: symbol Manual:COMP_C314 -> ShiroFOCLib:COMP_C314
- R310: symbol Manual:COMP_R310 -> ShiroFOCLib:COMP_R310
- R311: symbol Manual:COMP_R311 -> ShiroFOCLib:COMP_R311
- R312: symbol Manual:COMP_R312 -> ShiroFOCLib:COMP_R312
- TP301: symbol Manual:COMP_TP301 -> ShiroFOCLib:COMP_TP301
- TP302: symbol Manual:COMP_TP302 -> ShiroFOCLib:COMP_TP302
- U4: footprint Manual:QFN_IN32G4_STM -> ShiroFOCLib:QFN_IN32G4_STM; symbol Manual:STSPIN32G4_Functional -> ShiroFOCLib:STSPIN32G4_Functional
Changed lines of the file:
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@@
 	)
 	(symbol
-		(lib_id "Manual:FLAG")
+		(lib_id "ShiroFOCLib:FLAG")
 		(at 176.53 127 0)
 		(unit 1)
@@
 	)
 	(symbol
-		(lib_id "Manual:PWR_VM")
+		(lib_id "ShiroFOCLib:PWR_VM")
 		(at 137.16 88.9 0)
 		(unit 1)
@@
 	)
 	(symbol
-		(lib_id "Manual:PWR_GND")
+		(lib_id "ShiroFOCLib:PWR_GND")
 		(at 137.16 123.19 0)
 		(unit 1)
@@
 	)
 	(symbol
-		(lib_id "Manual:COMP_TP302")
+		(lib_id "ShiroFOCLib:COMP_TP302")
 		(at 140.97 189.23 0)
 		(unit 1)
@@
 	)
 	(symbol
-		(lib_id "Manual:PWR_GND")
+		(lib_id "ShiroFOCLib:PWR_GND")
 		(at 210.82 217.17 0)
 		(unit 1)
@@
 	)
 	(symbol
-		(lib_id "Manual:FLAG")
+		(lib_id "ShiroFOCLib:FLAG")
 		(at 176.53 144.78 0)
 		(unit 1)
@@
 	)
 	(symbol
-		(lib_id "Manual:PWR_GND")
+		(lib_id "ShiroFOCLib:PWR_GND")
 		(at 53.34 208.28 0)
 		(unit 1)
@@
 	)
 	(symbol
-		(lib_id "Manual:COMP_R310")
+		(lib_id "ShiroFOCLib:COMP_R310")
 		(at 53.34 166.37 0)
 		(unit 1)
@@
 	)
 	(symbol
-		(lib_id "Manual:COMP_C314")
+		(lib_id "ShiroFOCLib:COMP_C314")
 		(at 129.54 207.01 0)
 		(unit 1)
@@
 	)
 	(symbol
-		(lib_id "Manual:STSPIN32G4_Functional")
+		(lib_id "ShiroFOCLib:STSPIN32G4_Functional")
 		(at 210.82 153.67 0)
 		(unit 3)
@@
 			)
 		)
-		(property "Footprint" "Manual:QFN_IN32G4_STM"
+		(property "Footprint" "ShiroFOCLib:QFN_IN32G4_STM"
 			(at 210.82 217.17 0)
 			(effects
@@
 	)
 	(symbol
-		(lib_id "Manual:COMP_C311")
+		(lib_id "ShiroFOCLib:COMP_C311")
 		(at 137.16 110.49 0)
 		(unit 1)
@@
 	)
 	(symbol
-		(lib_id "Manual:COMP_C312")
+		(lib_id "ShiroFOCLib:COMP_C312")
 		(at 339.09 100.33 0)
 		(unit 1)
@@
 	)
 	(symbol
-		(lib_id "Manual:PWR_GND")
+		(lib_id "ShiroFOCLib:PWR_GND")
 		(at 339.09 111.76 0)
 		(unit 1)
@@
 	)
 	(symbol
-		(lib_id "Manual:PWR_VCC")
+		(lib_id "ShiroFOCLib:PWR_VCC")
 		(at 370.84 55.88 0)
 		(unit 1)
@@
 	)
 	(symbol
-		(lib_id "Manual:FLAG")
+		(lib_id "ShiroFOCLib:FLAG")
 		(at 19.05 281.94 0)
 		(unit 1)
@@
 	)
 	(symbol
-		(lib_id "Manual:COMP_R311")
+		(lib_id "ShiroFOCLib:COMP_R311")
 		(at 53.34 195.58 0)
 		(unit 1)
@@
 	)
 	(symbol
-		(lib_id "Manual:COMP_C313")
+		(lib_id "ShiroFOCLib:COMP_C313")
 		(at 370.84 100.33 0)
 		(unit 1)
@@
 	)
 	(symbol
-		(lib_id "Manual:PWR_GND")
+		(lib_id "ShiroFOCLib:PWR_GND")
 		(at 370.84 111.76 0)
 		(unit 1)
@@
 	)
 	(symbol
-		(lib_id "Manual:COMP_TP301")
+		(lib_id "ShiroFOCLib:COMP_TP301")
 		(at 355.6 76.2 0)
 		(unit 1)
@@
 	)
 	(symbol
-		(lib_id "Manual:PWR_3V3")
+		(lib_id "ShiroFOCLib:PWR_3V3")
 		(at 53.34 151.13 0)
 		(unit 1)
@@
 	)
 	(symbol
-		(lib_id "Manual:COMP_R312")
+		(lib_id "ShiroFOCLib:COMP_R312")
 		(at 96.52 181.61 0)
 		(unit 1)
@@
 	)
 	(symbol
-		(lib_id "Manual:FLAG")
+		(lib_id "ShiroFOCLib:FLAG")
 		(at 176.53 162.56 0)
 		(unit 1)
@@
 	)
 	(symbol
-		(lib_id "Manual:PWR_GND")
+		(lib_id "ShiroFOCLib:PWR_GND")
 		(at 129.54 218.44 0)
 		(unit 1)
