File: ShiroFOC/Manual_Layout_P3/07_Brake_Chopper.kicad_sch (KiCad schematic)
At the start: 29 parts, among them J501 BRAKE RESISTOR, J502 BRAKE NTC, Q501 CSD19531Q5A 100V, U501 UCC27517ADBVR, U502 TLV3012BIDBVR

Commit message: pcb layout blocks
Parts:
- removed D504: B5100C 100V 5A, Diode_SMD:D_SMC, symbol Manual:COMP_D504
- removed R507: 150k 0.1% 200V, Resistor_SMD:R_1206_3216Metric, symbol Manual:COMP_R507
- removed R508: 150k 0.1% 200V, Resistor_SMD:R_1206_3216Metric, symbol Manual:COMP_R508
- C504: Selection Note Divider noise filter, nominal 12.2us time constant. Adds re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 -> Divider noise filter, nominal 12.8us time constant with 470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
- R506: value 150k 0.1% 200V -> 470k 1% 75V; footprint Resistor_SMD:R_1206_3216Metric -> Resistor_SMD:R_0603_1608Metric; LCSC (none) -> C114622; MPN RT1206BRD07150KL -> RC0603FR-07470KL; Procurement Select to specification: 150k 0.1% 100V; R_1206_3216Metric -> RC0603FR-07470KL; 470k 1%; 0603; 75V continuous rating; Rating 0.1%; 25ppm/K; 0.25W; 200V -> 1%; 100ppm/K; 0.1W; 75V continuous; Selection Note Three series resistors form 450k high-side divider; about 1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 -> Single upper divider resistor replaces R506-R508; about 44.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
- R509: value 12.7k 0.1% -> 13.3k 1%; LCSC (none) -> C274352; MPN (none) -> RC0402FR-0713K3L; Procurement 0402; preserve Value/tolerance requirements; exact part not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 -> RC0402FR-0713K3L; 13.3k 1%; 0402; Rating 0.1%; 25ppm/K; 0.1W; 75V -> 1%; 100ppm/K; 0.063W; 50V; Selection Note Divider lower leg; threshold approximately 45.9V rising wit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 -> Divider lower leg; nominal threshold 45.8V rising with R506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
- R510: value 1M 0.1% -> 1M 1%; LCSC (none) -> C138033; MPN (none) -> RC0402FR-071ML; Procurement 0402; preserve Value/tolerance requirements; exact part not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 -> RC0402FR-071ML; 1M 1%; 0402; Rating 0.1%; 25ppm/K; 0.1W; 75V -> 1%; 100ppm/K; 0.063W; 50V; Selection Note Positive feedback; release threshold approximately 44.2V. N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 -> Positive feedback; nominal release threshold 44.1V with R50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
- U502: Nominal Thresholds ON 45.9V; OFF 44.2V; tolerances and dynamic overshoot apply -> ON 45.8V; OFF 44.1V; 1% resistor-only ON corners 44.94-46.7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
Connections:
- net at C504.1, R509.1, R510.2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: now also R506.2
Other:
- note added: "U502: nominal ON 45.8 V / OFF 44.1 V. Board-bus backup only; thresholds have tolerance and dynamic overshoot."
- note removed: "U502: nominal ON 45.9 V / OFF 44.2 V. Board-bus backup only; thresholds have tolerance and dynamic overshoot."
- moved on the sheet: R506

Commit message: CAN layout
Parts:
- C501: symbol Manual:COMP_C501 -> ShiroFOCLib:COMP_C501
- C502: symbol Manual:COMP_C502 -> ShiroFOCLib:COMP_C502
- C503: symbol Manual:COMP_C503 -> ShiroFOCLib:COMP_C503
- C504: symbol Manual:COMP_C504 -> ShiroFOCLib:COMP_C504
- D501: symbol Manual:COMP_D501 -> ShiroFOCLib:COMP_D501
- D502: symbol Manual:COMP_D502 -> ShiroFOCLib:COMP_D502
- D503: symbol Manual:COMP_D503 -> ShiroFOCLib:COMP_D503
- J501: symbol Manual:COMP_J501 -> ShiroFOCLib:COMP_J501
- Q501: footprint Manual:CSD19531Q5A_Q5A_DQJ0008A -> ShiroFOCLib:CSD19531Q5A_Q5A_DQJ0008A; symbol Manual:COMP_Q501 -> ShiroFOCLib:COMP_Q501
- R501: symbol Manual:COMP_R501 -> ShiroFOCLib:COMP_R501
- R502: symbol Manual:COMP_R502 -> ShiroFOCLib:COMP_R502
- R503: symbol Manual:COMP_R503 -> ShiroFOCLib:COMP_R503
- R504: symbol Manual:COMP_R504 -> ShiroFOCLib:COMP_R504
- R505: symbol Manual:COMP_R505 -> ShiroFOCLib:COMP_R505
- R506: symbol Manual:COMP_R506 -> ShiroFOCLib:COMP_R506
- R509: symbol Manual:COMP_R509 -> ShiroFOCLib:COMP_R509
- R510: symbol Manual:COMP_R510 -> ShiroFOCLib:COMP_R510
- TP501: symbol Manual:COMP_TP501 -> ShiroFOCLib:COMP_TP501
- TP502: symbol Manual:COMP_TP502 -> ShiroFOCLib:COMP_TP502
- U501: footprint Manual:UCC27517A_DBV5 -> ShiroFOCLib:UCC27517A_DBV5; symbol Manual:COMP_U501 -> ShiroFOCLib:COMP_U501
- U502: symbol Manual:COMP_U502 -> ShiroFOCLib:COMP_U502
Changed lines of the file:
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@@
 	)
 	(symbol
-		(lib_id "Manual:COMP_U501")
+		(lib_id "ShiroFOCLib:COMP_U501")
 		(at 220.98 127 0)
 		(unit 1)
@@
 			)
 		)
-		(property "Footprint" "Manual:UCC27517A_DBV5"
+		(property "Footprint" "ShiroFOCLib:UCC27517A_DBV5"
 			(at 220.98 147.32 0)
 			(effects
@@
 	)
 	(symbol
-		(lib_id "Manual:COMP_R509")
+		(lib_id "ShiroFOCLib:COMP_R509")
 		(at 38.1 198.12 0)
 		(unit 1)
@@
 	)
 	(symbol
-		(lib_id "Manual:COMP_D501")
+		(lib_id "ShiroFOCLib:COMP_D501")
 		(at 270.51 160.02 0)
 		(unit 1)
@@
 	)
 	(symbol
-		(lib_id "Manual:PWR_GND")
+		(lib_id "ShiroFOCLib:PWR_GND")
 		(at 304.8 177.8 0)
 		(unit 1)
@@
 	)
 	(symbol
-		(lib_id "Manual:COMP_Q501")
+		(lib_id "ShiroFOCLib:COMP_Q501")
 		(at 304.8 127 0)
 		(unit 1)
@@
 			)
 		)
-		(property "Footprint" "Manual:CSD19531Q5A_Q5A_DQJ0008A"
+		(property "Footprint" "ShiroFOCLib:CSD19531Q5A_Q5A_DQJ0008A"
 			(at 304.8 144.78 0)
 			(effects
@@
 	)
 	(symbol
-		(lib_id "Manual:PWR_VCC")
+		(lib_id "ShiroFOCLib:PWR_VCC")
 		(at 191.77 78.74 0)
 		(unit 1)
@@
 	)
 	(symbol
-		(lib_id "Manual:PWR_GND")
+		(lib_id "ShiroFOCLib:PWR_GND")
 		(at 243.84 106.68 0)
 		(unit 1)
@@
 	)
 	(symbol
-		(lib_id "Manual:COMP_R501")
+		(lib_id "ShiroFOCLib:COMP_R501")
 		(at 44.45 69.85 0)
 		(unit 1)
@@
 	)
 	(symbol
-		(lib_id "Manual:COMP_R510")
+		(lib_id "ShiroFOCLib:COMP_R510")
 		(at 96.52 132.08 0)
 		(unit 1)
@@
 	)
 	(symbol
-		(lib_id "Manual:PWR_3V3")
+		(lib_id "ShiroFOCLib:PWR_3V3")
 		(at 96.52 142.24 0)
 		(unit 1)
@@
 	)
 	(symbol
-		(lib_id "Manual:PWR_GND")
+		(lib_id "ShiroFOCLib:PWR_GND")
 		(at 228.6 232.41 0)
 		(unit 1)
@@
 	)
 	(symbol
-		(lib_id "Manual:COMP_C504")
+		(lib_id "ShiroFOCLib:COMP_C504")
 		(at 55.88 198.12 0)
 		(unit 1)
@@
 	)
 	(symbol
-		(lib_id "Manual:COMP_R506")
+		(lib_id "ShiroFOCLib:COMP_R506")
 		(at 38.1 146.05 0)
 		(unit 1)
@@
 	)
 	(symbol
-		(lib_id "Manual:COMP_R505")
+		(lib_id "ShiroFOCLib:COMP_R505")
 		(at 172.72 92.71 0)
 		(unit 1)
@@
 	)
 	(symbol
-		(lib_id "Manual:PWR_VM")
+		(lib_id "ShiroFOCLib:PWR_VM")
 		(at 269.24 48.26 0)
 		(unit 1)
@@
 	)
 	(symbol
-		(lib_id "Manual:COMP_C502")
+		(lib_id "ShiroFOCLib:COMP_C502")
 		(at 243.84 92.71 0)
 		(unit 1)
@@
 	)
 	(symbol
-		(lib_id "Manual:COMP_D502")
+		(lib_id "ShiroFOCLib:COMP_D502")
 		(at 88.9 50.8 0)
 		(unit 1)
@@
 	)
 	(symbol
-		(lib_id "Manual:PWR_GND")
+		(lib_id "ShiroFOCLib:PWR_GND")
 		(at 38.1 214.63 0)
 		(unit 1)
@@
 	)
 	(symbol
-		(lib_id "Manual:COMP_U502")
+		(lib_id "ShiroFOCLib:COMP_U502")
 		(at 96.52 186.69 0)
 		(unit 1)
@@
 	)
 	(symbol
-		(lib_id "Manual:COMP_TP502")
+		(lib_id "ShiroFOCLib:COMP_TP502")
 		(at 317.5 96.52 0)
 		(unit 1)
@@
 	)
 	(symbol
-		(lib_id "Manual:PWR_GND")
+		(lib_id "ShiroFOCLib:PWR_GND")
 		(at 289.56 232.41 0)
 		(unit 1)
@@
 	)
 	(symbol
-		(lib_id "Manual:PWR_GND")
+		(lib_id "ShiroFOCLib:PWR_GND")
 		(at 185.42 149.86 0)
 		(unit 1)
@@
 	)
 	(symbol
-		(lib_id "Manual:COMP_D503")
+		(lib_id "ShiroFOCLib:COMP_D503")
 		(at 153.67 80.01 0)
 		(unit 1)
@@
 	)
 	(symbol
-		(lib_id "Manual:PWR_GND")
+		(lib_id "ShiroFOCLib:PWR_GND")
 		(at 320.04 232.41 0)
 		(unit 1)
@@
 	)
 	(symbol
-		(lib_id "Manual:COMP_R502")
+		(lib_id "ShiroFOCLib:COMP_R502")
 		(at 66.04 50.8 0)
 		(unit 1)
@@
 	)
 	(symbol
-		(lib_id "Manual:PWR_3V3")
+		(lib_id "ShiroFOCLib:PWR_3V3")
 		(at 320.04 190.5 0)
 		(unit 1)
@@
 	)
 	(symbol
-		(lib_id "Manual:COMP_C501")
+		(lib_id "ShiroFOCLib:COMP_C501")
 		(at 210.82 92.71 0)
 		(unit 1)
@@
 	)
 	(symbol
-		(lib_id "Manual:PWR_GND")
+		(lib_id "ShiroFOCLib:PWR_GND")
 		(at 121.92 165.1 0)
 		(unit 1)
@@
 	)
 	(symbol
-		(lib_id "Manual:PWR_GND")
+		(lib_id "ShiroFOCLib:PWR_GND")
 		(at 172.72 105.41 0)
 		(unit 1)
@@
 	)
 	(symbol
-		(lib_id "Manual:PWR_VM")
+		(lib_id "ShiroFOCLib:PWR_VM")
 		(at 38.1 115.57 0)
 		(unit 1)
@@
 	)
 	(symbol
-		(lib_id "Manual:PWR_GND")
+		(lib_id "ShiroFOCLib:PWR_GND")
 		(at 96.52 210.82 0)
 		(unit 1)
@@
 	)
 	(symbol
-		(lib_id "Manual:COMP_R504")
+		(lib_id "ShiroFOCLib:COMP_R504")
 		(at 288.29 160.02 0)
 		(unit 1)
@@
 	)
 	(symbol
-		(lib_id "Manual:PWR_GND")
+		(lib_id "ShiroFOCLib:PWR_GND")
 		(at 44.45 82.55 0)
 		(unit 1)
@@
 	)
 	(symbol
-		(lib_id "Manual:COMP_C503")
+		(lib_id "ShiroFOCLib:COMP_C503")
 		(at 121.92 153.67 0)
 		(unit 1)
@@
 	)
 	(symbol
-		(lib_id "Manual:COMP_R503")
+		(lib_id "ShiroFOCLib:COMP_R503")
 		(at 267.97 127 0)
 		(unit 1)
@@
 	)
 	(symbol
-		(lib_id "Manual:COMP_TP501")
+		(lib_id "ShiroFOCLib:COMP_TP501")
 		(at 280.67 127 0)
 		(unit 1)
@@
 	)
 	(symbol
-		(lib_id "Manual:PWR_3V3")
+		(lib_id "ShiroFOCLib:PWR_3V3")
 		(at 241.3 190.5 0)
 		(unit 1)
@@
 	)
 	(symbol
-		(lib_id "Manual:COMP_J501")
+		(lib_id "ShiroFOCLib:COMP_J501")
 		(at 303.53 63.5 0)
 		(unit 1)

Commit message: progress + p4
Parts:
- removed D503: BAT54H, Diode_SMD:D_SOD-123F, symbol ShiroFOCLib:COMP_D503
- removed D505: BAT54S, Package_TO_SOT_SMD:SOT-23, symbol Diode:BAT54S
- added C506: 4.7uF, Capacitor_SMD:C_0603_1608Metric, symbol ShiroFOCLib:COMP_C603
- added U503: 74AHCT1G125W5-7, Package_TO_SOT_SMD:SOT-23-5, symbol ShiroFOCLib:74AHCT1G125_SOT25
- C504: footprint Capacitor_SMD:C_0603_1608Metric -> Capacitor_SMD:C_0402_1005Metric; MPN C1608C0G1H102J080AA -> CGA2B2C0G1H102J050BA; Procurement Select to specification: 1nF C0G; C_0603_1608Metric -> TDK CGA2B2C0G1H102J050BA; 0402; 1nF C0G 50V 5%
- C505: value 100nF 16V -> 100nF; Rating (none) -> 100nF, 16V, X7R, 0402
- D502: value BAT54H -> BAT54CM; footprint Diode_SMD:D_SOD-123F -> Package_TO_SOT_SMD:SOT-883; symbol ShiroFOCLib:COMP_D502 -> ShiroFOCLib:BAT54CM; MPN BAT54H,115 -> BAT54CM,315; Manufacturer (none) -> Nexperia; Rating See Value; generic low-voltage passives: R >=0.1 W / 50 V, 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 -> 30V; 200mA per diode; common cathode; DFN1006-3 (SOT883); Selection Note (none) -> Dual diode D502 replaces the separate D502/D503 command OR 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
- J501: footprint Connector_Wire:SolderWire-2sqmm_1x02_P7.8mm_D2mm_OD3.9mm -> Connector_Wire:SolderWire-0.75sqmm_1x02_P4.8mm_D1.25mm_OD2.3mm; Procurement Select to specification: BRAKE RESISTOR; SolderWire-2sqmm_1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 -> Select to specification: BRAKE RESISTOR; SolderWire-0.75sqm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
- J502: value BRAKE NTC -> 5V PWM FAN; footprint Connector_JST:JST_GH_SM02B-GHS-TB_1x02-1MP_P1.25mm_Horizontal -> Connector_JST:JST_GH_SM04B-GHS-TB_1x04-1MP_P1.25mm_Horizontal; symbol Connector_Generic:Conn_01x02 -> ShiroFOCLib:Fan_PWM_JST_GH_4; BOM Comments (none) -> 1=GND; 2=EXT_VCC continuous protected 5V; 3=tach NC; 4=FAN_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; MPN SM02B-GHS-TB(LF)(SN) -> SM04B-GHS-TB(LF)(SN); Manufacturer (none) -> JST; Rating (none) -> JST GH 1.25mm, 4 contacts, right angle
- Q501: value CSD19531Q5A 100V -> ISZ080N10NM6 100V; footprint ShiroFOCLib:CSD19531Q5A_Q5A_DQJ0008A -> ShiroFOCLib:ISZ080N10NM6_TSDSON8_FL; MPN CSD19531Q5A -> ISZ080N10NM6ATMA1; Manufacturer (none) -> Infineon Technologies; Rating See Value; generic low-voltage passives: R >=0.1 W / 50 V, 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 -> 100V VDS; +/-20V VGS; RDS(on) <=8.04mOhm at VGS=10V, 25C; Selection Note (none) -> 3.3x3.3mm fused-lead package; conduction loss about 0.17W a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
- R511: value 10k 1% -> 100R; Rating (none) -> 100R, 0402
- R512: value 4.7k 1% -> 100k; Rating (none) -> 100k, 0402
- U501: Manufacturer (none) -> Texas Instruments; Rating See Value; generic low-voltage passives: R >=0.1 W / 50 V, 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 -> 4.5-18V supply; 4A peak source/sink; input absolute limits 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
- U502: value TLV3012BIDBVR -> TLV3012BIDCKR; footprint Package_TO_SOT_SMD:SOT-23-6 -> Package_TO_SOT_SMD:SOT-363_SC-70-6; MPN TLV3012BIDBVR -> TLV3012BIDCKR; Manufacturer (none) -> Texas Instruments; Rating See Value; generic low-voltage passives: R >=0.1 W / 50 V, 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 -> 1.65-5.5V supply; internal 1.242V reference; push-pull comp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
Connections:
- net 3V3: no longer R511.1
- net BRAKE_OV_CMD: now also D502.2 (A2)
- net BRAKE_PWM_DRV: now also D502.3 (CC); no longer D502.1 (K)
- net GND: now also J502.1 (GND), J502.MP (MOUNT), R512.2, C506.2, U503.1 (~{OE}), U503.3 (GND); no longer J502.2 (Pin_2)
- net VM: now also J501.2; no longer J501.1
- net at Q501.5 (D), Q501.6 (D), Q501.7 (D)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: now also J501.1; no longer J501.2
- net at R502.2: now also D502.1 (A1); no longer D502.2 (A)
- net BRAKE_NTC_RAW: no longer names the net of R511.2, R512.1
- net BRAKE_NTC_RAW: now also U503.2 (A); no longer J502.1 (Pin_1)
- net NTC_BRAKE renamed EXT_VCC
- net EXT_VCC: now also J502.2 (+5V), C506.1, U503.5 (VCC); no longer R512.2
- new net FAN_PWM: R511.1
- new net FAN_PWM_5V: J502.4 (PWM), U503.4 (Y)
- no-connect marks 0 -> 1
Other:
- note added: "5V PWM FAN / SHARED PROTECTED SUPPLY"
- note added: "Brake NTC removed. Brake PWM and hardware bus-overvoltage clamp remain active."
- note added: "Place U501 decoupling / R503 / D501 at Q501. Connect U501 pin 2 (GND) and pin 4 (IN-) to GND; Kelvin return to Q501 source."
- note added: "U604 on External feedback supplies J601 + J502; 520mA nominal shared limit. PC1 / LPTIM1_OUT: 25kHz, non-inverting. R512 holds the buffer input LOW at reset. Firmware: keep PWM LOW on USB-only power; allow running only when motor VM is present. 0% stops the specified Noctua fan. Two-wire fans on pins 1/2 run whenever 5V_SYS is powered."
- note added: "Validate Q501 drain overshoot."
- note removed: "10k NTC at 25C; configure the actual probe curve in firmware. J502: 1 = NTC, 2 = GND. Probe insulated from resistor power terminals."
- note removed: "D504 catches lead inductance."
- note removed: "OPTIONAL EXTERNAL BRAKE-RESISTOR TEMPERATURE"
- note removed: "Open = high; short = low. Filter/clamps at MCU; twist probe pair. Thermal warning/derating only: do not disable hardware bus clamp on overtemperature."
- note removed: "Place U501 decoupling / R503 / D501 at Q501. Return the driver ground to Q501 source with a short Kelvin connection."
- moved on the sheet: C505, R511, R512
