File: ShiroFOC/Manual_Layout_P3/10_CAN.kicad_sch (KiCad schematic)
At the start: 15 parts, among them J801 CAN 1, J802 CAN 2, U801 TCAN3413DR

Commit message: CAN layout
Parts:
- removed JP801: TERM ENABLE, Jumper:SolderJumper-2_P1.3mm_Open_Pad1.0x1.5mm, symbol Manual:COMP_JP801
- removed R803: 0R CANH link, Resistor_SMD:R_0402_1005Metric, symbol Manual:COMP_R803
- removed R804: 0R CANL link, Resistor_SMD:R_0402_1005Metric, symbol Manual:COMP_R804
- added Q801: CSD17483F4, ShiroFOCLib:CSD17483F4_YJC0003A, symbol ShiroFOCLib:CSD17483F4
- added Q802: CSD87502Q2, ShiroFOCLib:CSD87502Q2_DLV0006A, symbol ShiroFOCLib:CSD87502Q2
- added R803: 4.7k, Resistor_SMD:R_0402_1005Metric, symbol ShiroFOCLib:COMP_R802
- added R804: 100k, Resistor_SMD:R_0402_1005Metric, symbol ShiroFOCLib:COMP_R802
- added R806: 10k, Resistor_SMD:R_0402_1005Metric, symbol ShiroFOCLib:COMP_R802
- C801: symbol Manual:COMP_C801 -> ShiroFOCLib:COMP_C801
- C802: symbol Manual:COMP_C802 -> ShiroFOCLib:COMP_C802
- D801: symbol Manual:COMP_D801 -> ShiroFOCLib:COMP_D801
- J801: symbol Manual:COMP_J801 -> ShiroFOCLib:COMP_J801
- J802: symbol Manual:COMP_J802 -> ShiroFOCLib:COMP_J802
- R801: symbol Manual:COMP_R801 -> ShiroFOCLib:COMP_R801
- R802: symbol Manual:COMP_R802 -> ShiroFOCLib:COMP_R802
- R805: symbol Manual:COMP_R805 -> ShiroFOCLib:COMP_R805
- TP1013: symbol Manual:COMP_TP1013 -> ShiroFOCLib:COMP_TP1013
- TP1014: symbol Manual:COMP_TP1014 -> ShiroFOCLib:COMP_TP1014
- TP1022: symbol Manual:COMP_TP1022 -> ShiroFOCLib:COMP_TP1022
- U801: value TCAN3413DR -> TCAN3413DRBR; footprint Package_SO:SOIC-8_3.9x4.9mm_P1.27mm -> ShiroFOCLib:TCAN3413_DRB8; symbol Manual:COMP_U801 -> ShiroFOCLib:COMP_U801; MPN TCAN3413DR -> TCAN3413DRBR; Manufacturer (none) -> Texas Instruments
Connections:
- net CANH_INT is gone; now on net CANH_BUS: U801.7 (CANH)
- net CANL_INT is gone; now on net CANL_BUS: U801.6 (CANL)
- net CANH_BUS: now also D801.2 (CANH_IN), J801.2, J802.2; no longer D801.1 (CANH_IN), J801.3, J802.3
- net CANL_BUS: now also D801.1 (CANL_IN), J801.3, J802.3, Q802.3 (D2); no longer D801.2 (CANL_IN), J801.2, J802.2
- net GND: now also U801.9 (EP), Q801.2 (S), R804.2
- net CAN_TERM_MID: no longer names the net of R802.2
- net CAN_TERM_MID: now also Q802.6 (D1)
- new net: Q802.1 (S1), Q802.4 (S2)
- new net: Q801.1 (G), R803.2, R804.1
- new net CAN_TERM_DISABLE: R803.1
- new net CAN_TERM_GATE: Q801.3 (D), Q802.2 (G1), Q802.5 (G2), R806.2
- new net VCC: R806.1
Other:
- note added: "10 V gate pull-up provides full enhancement at normal CAN levels. Intended bus range: 0 to 5 V vs local GND. 30 V MOSFETs: this branch does not retain the transceiver's full bus-fault / common-mode tolerance. Q802 exposed drain lands: D1 = pin 6, D2 = pin 3. Project footprints assigned; drain pads numbered 6 and 3."
- note added: "CONTROL (PC15, former status LED GPIO) HIGH: termination OFF; RGB indicator BLUE. LOW / reset Hi-Z: termination ON; indicator PURPLE. ON requires the 10 V VCC rail. Set PC15 before releasing CAN_STB. Allow 1 ms for gate settling; change only while CAN is idle. Enable only at the two physical bus ends. Do not blink this GPIO as a general status LED."
- note added: "SOFTWARE-CONTROLLED 120 OHM TERMINATION"
- note added: "Software-controlled termination below. Enable only at the two bus ends."
- note added: "Sources joined; floating node"
- note removed: "R802 fitted on every board. Close JP801 only at a bus end. Default: solder jumper OPEN."
- moved on the sheet: R802

Commit message: progress + p4
Connections:
- net GND: now also J801.MP (MOUNT), J802.MP (MOUNT)
Changed lines of the file:
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@@
+	(wire
+		(pts
+			(xy 266.7 111.76) (xy 266.7 115.57)
+		)
+		(stroke
+			(width 0)
+			(type default)
+		)
+	)
 	(wire
 		(pts
@@
 		(pts
 			(xy 127 35.56) (xy 142.24 35.56)
+		)
+		(stroke
+			(width 0)
+			(type default)
+		)
+	)
+	(wire
+		(pts
+			(xy 266.7 167.64) (xy 266.7 171.45)
 		)
 		(stroke
@@
 		(on_board no)
 		(dnp no)
-		(property "Reference" "#PWRTERM10V"
+		(property "Reference" "#PWRTERM10V0101"
 			(at 134.62 210.82 0)
 			(effects
@@
 			(project "ShiroFOC_Manual"
 				(path "/2c8b7510-9664-4afd-8f00-ac42aa791be9/cdd56f0e-8dc5-44d0-8480-47c65cc22907"
-					(reference "#PWRTERM10V")
+					(reference "#PWRTERM10V0101")
 					(unit 1)
 				)
@@
 		(pin "1"
 		)
+		(pin "MP"
+		)
 		(instances
 			(project "ShiroFOC_Manual"
@@
 		(on_board no)
 		(dnp no)
-		(property "Reference" "#PWRTERMGND"
+		(property "Reference" "#PWRTERMGND0101"
 			(at 134.62 264.16 0)
 			(effects
@@
 			(project "ShiroFOC_Manual"
 				(path "/2c8b7510-9664-4afd-8f00-ac42aa791be9/cdd56f0e-8dc5-44d0-8480-47c65cc22907"
-					(reference "#PWRTERMGND")
+					(reference "#PWRTERMGND0101")
 					(unit 1)
 				)
@@
 	)
 	(symbol
+		(lib_id "ShiroFOCLib:PWR_GND")
+		(at 266.7 171.45 0)
+		(unit 1)
+		(exclude_from_sim no)
+		(in_bom no)
+		(on_board no)
+		(dnp no)
+		(property "Reference" "#PWR_MOUNT_J802"
+			(at 266.7 171.45 0)
+			(effects
+				(font
+					(size 1.27 1.27)
+				)
+				(hide yes)
+			)
+		)
+		(property "Value" "GND"
+			(at 266.7 175.26 0)
+			(effects
+				(font
+					(size 1.016 1.016)
+				)
+			)
+		)
+		(property "Footprint" ""
+			(at 266.7 171.45 0)
+			(effects
+				(font
+					(size 1.27 1.27)
+				)
+			)
+		)
+		(property "Datasheet" ""
+			(at 266.7 171.45 0)
+			(effects
+				(font
+					(size 1.27 1.27)
+				)
+			)
+		)
+		(property "Description" ""
+			(at 266.7 171.45 0)
+			(effects
+				(font
+					(size 1.27 1.27)
+				)
+			)
+		)
+		(pin "1"
+		)
+		(instances
+			(project "ShiroFOC_Manual"
+				(path "/2c8b7510-9664-4afd-8f00-ac42aa791be9/cdd56f0e-8dc5-44d0-8480-47c65cc22907"
+					(reference "#PWR_MOUNT_J802")
+					(unit 1)
+				)
+			)
+		)
+	)
+	(symbol
 		(lib_id "ShiroFOCLib:COMP_C802")
 		(at 142.24 45.72 0)
@@
 		(pin "4"
 		)
+		(pin "MP"
+		)
 		(instances
 			(project "ShiroFOC_Manual"
@@
 					(unit 1)
 				)
+			)
+		)
+	)
+	(symbol
+		(lib_id "ShiroFOCLib:PWR_GND")
+		(at 266.7 115.57 0)
+		(unit 1)
+		(exclude_from_sim no)
+		(in_bom no)
+		(on_board no)
+		(dnp no)
+		(property "Reference" "#PWR_MOUNT_J801"
+			(at 266.7 115.57 0)
+			(effects
+				(font
+					(size 1.27 1.27)
+				)
+				(hide yes)
+			)
+		)
+		(property "Value" "GND"
+			(at 266.7 119.38 0)
+			(effects
+				(font
+					(size 1.016 1.016)
+				)
+			)
+		)
+		(property "Footprint" ""
+			(at 266.7 115.57 0)
+			(effects
+				(font
+					(size 1.27 1.27)
+				)
+			)
+		)
+		(property "Datasheet" ""
+			(at 266.7 115.57 0)
+			(effects
+				(font
+					(size 1.27 1.27)
+				)
+			)
+		)
+		(property "Description" ""
+			(at 266.7 115.57 0)
+			(effects
+				(font
+					(size 1.27 1.27)
+				)
+			)
+		)
+		(pin "1"
+		)
+		(instances
+			(project "ShiroFOC_Manual"
+				(path "/2c8b7510-9664-4afd-8f00-ac42aa791be9/cdd56f0e-8dc5-44d0-8480-47c65cc22907"
+					(reference "#PWR_MOUNT_J801")
+					(unit 1)
+				)

Commit message: can connector rewiring
Connections:
- net CANH_BUS: now also D801.1 (CANH_IN); no longer D801.2 (CANH_IN)
- net CANL_BUS: now also D801.2 (CANL_IN); no longer D801.1 (CANL_IN)

Commit message: backup before i revise op amp resistor placement
Connections:
- net CAN_SHIELD is gone; now on net GND: J801.4, J802.4
Changed lines of the file:
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@@
+	)
+	(junction
+		(at 266.7 114.3)
+		(diameter 0)
+		(color 0 0 0 0)
 	)
 	(junction
@@
 	)
 	(junction
+		(at 248.92 114.3)
+		(diameter 0)
+		(color 0 0 0 0)
+	)
+	(junction
 		(at 109.22 35.56)
 		(diameter 0)
@@
 	(wire
 		(pts
-			(xy 248.92 102.87) (xy 248.92 158.75)
+			(xy 248.92 102.87) (xy 248.92 114.3)
 		)
 		(stroke
@@
 	(wire
 		(pts
+			(xy 248.92 114.3) (xy 266.7 114.3)
+		)
+		(stroke
+			(width 0)
+			(type default)
+		)
+	)
+	(wire
+		(pts
 			(xy 184.15 110.49) (xy 184.15 129.54)
 		)
@@
 	(wire
 		(pts
-			(xy 266.7 111.76) (xy 266.7 115.57)
+			(xy 266.7 111.76) (xy 266.7 114.3)
 		)
 		(stroke
@@
 	(wire
 		(pts
+			(xy 248.92 114.3) (xy 248.92 158.75)
+		)
+		(stroke
+			(width 0)
+			(type default)
+		)
+	)
+	(wire
+		(pts
 			(xy 142.24 35.56) (xy 142.24 40.64)
 		)
@@
 		)
 		(stroke
+			(width 0)
+			(type default)
+		)
+	)
+	(wire
+		(pts
+			(xy 266.7 114.3) (xy 266.7 115.57)
+		)
+		(stroke

Commit message: weekend progress
Parts:
- J801, J802: footprint Connector_JST:JST_GH_BM04B-GHS-TBT_1x04-1MP_P1.25mm_Vertical -> Connector_JST:JST_GH_SM03B-GHS-TB_1x03-1MP_P1.25mm_Horizontal; MPN BM04B-GHS-TBT -> SM03B-GHS-TB
Connections:
- net GND: no longer J801.4, J802.4
Other:
- note added: "Both headers: 1 GND | 2 CANH | 3 CANL. JST-GH 3-pin; mounting tabs grounded."
- note removed: "Both headers: 1 GND | 2 CANL | 3 CANH | 4 shield/drain. Pin 4 carries no supply."
Changed lines of the file:
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@@
 		(comment 1 "MOSFET termination on PC15; purple ON, blue OFF")
 	)
-	(text "Both headers: 1 GND | 2 CANL | 3 CANH | 4 shield/drain. Pin 4 carries no supply."
+	(text "Both headers: 1 GND | 2 CANH | 3 CANL. JST-GH 3-pin; mounting tabs grounded."
 		(exclude_from_sim no)
 		(at 15.24 171.45 0)
@@
 	)
 	(junction
-		(at 266.7 114.3)
-		(diameter 0)
-		(color 0 0 0 0)
-	)
-	(junction
 		(at 165.1 233.68)
 		(diameter 0)
@@
 	)
 	(junction
-		(at 248.92 114.3)
-		(diameter 0)
-		(color 0 0 0 0)
-	)
-	(junction
 		(at 109.22 35.56)
 		(diameter 0)
@@
 	(wire
 		(pts
-			(xy 248.92 102.87) (xy 248.92 114.3)
-		)
-		(stroke
-			(width 0)
-			(type default)
-		)
-	)
-	(wire
-		(pts
 			(xy 194.31 80.01) (xy 194.31 129.54)
 		)
@@
 	(wire
 		(pts
-			(xy 248.92 114.3) (xy 266.7 114.3)
-		)
-		(stroke
-			(width 0)
-			(type default)
-		)
-	)
-	(wire
-		(pts
 			(xy 184.15 110.49) (xy 184.15 129.54)
 		)
@@
 	(wire
 		(pts
-			(xy 266.7 111.76) (xy 266.7 114.3)
-		)
-		(stroke
-			(width 0)
-			(type default)
-		)
-	)
-	(wire
-		(pts
-			(xy 248.92 102.87) (xy 252.73 102.87)
-		)
-		(stroke
-			(width 0)
-			(type default)
-		)
-	)
-	(wire
-		(pts
 			(xy 165.1 233.68) (xy 165.1 248.92)
 		)
@@
 	(wire
 		(pts
-			(xy 248.92 114.3) (xy 248.92 158.75)
-		)
-		(stroke
-			(width 0)
-			(type default)
-		)
-	)
-	(wire
-		(pts
 			(xy 142.24 35.56) (xy 142.24 40.64)
 		)
@@
 	(wire
 		(pts
-			(xy 248.92 158.75) (xy 252.73 158.75)
-		)
-		(stroke
-			(width 0)
-			(type default)
-		)
-	)
-	(wire
-		(pts
 			(xy 177.8 205.74) (xy 177.8 213.36)
 		)
@@
 	(wire
 		(pts
-			(xy 266.7 114.3) (xy 266.7 115.57)
+			(xy 266.7 111.76) (xy 266.7 115.57)
 		)
 		(stroke
@@
 		)
 	)
-	(label "CAN_SHIELD"
-		(at 248.92 120.65 0)
-		(effects
-			(font
-				(size 1.016 1.016)
-			)
-			(justify left bottom)
-		)
-	)
 	(global_label "CAN_TERM_DISABLE"
 		(shape input)
@@
 			)
 		)
-		(property "Footprint" "Connector_JST:JST_GH_BM04B-GHS-TBT_1x04-1MP_P1.25mm_Vertical"
+		(property "Footprint" "Connector_JST:JST_GH_SM03B-GHS-TB_1x03-1MP_P1.25mm_Horizontal"
 			(at 266.7 109.22 0)
 			(effects
@@
 			)
 		)
-		(property "MPN" "BM04B-GHS-TBT"
+		(property "MPN" "SM03B-GHS-TB"
 			(at 266.7 109.22 0)
 			(effects
@@
 			)
 		)
-		(pin "4"
-		)
 		(pin "3"
 		)
@@
 			)
 		)
-		(property "Footprint" "Connector_JST:JST_GH_BM04B-GHS-TBT_1x04-1MP_P1.25mm_Vertical"
+		(property "Footprint" "Connector_JST:JST_GH_SM03B-GHS-TB_1x03-1MP_P1.25mm_Horizontal"
 			(at 266.7 165.1 0)
 			(effects
@@
 			)
 		)
-		(property "MPN" "BM04B-GHS-TBT"
+		(property "MPN" "SM03B-GHS-TB"
 			(at 266.7 165.1 0)
 			(effects
@@
 		(pin "1"
 		)
-		(pin "4"
-		)
 		(pin "MP"
