File: ShiroFOC/Manual_Layout_P3/MCUclockSWD.kicad_sch (KiCad schematic)
At the start: 25 parts, among them J1001 TC2030-NL SWD, SW301 RESET, U4 STSPIN32G4, Y301 24MHz 7pF

Commit message: pcb layout blocks
Connections:
- net NTC_BRAKE: now also U4.10 (PC1); no longer U4.11 (PC2)
- net NTC_PHASE_B: now also U4.11 (PC2); no longer U4.9 (PC0)
- net NTC_PHASE_C: now also U4.13 (PA0); no longer U4.10 (PC1)
- net VBUS_SENSE: now also U4.9 (PC0); no longer U4.13 (PA0)

Commit message: CAN layout
Parts:
- added Q301: BSS138AKM-Q, Package_TO_SOT_SMD:SOT-883, symbol ShiroFOCLib:BSS138AKM_Q
- added R315: 10k, Resistor_SMD:R_0402_1005Metric, symbol ShiroFOCLib:COMP_R802
- C301: symbol Manual:COMP_C301 -> ShiroFOCLib:COMP_C301
- C302: symbol Manual:COMP_C302 -> ShiroFOCLib:COMP_C302
- C303: symbol Manual:COMP_C303 -> ShiroFOCLib:COMP_C303
- C304: symbol Manual:COMP_C304 -> ShiroFOCLib:COMP_C304
- C305: symbol Manual:COMP_C305 -> ShiroFOCLib:COMP_C305
- C306: symbol Manual:COMP_C306 -> ShiroFOCLib:COMP_C306
- C307: symbol Manual:COMP_C307 -> ShiroFOCLib:COMP_C307
- C308: symbol Manual:COMP_C308 -> ShiroFOCLib:COMP_C308
- C309: symbol Manual:COMP_C309 -> ShiroFOCLib:COMP_C309
- C310: symbol Manual:COMP_C310 -> ShiroFOCLib:COMP_C310
- D301: value RED -> LTST-C19HE1WT; footprint LED_SMD:LED_0603_1608Metric -> LED_SMD:LED_LiteOn_LTST-C19HE1WT; symbol Manual:COMP_D301 -> ShiroFOCLib:LTST_C19HE1WT; BOM Comments (none) -> 1.6 x 1.6 mm RGB; blue power indication, red termination en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; DigiKey (none) -> 160-2162-1-ND; MPN (none) -> LTST-C19HE1WT; Manufacturer (none) -> Lite-On; Package (none) -> 0606 / 1616, 1.6 x 1.6 x 0.35 mm; Procurement Select to specification: RED; LED_0603_1608Metric -> (none); Rating See Value; generic low-voltage passives: R >=0.1 W / 50 V, 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 -> (none)
- R301: symbol Manual:COMP_R301 -> ShiroFOCLib:COMP_R301
- R302: symbol Manual:COMP_R302 -> ShiroFOCLib:COMP_R302
- R303: symbol Manual:COMP_R303 -> ShiroFOCLib:COMP_R303
- R304: value 2.2k -> 15k; symbol Manual:COMP_R304 -> ShiroFOCLib:COMP_R304; BOM Comments (none) -> Red channel: approximately 0.2 mA at 5 V for a subdued indi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; Rating See Value; generic low-voltage passives: R >=0.1 W / 50 V, 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 -> 1%, >=0.063 W, >=25 V
- TP1008: symbol Manual:COMP_TP1008 -> ShiroFOCLib:COMP_TP1008
- TP1009: symbol Manual:COMP_TP1009 -> ShiroFOCLib:COMP_TP1009
- TP1021: value STATUS_LED_N -> CAN_TERM_DISABLE; symbol Manual:COMP_TP1021 -> ShiroFOCLib:COMP_TP1021; Test_Net /MCU / clock / SWD/SPARE_GPIO_1 -> CAN_TERM_DISABLE
- TP1023: symbol Manual:COMP_TP1023 -> ShiroFOCLib:COMP_TP1023
- TP1024: symbol Manual:COMP_TP1024 -> ShiroFOCLib:COMP_TP1024
- TP303: symbol Manual:COMP_TP303 -> ShiroFOCLib:COMP_TP303
- U4: footprint Manual:QFN_IN32G4_STM -> ShiroFOCLib:QFN_IN32G4_STM; symbol Manual:STSPIN32G4_Functional -> ShiroFOCLib:STSPIN32G4_Functional
- Y301: symbol Manual:COMP_Y301 -> ShiroFOCLib:COMP_Y301
Connections:
- net 3V3: no longer R304.1
- net GND: now also Q301.2 (S), R315.2
- net at R304.2: now also D301.1 (RK); no longer D301.2 (A)
- net STATUS_LED_N renamed CAN_TERM_DISABLE
- net CAN_TERM_DISABLE: no longer D301.1 (K)
- new net: Q301.3 (D), R304.1
- new net: D301.3 (BK), R315.1
- new net 5V_SYS: D301.4 (A)
- new net CAN_TERM_GATE: Q301.1 (G)
- no-connect marks 1 -> 2
Other:
- note added: "BLUE = 5 V power present; PURPLE = power + termination enabled. Green unused. PC15 HIGH disables termination and red. Reset Hi-Z defaults to PURPLE once 10 V VCC is present. PC15: low-speed push-pull; keep LSE disabled. No status blinking. Q301 isolates LED current from the CAN termination gate drive. With USB-only power / no 10 V rail: blue only; termination unavailable."
- note added: "POWER / CAN TERMINATION INDICATOR"
- note removed: "STATUS LED: PC15, active low / open drain. R304 limits LED sink current; keep LSE disabled. PC2 is now ADC12_IN8 for the external brake NTC."
- moved on the sheet: R304

Commit message: progress
Parts:
- Q301: value BSS138AKM-Q -> CSD17483F4; footprint Package_TO_SOT_SMD:SOT-883 -> ShiroFOCLib:CSD17483F4_YJC0003A; symbol ShiroFOCLib:BSS138AKM_Q -> ShiroFOCLib:CSD17483F4; BOM Comments (none) -> V1 substitution for BSS138AKM-QYL. Direct nominal 10 V CAN_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; MPN BSS138AKM-QYL -> CSD17483F4; Manufacturer Nexperia -> Texas Instruments; Package SOT883 / DFN1006-3, 1.0 x 0.6 mm -> YJC0003A, 1.0 x 0.6 mm, 3-pin PicoStar
Changed lines of the file:
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@@
 	)
 	(symbol
-		(lib_id "ShiroFOCLib:BSS138AKM_Q")
+		(lib_id "ShiroFOCLib:CSD17483F4")
 		(at 345.44 124.46 0)
 		(unit 1)
@@
 			)
 		)
-		(property "Value" "BSS138AKM-Q"
+		(property "Value" "CSD17483F4"
 			(at 351.79 125.73 0)
 			(effects
@@
 			)
 		)
-		(property "Footprint" "Package_TO_SOT_SMD:SOT-883"
+		(property "Footprint" "ShiroFOCLib:CSD17483F4_YJC0003A"
 			(at 345.44 124.46 0)
 			(effects
@@
 			)
 		)
-		(property "Datasheet" "https://assets.nexperia.com/documents/data-sheet/BSS138AKM-Q.pdf"
+		(property "Datasheet" "https://www.ti.com/lit/ds/symlink/csd17483f4.pdf"
 			(at 345.44 124.46 0)
 			(effects
@@
 			)
 		)
-		(property "Description" "60 V N-MOSFET, +/-20 V gate rating. Pin 1 G, 2 S, 3 D. Red LED driver follows CAN_TERM_GATE without LED current loading the termination gates."
+		(property "Description" "30 V N-MOSFET, +12 V maximum gate-to-source voltage. Pin 1 G, 2 S, 3 D. Red LED driver follows CAN_TERM_GATE."
 			(at 0 0 0)
 			(effects
@@
 			)
 		)
-		(property "Manufacturer" "Nexperia"
+		(property "Manufacturer" "Texas Instruments"
 			(at 0 0 0)
 			(effects
@@
 			)
 		)
-		(property "MPN" "BSS138AKM-QYL"
+		(property "MPN" "CSD17483F4"
 			(at 0 0 0)
 			(effects
@@
 			)
 		)
-		(property "Package" "SOT883 / DFN1006-3, 1.0 x 0.6 mm"
+		(property "Package" "YJC0003A, 1.0 x 0.6 mm, 3-pin PicoStar"
 			(at 0 0 0)
 			(effects
@@
 			(at 0 0 0)
 			(effects
+				(font
+					(size 1.27 1.27)
+				)
+				(justify left)
+				(hide yes)
+			)
+		)
+		(property "BOM Comments" "V1 substitution for BSS138AKM-QYL. Direct nominal 10 V CAN_TERM_GATE drive; +12 V absolute maximum VGS, so verify gate transients on the prototype. Gate failure may affect CAN termination. Reverting to BSS138AKM-QYL requires its SOT-883 footprint; it is not a drop-in substitution."
+			(at 0 0 0)
+			(effects

Commit message: progress + p4
Parts:
- TP1023: value EXT_SENSOR_FAULT_N -> EXT_POWER_FAULT_N; Test_Net EXT_SENSOR_FAULT_N -> EXT_POWER_FAULT_N
Connections:
- net EXT_SENSOR_FAULT_N renamed EXT_POWER_FAULT_N
- net NTC_BRAKE renamed FAN_PWM
Other:
- note added: "PC1 / pin 10: FAN_PWM = LPTIM1_OUT, 25kHz -> U503 AHCT buffer. R512 holds buffer input LOW at reset. Firmware keeps LOW until motor VM is present. PC13: EXT_POWER_FAULT_N = shared sensor/fan limiter U604 (active low)."
Changed lines of the file:
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@@
 		)
 	)
-	(global_label "EXT_SENSOR_FAULT_N"
+	(global_label "EXT_POWER_FAULT_N"
 		(shape bidirectional)
 		(at 88.9 121.92 180)
@@
 		)
 	)
-	(global_label "NTC_BRAKE"
-		(shape bidirectional)
+	(global_label "FAN_PWM"
+		(shape output)
 		(at 179.07 67.31 0)
 		(effects
@@
 			)
 		)
-		(property "Value" "EXT_SENSOR_FAULT_N"
+		(property "Value" "EXT_POWER_FAULT_N"
 			(at 88.9 119.38 0)
 			(effects
@@
 			)
 		)
-		(property "Test_Net" "EXT_SENSOR_FAULT_N"
+		(property "Test_Net" "EXT_POWER_FAULT_N"
 			(at 88.9 121.92 0)
 			(effects
@@
 		(on_board no)
 		(dnp no)
-		(property "Reference" "#PWRRGB5V"
+		(property "Reference" "#PWRRGB5V0101"
 			(at 314.96 91.44 0)
 			(effects
@@
 			(project "ShiroFOC_Manual"
 				(path "/2c8b7510-9664-4afd-8f00-ac42aa791be9/72c68966-ddbf-45d8-a1a7-ab83562ae772"
-					(reference "#PWRRGB5V")
+					(reference "#PWRRGB5V0101")
 					(unit 1)
 				)
@@
 		(on_board no)
 		(dnp no)
-		(property "Reference" "#PWRRGBBLUE"
+		(property "Reference" "#PWRRGBBLUE0101"
 			(at 378.46 134.62 0)
 			(effects
@@
 			(project "ShiroFOC_Manual"
 				(path "/2c8b7510-9664-4afd-8f00-ac42aa791be9/72c68966-ddbf-45d8-a1a7-ab83562ae772"
-					(reference "#PWRRGBBLUE")
+					(reference "#PWRRGBBLUE0101")
 					(unit 1)
 				)
@@
 		(on_board no)
 		(dnp no)
-		(property "Reference" "#PWRRGBRED"
+		(property "Reference" "#PWRRGBRED0101"
 			(at 347.98 134.62 0)
 			(effects
@@
 			(project "ShiroFOC_Manual"
 				(path "/2c8b7510-9664-4afd-8f00-ac42aa791be9/72c68966-ddbf-45d8-a1a7-ab83562ae772"
-					(reference "#PWRRGBRED")
+					(reference "#PWRRGBRED0101")
 					(unit 1)
 				)
@@
 		)
 	)
+	(text "PC1 / pin 10: FAN_PWM = LPTIM1_OUT, 25kHz -> U503 AHCT buffer.\nR512 holds buffer input LOW at reset. Firmware keeps LOW until motor VM is present.\nPC13: EXT_POWER_FAULT_N = shared sensor/fan limiter U604 (active low)."
+		(at 195.58 22.86 0)
+		(effects
+			(font
+				(size 1.016 1.016)
+			)
+			(justify left top)
+		)
+	)

Commit message: weekend progress
Connections:
- net NTC_PHASE_A: now also U4.11 (PC2); no longer U4.12 (PC3)
- net NTC_PHASE_B: now also U4.12 (PC3); no longer U4.11 (PC2)
Changed lines of the file:
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@@
 		)
 	)
-	(global_label "NTC_PHASE_A"
+	(global_label "NTC_PHASE_B"
 		(shape bidirectional)
 		(at 179.07 72.39 0)
@@
 		)
 	)
-	(global_label "NTC_PHASE_B"
+	(global_label "NTC_PHASE_A"
 		(shape bidirectional)
 		(at 179.07 69.85 0)
