File: ShiroFOC/Manual_Layout_P3/01_DC_Link.kicad_sch (KiCad schematic)
At the start: 71 parts, among them J101 AMASS XT60PW-M

Commit message: CAN layout
Parts:
- C104: symbol Manual:COMP_C104 -> ShiroFOCLib:COMP_C104
- C105: symbol Manual:COMP_C105 -> ShiroFOCLib:COMP_C105
- C106: symbol Manual:COMP_C106 -> ShiroFOCLib:COMP_C106
- C107: symbol Manual:COMP_C107 -> ShiroFOCLib:COMP_C107
- C108: symbol Manual:COMP_C108 -> ShiroFOCLib:COMP_C108
- D101: symbol Manual:COMP_D101 -> ShiroFOCLib:COMP_D101
- J101: symbol Manual:COMP_J101 -> ShiroFOCLib:COMP_J101
- R101: symbol Manual:COMP_R101 -> ShiroFOCLib:COMP_R101
- R102: symbol Manual:COMP_R102 -> ShiroFOCLib:COMP_R102
- R103: symbol Manual:COMP_R103 -> ShiroFOCLib:COMP_R103
- R105: symbol Manual:COMP_R105 -> ShiroFOCLib:COMP_R105
- R106: symbol Manual:COMP_R106 -> ShiroFOCLib:COMP_R106
- TP101, TP104, TP105: symbol Manual:COMP_TP101 -> ShiroFOCLib:COMP_TP101
- TP102: symbol Manual:COMP_TP102 -> ShiroFOCLib:COMP_TP102
- TP103: symbol Manual:COMP_TP103 -> ShiroFOCLib:COMP_TP103
Changed lines of the file:
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@@
 	)
 	(symbol
-		(lib_id "Manual:COMP_C105")
+		(lib_id "ShiroFOCLib:COMP_C105")
 		(at 191.77 72.39 0)
 		(unit 1)
@@
 	)
 	(symbol
-		(lib_id "Manual:PWR_GND")
+		(lib_id "ShiroFOCLib:PWR_GND")
 		(at 255.27 158.75 0)
 		(unit 1)
@@
 	)
 	(symbol
-		(lib_id "Manual:COMP_TP101")
+		(lib_id "ShiroFOCLib:COMP_TP101")
 		(at 322.58 95.25 0)
 		(unit 1)
@@
 	)
 	(symbol
-		(lib_id "Manual:PWR_GND")
+		(lib_id "ShiroFOCLib:PWR_GND")
 		(at 31.75 157.48 0)
 		(unit 1)
@@
 	)
 	(symbol
-		(lib_id "Manual:COMP_C108")
+		(lib_id "ShiroFOCLib:COMP_C108")
 		(at 255.27 148.59 0)
 		(unit 1)
@@
 	)
 	(symbol
-		(lib_id "Manual:COMP_R101")
+		(lib_id "ShiroFOCLib:COMP_R101")
 		(at 260.35 72.39 0)
 		(unit 1)
@@
 	)
 	(symbol
-		(lib_id "Manual:COMP_TP101")
+		(lib_id "ShiroFOCLib:COMP_TP101")
 		(at 63.5 49.53 0)
 		(unit 1)
@@
 	)
 	(symbol
-		(lib_id "Manual:COMP_R103")
+		(lib_id "ShiroFOCLib:COMP_R103")
 		(at 190.5 119.38 0)
 		(unit 1)
@@
 	)
 	(symbol
-		(lib_id "Manual:COMP_R102")
+		(lib_id "ShiroFOCLib:COMP_R102")
 		(at 31.75 124.46 0)
 		(unit 1)
@@
 	)
 	(symbol
-		(lib_id "Manual:COMP_R106")
+		(lib_id "ShiroFOCLib:COMP_R106")
 		(at 250.19 119.38 0)
 		(unit 1)
@@
 	)
 	(symbol
-		(lib_id "Manual:FLAG")
+		(lib_id "ShiroFOCLib:FLAG")
 		(at 323.85 62.23 0)
 		(unit 1)
@@
 	)
 	(symbol
-		(lib_id "Manual:COMP_D101")
+		(lib_id "ShiroFOCLib:COMP_D101")
 		(at 99.06 135.89 0)
 		(unit 1)
@@
 	)
 	(symbol
-		(lib_id "Manual:PWR_GND")
+		(lib_id "ShiroFOCLib:PWR_GND")
 		(at 227.33 152.4 0)
 		(unit 1)
@@
 	)
 	(symbol
-		(lib_id "Manual:COMP_TP102")
+		(lib_id "ShiroFOCLib:COMP_TP102")
 		(at 63.5 91.44 180)
 		(unit 1)
@@
 	)
 	(symbol
-		(lib_id "Manual:PWR_GND")
+		(lib_id "ShiroFOCLib:PWR_GND")
 		(at 45.72 92.71 0)
 		(unit 1)
@@
 	)
 	(symbol
-		(lib_id "Manual:COMP_J101")
+		(lib_id "ShiroFOCLib:COMP_J101")
 		(at 27.94 72.39 0)
 		(unit 1)
@@
 	)
 	(symbol
-		(lib_id "Manual:COMP_TP103")
+		(lib_id "ShiroFOCLib:COMP_TP103")
 		(at 255.27 132.08 0)
 		(unit 1)
@@
 	)
 	(symbol
-		(lib_id "Manual:COMP_C107")
+		(lib_id "ShiroFOCLib:COMP_C107")
 		(at 31.75 146.05 0)
 		(unit 1)
@@
 	)
 	(symbol
-		(lib_id "Manual:FLAG")
+		(lib_id "ShiroFOCLib:FLAG")
 		(at 351.79 62.23 0)
 		(unit 1)
@@
 	)
 	(symbol
-		(lib_id "Manual:PWR_VM")
+		(lib_id "ShiroFOCLib:PWR_VM")
 		(at 162.56 119.38 0)
 		(unit 1)
@@
 	)
 	(symbol
-		(lib_id "Manual:PWR_VM")
+		(lib_id "ShiroFOCLib:PWR_VM")
 		(at 45.72 49.53 0)
 		(unit 1)
@@
 	)
 	(symbol
-		(lib_id "Manual:COMP_C106")
+		(lib_id "ShiroFOCLib:COMP_C106")
 		(at 226.06 72.39 0)
 		(unit 1)
@@
 	)
 	(symbol
-		(lib_id "Manual:PWR_GND")
+		(lib_id "ShiroFOCLib:PWR_GND")
 		(at 99.06 149.86 0)
 		(unit 1)
@@
 	)
 	(symbol
-		(lib_id "Manual:COMP_C104")
+		(lib_id "ShiroFOCLib:COMP_C104")
 		(at 157.48 72.39 0)
 		(unit 1)
@@
 	)
 	(symbol
-		(lib_id "Manual:PWR_VM")
+		(lib_id "ShiroFOCLib:PWR_VM")
 		(at 31.75 113.03 0)
 		(unit 1)
@@
 	)
 	(symbol
-		(lib_id "Manual:COMP_TP101")
+		(lib_id "ShiroFOCLib:COMP_TP101")
 		(at 358.14 95.25 0)
 		(unit 1)
@@
 	)
 	(symbol
-		(lib_id "Manual:COMP_R105")
+		(lib_id "ShiroFOCLib:COMP_R105")
 		(at 227.33 140.97 0)
 		(unit 1)
@@
 	)
 	(symbol
-		(lib_id "Manual:PWR_VM")
+		(lib_id "ShiroFOCLib:PWR_VM")
 		(at 99.06 121.92 0)
 		(unit 1)

Commit message: progress + p4
Parts:
- J101: value AMASS XT60PW-M -> DC input - solder wires; footprint Connector_AMASS:AMASS_XT60PW-M_1x02_P7.20mm_Horizontal -> ShiroFOCLib:WireSolder_DC_1x02_P6.35mm_D2.70mm_Pad4.10mm; symbol ShiroFOCLib:COMP_J101 -> ShiroFOCLib:DirectWire_DC_2; Assembly FIT -> Direct-solder wires; no connector fitted; MPN XT60PW-M -> (none); Rating See Value; generic low-voltage passives: R >=0.1 W / 50 V, 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 -> Wire gauge and current limited by completed PCB copper and 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; now left out of the parts list
Other:
- note added: "18-42 V operating bus • direct-solder DC wires • external fuse / precharge required"
- note removed: "18-42 V operating bus • keyed XT60 • external fuse / precharge required"
Changed lines of the file:
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@@
 		)
 	)
-	(text "18-42 V operating bus • keyed XT60 • external fuse / precharge required"
+	(text "18-42 V operating bus • direct-solder DC wires • external fuse / precharge required"
 		(exclude_from_sim no)
 		(at 17.78 29.21 0)
@@
 	)
 	(symbol
-		(lib_id "ShiroFOCLib:COMP_J101")
+		(lib_id "ShiroFOCLib:DirectWire_DC_2")
 		(at 27.94 72.39 0)
 		(unit 1)
 		(exclude_from_sim no)
-		(in_bom yes)
+		(in_bom no)
 		(on_board yes)
 		(dnp no)
@@
 			)
 		)
-		(property "Value" "AMASS XT60PW-M"
+		(property "Value" "DC input - solder wires"
 			(at 27.94 82.55 0)
 			(effects
@@
 			)
 		)
-		(property "Footprint" "Connector_AMASS:AMASS_XT60PW-M_1x02_P7.20mm_Horizontal"
+		(property "Footprint" "ShiroFOCLib:WireSolder_DC_1x02_P6.35mm_D2.70mm_Pad4.10mm"
 			(at 27.94 82.55 0)
 			(effects
@@
 			)
 		)
-		(property "Description" ""
+		(property "Description" "Direct-solder plated wire terminals; no fitted connector"
 			(at 27.94 72.39 0)
 			(effects
@@
 			)
 		)
-		(property "MPN" "XT60PW-M"
+		(property "MPN" ""
 			(at 27.94 82.55 0)
 			(effects
@@
 			)
 		)
-		(property "Assembly" "FIT"
+		(property "Assembly" "Direct-solder wires; no connector fitted"
 			(at 27.94 82.55 0)
 			(effects
@@
 			)
 		)
-		(property "Rating" "See Value; generic low-voltage passives: R >=0.1 W / 50 V, C >=16 V X7R unless specified"
+		(property "Rating" "Wire gauge and current limited by completed PCB copper and assembly"
 			(at 27.94 82.55 0)
 			(effects

Commit message: weekend progress
Parts:
- J101: footprint ShiroFOCLib:WireSolder_DC_1x02_P6.35mm_D2.70mm_Pad4.10mm -> ShiroFOCLib:WireSolder_DC_1x02_P6.35mm_D3.00mm_Pad5.00x4.10mm_4xD0.40mm
Changed lines of the file:
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@@
 			)
 		)
-		(property "Footprint" "ShiroFOCLib:WireSolder_DC_1x02_P6.35mm_D2.70mm_Pad4.10mm"
+		(property "Footprint" "ShiroFOCLib:WireSolder_DC_1x02_P6.35mm_D3.00mm_Pad5.00x4.10mm_4xD0.40mm"
 			(at 27.94 82.55 0)
 			(effects

Commit message: half bridge progress
Parts:
- J101: footprint ShiroFOCLib:WireSolder_DC_1x02_P6.35mm_D3.00mm_Pad5.00x4.10mm_4xD0.40mm -> ShiroFOCLib:WireSolder_DC_1x02_P6.85mm_D3.00mm_Pad5.00x4.10mm_4xD0.40mm
Changed lines of the file:
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@@
 			)
 		)
-		(property "Footprint" "ShiroFOCLib:WireSolder_DC_1x02_P6.35mm_D3.00mm_Pad5.00x4.10mm_4xD0.40mm"
+		(property "Footprint" "ShiroFOCLib:WireSolder_DC_1x02_P6.85mm_D3.00mm_Pad5.00x4.10mm_4xD0.40mm"
 			(at 27.94 82.55 0)
 			(effects
