File: ShiroFOC/Manual_Layout_P3/01_DC_Link.kicad_sch (KiCad schematic)
At the start: 71 parts, among them J101 DC input - solder wires

Commit message: mosfet stages and opamps revamped
Parts:
- removed C125, C126, C142, C143, C159, C160: 10uF DNP, Capacitor_SMD:C_1210_3225Metric, symbol Device:C
