File: ShiroFOC/Manual_Layout_P3/Three-phase bridge.kicad_sch (KiCad schematic)
At the start: 19 parts, among them J1 MOTOR U/V/W, U1 CSD88599Q5DC, U2 CSD88599Q5DC, U3 CSD88599Q5DC

Commit message: usb and pwr mux
Parts:
- added C413, C423, C433: TUNE DNP, Capacitor_SMD:C_1206_3216Metric, symbol Device:C
- added R415, R425, R435: TUNE DNP, Resistor_SMD:R_1206_3216Metric, symbol Device:R
- added TP411, TP421, TP431: GL, TestPoint:TestPoint_Pad_D1.0mm, symbol Manual:COMP_TP101
- added TP412, TP422, TP432: SOURCE, TestPoint:TestPoint_Pad_D1.0mm, symbol Manual:COMP_TP101
- added TP413, TP423, TP433: PHASE, TestPoint:TestPoint_Pad_D1.0mm, symbol Manual:COMP_TP101
- J1: footprint Connector_Wire:SolderWire-6sqmm_1x03_P14mm_D3.5mm_OD7mm -> Connector_AMASS:AMASS_MR30PW-M_1x03_P3.50mm_Horizontal
Connections:
- net GLS1: now also TP411.1
- net GLS2: now also TP421.1
- net GLS3: now also TP431.1
- net PHASE_U: now also R415.1, TP413.1
- net PHASE_V: now also R425.1, TP423.1
- net PHASE_W: now also R435.1, TP433.1
- net LS_SOURCE_U: now reaches R3.1 (POWER+), U1.12 (PGND), U1.13 (PGND), U1.14 (PGND), U1.15 (PGND), U1.16 (PGND), U1.17 (PGND), U1.18 (PGND), U1.19 (PGND), U1.20 (PGND)
- net LS_SOURCE_U: now also C413.2, TP412.1
- net LS_SOURCE_W: now reaches R5.1 (POWER+), U3.12 (PGND), U3.13 (PGND), U3.14 (PGND), U3.15 (PGND), U3.16 (PGND), U3.17 (PGND), U3.18 (PGND), U3.19 (PGND), U3.20 (PGND)
- net LS_SOURCE_W: now also C433.2, TP432.1
- net LS_SOURCE_V: now reaches R1.1 (POWER+), U2.12 (PGND), U2.13 (PGND), U2.14 (PGND), U2.15 (PGND), U2.16 (PGND), U2.17 (PGND), U2.18 (PGND), U2.19 (PGND), U2.20 (PGND)
- net LS_SOURCE_V: now also C423.2, TP422.1
- new net: C423.1, R425.2
- new net: C413.1, R415.2
- new net: C433.1, R435.2
Other:
- note added: "PHASE U / OPTIONAL RC"
- note added: "PHASE V / OPTIONAL RC"
- note added: "PHASE W / OPTIONAL RC"
- note added: "RC snubbers: all DNP. Tune from measured ringing; verify resistor pulse/average power. Return each RC to the local MOSFET PGND power pad BEFORE the shunt. GL/SOURCE pads measure low-side Vgs; PHASE is a switching node."

Commit message: CAN layout
Parts:
- J1: symbol Manual:Motor_Phase_Terminals_3 -> ShiroFOCLib:Motor_Phase_Terminals_3
- R1, R3, R5: footprint Manual:R_Shunt_LR2512D_0m5_3W_Kelvin -> ShiroFOCLib:R_Shunt_LR2512D_0m5_3W_Kelvin; symbol Manual:LR2512D_Kelvin -> ShiroFOCLib:LR2512D_Kelvin
- TP411, TP412, TP413, TP421, TP422, TP423, TP431, TP432, TP433: symbol Manual:COMP_TP101 -> ShiroFOCLib:COMP_TP101
- U1, U2, U3: footprint Manual:DMM0022A -> ShiroFOCLib:DMM0022A; symbol Manual:CSD88599Q5DC -> ShiroFOCLib:CSD88599Q5DC
Changed lines of the file:
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@@
 	)
 	(symbol
-		(lib_id "Manual:LR2512D_Kelvin")
+		(lib_id "ShiroFOCLib:LR2512D_Kelvin")
 		(at 34.29 67.31 0)
 		(unit 1)
@@
 			)
 		)
-		(property "Footprint" "Manual:R_Shunt_LR2512D_0m5_3W_Kelvin"
+		(property "Footprint" "ShiroFOCLib:R_Shunt_LR2512D_0m5_3W_Kelvin"
 			(at 32.512 67.31 90)
 			(effects
@@
 	)
 	(symbol
-		(lib_id "Manual:CSD88599Q5DC")
+		(lib_id "ShiroFOCLib:CSD88599Q5DC")
 		(at 227.33 50.8 0)
 		(unit 1)
@@
 			)
 		)
-		(property "Footprint" "Manual:DMM0022A"
+		(property "Footprint" "ShiroFOCLib:DMM0022A"
 			(at 223.52 74.93 0)
 			(effects
@@
 	)
 	(symbol
-		(lib_id "Manual:COMP_TP101")
+		(lib_id "ShiroFOCLib:COMP_TP101")
 		(at 200.66 147.32 0)
 		(unit 1)
@@
 	)
 	(symbol
-		(lib_id "Manual:COMP_TP101")
+		(lib_id "ShiroFOCLib:COMP_TP101")
 		(at 218.44 147.32 0)
 		(unit 1)
@@
 	)
 	(symbol
-		(lib_id "Manual:COMP_TP101")
+		(lib_id "ShiroFOCLib:COMP_TP101")
 		(at 149.86 147.32 0)
 		(unit 1)
@@
 	)
 	(symbol
-		(lib_id "Manual:LR2512D_Kelvin")
+		(lib_id "ShiroFOCLib:LR2512D_Kelvin")
 		(at 120.65 67.31 0)
 		(unit 1)
@@
 			)
 		)
-		(property "Footprint" "Manual:R_Shunt_LR2512D_0m5_3W_Kelvin"
+		(property "Footprint" "ShiroFOCLib:R_Shunt_LR2512D_0m5_3W_Kelvin"
 			(at 118.872 67.31 90)
 			(effects
@@
 	)
 	(symbol
-		(lib_id "Manual:LR2512D_Kelvin")
+		(lib_id "ShiroFOCLib:LR2512D_Kelvin")
 		(at 209.55 67.31 0)
 		(unit 1)
@@
 			)
 		)
-		(property "Footprint" "Manual:R_Shunt_LR2512D_0m5_3W_Kelvin"
+		(property "Footprint" "ShiroFOCLib:R_Shunt_LR2512D_0m5_3W_Kelvin"
 			(at 207.772 67.31 90)
 			(effects
@@
 	)
 	(symbol
-		(lib_id "Manual:CSD88599Q5DC")
+		(lib_id "ShiroFOCLib:CSD88599Q5DC")
 		(at 52.07 50.8 0)
 		(unit 1)
@@
 			)
 		)
-		(property "Footprint" "Manual:DMM0022A"
+		(property "Footprint" "ShiroFOCLib:DMM0022A"
 			(at 48.26 74.93 0)
 			(effects
@@
 	)
 	(symbol
-		(lib_id "Manual:COMP_TP101")
+		(lib_id "ShiroFOCLib:COMP_TP101")
 		(at 132.08 147.32 0)
 		(unit 1)
@@
 	)
 	(symbol
-		(lib_id "Manual:COMP_TP101")
+		(lib_id "ShiroFOCLib:COMP_TP101")
 		(at 68.58 147.32 0)
 		(unit 1)
@@
 	)
 	(symbol
-		(lib_id "Manual:COMP_TP101")
+		(lib_id "ShiroFOCLib:COMP_TP101")
 		(at 114.3 147.32 0)
 		(unit 1)
@@
 	)
 	(symbol
-		(lib_id "Manual:COMP_TP101")
+		(lib_id "ShiroFOCLib:COMP_TP101")
 		(at 182.88 147.32 0)
 		(unit 1)
@@
 	)
 	(symbol
-		(lib_id "Manual:CSD88599Q5DC")
+		(lib_id "ShiroFOCLib:CSD88599Q5DC")
 		(at 138.43 50.8 0)
 		(unit 1)
@@
 			)
 		)
-		(property "Footprint" "Manual:DMM0022A"
+		(property "Footprint" "ShiroFOCLib:DMM0022A"
 			(at 134.62 74.93 0)
 			(effects
@@
 	)
 	(symbol
-		(lib_id "Manual:Motor_Phase_Terminals_3")
+		(lib_id "ShiroFOCLib:Motor_Phase_Terminals_3")
 		(at 257.81 123.19 0)
 		(mirror y)
@@
 	)
 	(symbol
-		(lib_id "Manual:COMP_TP101")
+		(lib_id "ShiroFOCLib:COMP_TP101")
 		(at 33.02 147.32 0)
 		(unit 1)
@@
 	)
 	(symbol
-		(lib_id "Manual:COMP_TP101")
+		(lib_id "ShiroFOCLib:COMP_TP101")
 		(at 50.8 147.32 0)
 		(unit 1)

Commit message: progress
Parts:
- J1: value MOTOR U/V/W -> MR60PW-M; footprint Connector_AMASS:AMASS_MR30PW-M_1x03_P3.50mm_Horizontal -> ShiroFOCLib:AMASS_MR60PW-M_1x03_P5.50mm_Horizontal; symbol ShiroFOCLib:Motor_Phase_Terminals_3 -> ShiroFOCLib:AMASS_MR60PW_M; MPN PCB feature -> MR60PW-M; Manufacturer PCB -> AMASS; Package (none) -> Horizontal through-hole, 3 contacts, 5.50 mm pitch; now in the parts list
Changed lines of the file:
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@@
 	)
 	(symbol
-		(lib_id "ShiroFOCLib:Motor_Phase_Terminals_3")
+		(lib_id "ShiroFOCLib:AMASS_MR60PW_M")
 		(at 257.81 123.19 0)
 		(mirror y)
 		(unit 1)
 		(exclude_from_sim no)
-		(in_bom no)
+		(in_bom yes)
 		(on_board yes)
 		(dnp no)
@@
 			)
 		)
-		(property "Value" "MOTOR U/V/W"
+		(property "Value" "MR60PW-M"
 			(at 257.81 110.49 0)
 			(effects
@@
 			)
 		)
-		(property "Footprint" "Connector_AMASS:AMASS_MR30PW-M_1x03_P3.50mm_Horizontal"
+		(property "Footprint" "ShiroFOCLib:AMASS_MR60PW-M_1x03_P5.50mm_Horizontal"
 			(at 280.924 100.33 0)
 			(effects
@@
 			)
 		)
-		(property "Datasheet" "~"
+		(property "Datasheet" "https://www.china-amass.com/public/upload/20240530/b96cfb0ffabb422135a2a15093576222.pdf"
 			(at 257.81 123.19 0)
 			(effects
@@
 			)
 		)
-		(property "Description" "Three plated motor-wire solder terminals"
+		(property "Description" "AMASS MR60PW-M horizontal male 3-pole motor connector; project pin assignment 1=U, 2=V, 3=W"
 			(at 257.81 135.128 0)
 			(effects
@@
 			)
 		)
-		(property "MPN" "PCB feature"
+		(property "MPN" "MR60PW-M"
 			(at 280.924 100.33 0)
 			(effects
@@
 			)
 		)
-		(property "Manufacturer" "PCB"
+		(property "Manufacturer" "AMASS"
 			(at 280.924 100.33 0)
 			(effects
 				(font
+					(size 1.27 1.27)
+				)
+				(hide yes)
+			)
+		)
+		(property "Package" "Horizontal through-hole, 3 contacts, 5.50 mm pitch"
+			(at 257.81 123.19 0)
+			(effects
+				(font

Commit message: progress + p4
Parts:
- J1: value MR60PW-M -> Motor phases - solder wires; footprint ShiroFOCLib:AMASS_MR60PW-M_1x03_P5.50mm_Horizontal -> ShiroFOCLib:WireSolder_Phase_1x03_P6.35mm_D2.90mm_Pad4.10mm; symbol ShiroFOCLib:AMASS_MR60PW_M -> ShiroFOCLib:DirectWire_Phase_3; MPN MR60PW-M -> (none); Manufacturer AMASS -> (none); Package Horizontal through-hole, 3 contacts, 5.50 mm pitch -> Plated wire holes; 2.90 mm drill; 6.35 mm pitch; now left out of the parts list
Changed lines of the file:
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@@
 	)
 	(symbol
-		(lib_id "ShiroFOCLib:AMASS_MR60PW_M")
+		(lib_id "ShiroFOCLib:DirectWire_Phase_3")
 		(at 257.81 123.19 0)
 		(mirror y)
 		(unit 1)
 		(exclude_from_sim no)
-		(in_bom yes)
+		(in_bom no)
 		(on_board yes)
 		(dnp no)
@@
 			)
 		)
-		(property "Value" "MR60PW-M"
+		(property "Value" "Motor phases - solder wires"
 			(at 257.81 110.49 0)
 			(effects
@@
 			)
 		)
-		(property "Footprint" "ShiroFOCLib:AMASS_MR60PW-M_1x03_P5.50mm_Horizontal"
+		(property "Footprint" "ShiroFOCLib:WireSolder_Phase_1x03_P6.35mm_D2.90mm_Pad4.10mm"
 			(at 280.924 100.33 0)
 			(effects
@@
 			)
 		)
-		(property "Datasheet" "https://www.china-amass.com/public/upload/20240530/b96cfb0ffabb422135a2a15093576222.pdf"
+		(property "Datasheet" ""
 			(at 257.81 123.19 0)
 			(effects
@@
 			)
 		)
-		(property "Description" "AMASS MR60PW-M horizontal male 3-pole motor connector; project pin assignment 1=U, 2=V, 3=W"
+		(property "Description" "Direct-solder plated wire terminals; no fitted connector"
 			(at 257.81 135.128 0)
 			(effects
@@
 			)
 		)
-		(property "MPN" "MR60PW-M"
+		(property "MPN" ""
 			(at 280.924 100.33 0)
 			(effects
@@
 			)
 		)
-		(property "Manufacturer" "AMASS"
+		(property "Manufacturer" ""
 			(at 280.924 100.33 0)
 			(effects
@@
 			)
 		)
-		(property "Package" "Horizontal through-hole, 3 contacts, 5.50 mm pitch"
+		(property "Package" "Plated wire holes; 2.90 mm drill; 6.35 mm pitch"
 			(at 257.81 123.19 0)
 			(effects

Commit message: weekend progress
Parts:
- J1: footprint ShiroFOCLib:WireSolder_Phase_1x03_P6.35mm_D2.90mm_Pad4.10mm -> ShiroFOCLib:WireSolder_Phase_1x03_P6.35mm_D3.00mm_Pad5.00x4.10mm_4xD0.40mm
Changed lines of the file:
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@@
 			)
 		)
-		(property "Footprint" "ShiroFOCLib:WireSolder_Phase_1x03_P6.35mm_D2.90mm_Pad4.10mm"
+		(property "Footprint" "ShiroFOCLib:WireSolder_Phase_1x03_P6.35mm_D3.00mm_Pad5.00x4.10mm_4xD0.40mm"
 			(at 280.924 100.33 0)
 			(effects

Commit message: half bridge progress
Parts:
- J1: footprint ShiroFOCLib:WireSolder_Phase_1x03_P6.35mm_D3.00mm_Pad5.00x4.10mm_4xD0.40mm -> ShiroFOCLib:WireSolder_Phase_1x03_P6.85mm_D3.00mm_Pad5.00x4.10mm_4xD0.40mm
Changed lines of the file:
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@@
 		(fields_autoplaced yes)
 		(property "Reference" "U3"
-			(at 227.33 39.624 0)
+			(at 227.33 38.1 0)
 			(effects
 				(font
@@
 		)
 		(property "Value" "CSD88599Q5DC"
-			(at 226.06 41.91 0)
+			(at 227.33 40.64 0)
 			(effects
 				(font
@@
 			)
 		)
-		(property "Footprint" "ShiroFOCLib:WireSolder_Phase_1x03_P6.35mm_D3.00mm_Pad5.00x4.10mm_4xD0.40mm"
+		(property "Footprint" "ShiroFOCLib:WireSolder_Phase_1x03_P6.85mm_D3.00mm_Pad5.00x4.10mm_4xD0.40mm"
 			(at 280.924 100.33 0)
 			(effects
