File: ShiroFOC/Manual_Layout_P3/Three-phase bridge.kicad_sch (KiCad schematic)
At the start: 34 parts, among them J1 Motor phases - solder wires, U1 CSD88599Q5DC, U2 CSD88599Q5DC, U3 CSD88599Q5DC

Commit message: shunts updated
Parts:
- R1, R3, R5: footprint ShiroFOCLib:R_Shunt_LR2512D_0m5_3W_Kelvin -> ShiroFOCLib:R_Shunt_HCS1206_0m5_2W_Kelvin; symbol ShiroFOCLib:LR2512D_Kelvin -> ShiroFOCLib:HCS1206_Kelvin; LCSC (none) -> C346511; MPN LR2512D-3W-0.5mR-1% -> HCS1206FTL500; Manufacturer Milliohm -> Stackpole Electronics; Power Rating 3 W; derate above 70 C to zero at 170 C per supplied datash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 -> 2 W at 100 C terminal temperature; derate to zero at 170 C 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; TCR (none) -> 200 ppm/C maximum magnitude; Tolerance (none) -> 1%
Changed lines of the file:
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@@
 	)
 	(symbol
-		(lib_id "ShiroFOCLib:LR2512D_Kelvin")
+		(lib_id "ShiroFOCLib:HCS1206_Kelvin")
 		(at 34.29 67.31 0)
 		(unit 1)
@@
 			)
 		)
-		(property "Footprint" "ShiroFOCLib:R_Shunt_LR2512D_0m5_3W_Kelvin"
+		(property "Footprint" "ShiroFOCLib:R_Shunt_HCS1206_0m5_2W_Kelvin"
 			(at 32.512 67.31 90)
 			(effects
@@
 			)
 		)
-		(property "Datasheet" "${KIPRJMOD}/../DataSheets/LR2512D_C500733.pdf"
+		(property "Datasheet" "${KIPRJMOD}/../DataSheets/HCS1206_C346511.pdf"
 			(at 34.29 67.31 0)
 			(effects
@@
 			)
 		)
-		(property "Power Rating" "3 W; derate above 70 C to zero at 170 C per supplied datasheet; actual cooling requires validation."
-			(at 0 0 0)
-			(effects
-				(font
-					(size 1.27 1.27)
-				)
-				(hide yes)
-			)
-		)
-		(property "Manufacturer" "Milliohm"
-			(at 0 0 0)
-			(effects
-				(font
-					(size 1.27 1.27)
-				)
-				(hide yes)
-			)
-		)
-		(property "MPN" "LR2512D-3W-0.5mR-1%"
+		(property "Power Rating" "2 W at 100 C terminal temperature; derate to zero at 170 C per HCS datasheet. Validate PCB cooling."
+			(at 0 0 0)
+			(effects
+				(font
+					(size 1.27 1.27)
+				)
+				(hide yes)
+			)
+		)
+		(property "Manufacturer" "Stackpole Electronics"
+			(at 0 0 0)
+			(effects
+				(font
+					(size 1.27 1.27)
+				)
+				(hide yes)
+			)
+		)
+		(property "MPN" "HCS1206FTL500"
 			(at 0 0 0)
 			(effects
@@
 			)
 		)
+		(property "LCSC" "C346511" (at 0 0 0) (effects (font (size 1.27 1.27)) (hide yes)))
+		(property "Tolerance" "1%" (at 0 0 0) (effects (font (size 1.27 1.27)) (hide yes)))
+		(property "TCR" "200 ppm/C maximum magnitude" (at 0 0 0) (effects (font (size 1.27 1.27)) (hide yes)))
 	)
 	(symbol
@@
 	)
 	(symbol
-		(lib_id "ShiroFOCLib:LR2512D_Kelvin")
+		(lib_id "ShiroFOCLib:HCS1206_Kelvin")
 		(at 120.65 67.31 0)
 		(unit 1)
@@
 			)
 		)
-		(property "Footprint" "ShiroFOCLib:R_Shunt_LR2512D_0m5_3W_Kelvin"
+		(property "Footprint" "ShiroFOCLib:R_Shunt_HCS1206_0m5_2W_Kelvin"
 			(at 118.872 67.31 90)
 			(effects
@@
 			)
 		)
-		(property "Datasheet" "${KIPRJMOD}/../DataSheets/LR2512D_C500733.pdf"
+		(property "Datasheet" "${KIPRJMOD}/../DataSheets/HCS1206_C346511.pdf"
 			(at 120.65 67.31 0)
 			(effects
@@
 			)
 		)
-		(property "Power Rating" "3 W; derate above 70 C to zero at 170 C per supplied datasheet; actual cooling requires validation."
-			(at 0 0 0)
-			(effects
-				(font
-					(size 1.27 1.27)
-				)
-				(hide yes)
-			)
-		)
-		(property "Manufacturer" "Milliohm"
-			(at 0 0 0)
-			(effects
-				(font
-					(size 1.27 1.27)
-				)
-				(hide yes)
-			)
-		)
-		(property "MPN" "LR2512D-3W-0.5mR-1%"
+		(property "Power Rating" "2 W at 100 C terminal temperature; derate to zero at 170 C per HCS datasheet. Validate PCB cooling."
+			(at 0 0 0)
+			(effects
+				(font
+					(size 1.27 1.27)
+				)
+				(hide yes)
+			)
+		)
+		(property "Manufacturer" "Stackpole Electronics"
+			(at 0 0 0)
+			(effects
+				(font
+					(size 1.27 1.27)
+				)
+				(hide yes)
+			)
+		)
+		(property "MPN" "HCS1206FTL500"
 			(at 0 0 0)
 			(effects
@@
 			)
 		)
+		(property "LCSC" "C346511" (at 0 0 0) (effects (font (size 1.27 1.27)) (hide yes)))
+		(property "Tolerance" "1%" (at 0 0 0) (effects (font (size 1.27 1.27)) (hide yes)))
+		(property "TCR" "200 ppm/C maximum magnitude" (at 0 0 0) (effects (font (size 1.27 1.27)) (hide yes)))
 	)
 	(symbol
@@
 	)
 	(symbol
-		(lib_id "ShiroFOCLib:LR2512D_Kelvin")
+		(lib_id "ShiroFOCLib:HCS1206_Kelvin")
 		(at 209.55 67.31 0)
 		(unit 1)
@@
 			)
 		)
-		(property "Footprint" "ShiroFOCLib:R_Shunt_LR2512D_0m5_3W_Kelvin"
+		(property "Footprint" "ShiroFOCLib:R_Shunt_HCS1206_0m5_2W_Kelvin"
 			(at 207.772 67.31 90)
 			(effects
@@
 			)
 		)
-		(property "Datasheet" "${KIPRJMOD}/../DataSheets/LR2512D_C500733.pdf"
+		(property "Datasheet" "${KIPRJMOD}/../DataSheets/HCS1206_C346511.pdf"
 			(at 209.55 67.31 0)
 			(effects
@@
 			)
 		)
-		(property "Power Rating" "3 W; derate above 70 C to zero at 170 C per supplied datasheet; actual cooling requires validation."
-			(at 0 0 0)
-			(effects
-				(font
-					(size 1.27 1.27)
-				)
-				(hide yes)
-			)
-		)
-		(property "Manufacturer" "Milliohm"
-			(at 0 0 0)
-			(effects
-				(font
-					(size 1.27 1.27)
-				)
-				(hide yes)
-			)
-		)
-		(property "MPN" "LR2512D-3W-0.5mR-1%"
+		(property "Power Rating" "2 W at 100 C terminal temperature; derate to zero at 170 C per HCS datasheet. Validate PCB cooling."
+			(at 0 0 0)
+			(effects
+				(font
+					(size 1.27 1.27)
+				)
+				(hide yes)
+			)
+		)
+		(property "Manufacturer" "Stackpole Electronics"
+			(at 0 0 0)
+			(effects
+				(font
+					(size 1.27 1.27)
+				)
+				(hide yes)
+			)
+		)
+		(property "MPN" "HCS1206FTL500"
 			(at 0 0 0)
 			(effects
@@
 			)
 		)
+		(property "LCSC" "C346511" (at 0 0 0) (effects (font (size 1.27 1.27)) (hide yes)))
+		(property "Tolerance" "1%" (at 0 0 0) (effects (font (size 1.27 1.27)) (hide yes)))
+		(property "TCR" "200 ppm/C maximum magnitude" (at 0 0 0) (effects (font (size 1.27 1.27)) (hide yes)))
 	)
 	(symbol

Commit message: mosfet stages and opamps revamped
Parts:
- C11, C3, C7: value 4.7uF -> 10uF; BOM Comments Local VM bypass. Nominal capacitance; effective capacitance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 -> Local VM bypass; same part as DC-link ceramic bank. Approxi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; LCSC (none) -> C3840810; MPN C3225X7S2A475K200AB -> CL32Y106KCVZNWE; Manufacturer TDK -> Samsung Electro-Mechanics; Product URL https://product.tdk.com/en/search/capacitor/ceramic/mlcc/in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 -> https://product.samsungsem.com/mlcc/CL32Y106KCVZNW.do
Changed lines of the file:
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@@
 			)
 		)
+		(property "LCSC" "C346511"
+			(at 0 0 0)
+			(effects
+				(font
+					(size 1.27 1.27)
+				)
+				(hide yes)
+			)
+		)
+		(property "Tolerance" "1%"
+			(at 0 0 0)
+			(effects
+				(font
+					(size 1.27 1.27)
+				)
+				(hide yes)
+			)
+		)
+		(property "TCR" "200 ppm/C maximum magnitude"
+			(at 0 0 0)
+			(effects
+				(font
+					(size 1.27 1.27)
+				)
+				(hide yes)
+			)
+		)
 		(pin "1"
 		)
@@
 			)
 		)
-		(property "LCSC" "C346511" (at 0 0 0) (effects (font (size 1.27 1.27)) (hide yes)))
-		(property "Tolerance" "1%" (at 0 0 0) (effects (font (size 1.27 1.27)) (hide yes)))
-		(property "TCR" "200 ppm/C maximum magnitude" (at 0 0 0) (effects (font (size 1.27 1.27)) (hide yes)))
 	)
 	(symbol
@@
 			)
 		)
+		(property "LCSC" "C346511"
+			(at 0 0 0)
+			(effects
+				(font
+					(size 1.27 1.27)
+				)
+				(hide yes)
+			)
+		)
+		(property "Tolerance" "1%"
+			(at 0 0 0)
+			(effects
+				(font
+					(size 1.27 1.27)
+				)
+				(hide yes)
+			)
+		)
+		(property "TCR" "200 ppm/C maximum magnitude"
+			(at 0 0 0)
+			(effects
+				(font
+					(size 1.27 1.27)
+				)
+				(hide yes)
+			)
+		)
 		(pin "1"
 		)
@@
 			)
 		)
-		(property "LCSC" "C346511" (at 0 0 0) (effects (font (size 1.27 1.27)) (hide yes)))
-		(property "Tolerance" "1%" (at 0 0 0) (effects (font (size 1.27 1.27)) (hide yes)))
-		(property "TCR" "200 ppm/C maximum magnitude" (at 0 0 0) (effects (font (size 1.27 1.27)) (hide yes)))
 	)
 	(symbol
@@
 			)
 		)
+		(property "LCSC" "C346511"
+			(at 0 0 0)
+			(effects
+				(font
+					(size 1.27 1.27)
+				)
+				(hide yes)
+			)
+		)
+		(property "Tolerance" "1%"
+			(at 0 0 0)
+			(effects
+				(font
+					(size 1.27 1.27)
+				)
+				(hide yes)
+			)
+		)
+		(property "TCR" "200 ppm/C maximum magnitude"
+			(at 0 0 0)
+			(effects
+				(font
+					(size 1.27 1.27)
+				)
+				(hide yes)
+			)
+		)
 		(pin "1"
 		)
@@
 			)
 		)
-		(property "LCSC" "C346511" (at 0 0 0) (effects (font (size 1.27 1.27)) (hide yes)))
-		(property "Tolerance" "1%" (at 0 0 0) (effects (font (size 1.27 1.27)) (hide yes)))
-		(property "TCR" "200 ppm/C maximum magnitude" (at 0 0 0) (effects (font (size 1.27 1.27)) (hide yes)))
 	)
 	(symbol
@@
 			)
 		)
-		(property "Value" "4.7uF"
+		(property "Value" "10uF"
 			(at 62.484 32.766 0)
 			(effects
@@
 			)
 		)
-		(property "Datasheet" "https://product.tdk.com/info/en/documents/chara_sheet/C3225X7S2A475K200AB.pdf"
+		(property "Datasheet" "https://mm.digikey.com/Volume0/opasdata/d220001/medias/docus/3563/CL32Y106KCVZNWE_Tech_Article.pdf"
 			(at 62.23 30.48 0)
 			(effects
@@
 			)
 		)
-		(property "Product URL" "https://product.tdk.com/en/search/capacitor/ceramic/mlcc/info?part_no=C3225X7S2A475K200AB"
+		(property "Product URL" "https://product.samsungsem.com/mlcc/CL32Y106KCVZNW.do"
 			(at 0 0 0)
 			(effects
@@
 			)
 		)
-		(property "BOM Comments" "Local VM bypass. Nominal capacitance; effective capacitance and RMS ripple temperature require final PWM/layout validation. Generic STEP is visualization only; maximum component height 2.2 mm."
+		(property "BOM Comments" "Local VM bypass; same part as DC-link ceramic bank. Approximately 3.3 uF typical at 42 V before temperature, tolerance and aging. Validate RMS ripple heating. Generic STEP is visualization only; maximum component height 2.8 mm."
 			(at 0 0 0)
 			(effects
@@
 			)
 		)
-		(property "Manufacturer" "TDK"
+		(property "Manufacturer" "Samsung Electro-Mechanics"
 			(at 0 0 0)
 			(effects
@@
 			)
 		)
-		(property "MPN" "C3225X7S2A475K200AB"
+		(property "MPN" "CL32Y106KCVZNWE"
 			(at 0 0 0)
 			(effects
@@
 			)
 		)
+		(property "LCSC" "C3840810"
+			(at 0 0 0)
+			(effects
+				(font
+					(size 1 1)
+				)
+				(hide yes)
+			)
+		)
 		(pin "2"
 		)
@@
 			)
 		)
-		(property "Value" "4.7uF"
+		(property "Value" "10uF"
 			(at 148.844 32.766 0)
 			(effects
@@
 			)
 		)
-		(property "Datasheet" "https://product.tdk.com/info/en/documents/chara_sheet/C3225X7S2A475K200AB.pdf"
+		(property "Datasheet" "https://mm.digikey.com/Volume0/opasdata/d220001/medias/docus/3563/CL32Y106KCVZNWE_Tech_Article.pdf"
 			(at 148.59 30.48 0)
 			(effects
@@
 			)
 		)
-		(property "Product URL" "https://product.tdk.com/en/search/capacitor/ceramic/mlcc/info?part_no=C3225X7S2A475K200AB"
+		(property "Product URL" "https://product.samsungsem.com/mlcc/CL32Y106KCVZNW.do"
 			(at 0 0 0)
 			(effects
@@
 			)
 		)
-		(property "BOM Comments" "Local VM bypass. Nominal capacitance; effective capacitance and RMS ripple temperature require final PWM/layout validation. Generic STEP is visualization only; maximum component height 2.2 mm."
+		(property "BOM Comments" "Local VM bypass; same part as DC-link ceramic bank. Approximately 3.3 uF typical at 42 V before temperature, tolerance and aging. Validate RMS ripple heating. Generic STEP is visualization only; maximum component height 2.8 mm."
 			(at 0 0 0)
 			(effects
@@
 			)
 		)
-		(property "Manufacturer" "TDK"
+		(property "Manufacturer" "Samsung Electro-Mechanics"
 			(at 0 0 0)
 			(effects
@@
 			)
 		)
-		(property "MPN" "C3225X7S2A475K200AB"
+		(property "MPN" "CL32Y106KCVZNWE"
 			(at 0 0 0)
 			(effects
@@
 			)
 		)
+		(property "LCSC" "C3840810"
+			(at 0 0 0)
+			(effects
+				(font
+					(size 1 1)
+				)
+				(hide yes)
+			)
+		)
 		(pin "2"
 		)
@@
 			)
 		)
-		(property "Value" "4.7uF"
+		(property "Value" "10uF"
 			(at 237.744 32.766 0)
 			(effects
@@
 			)
 		)
-		(property "Datasheet" "https://product.tdk.com/info/en/documents/chara_sheet/C3225X7S2A475K200AB.pdf"
+		(property "Datasheet" "https://mm.digikey.com/Volume0/opasdata/d220001/medias/docus/3563/CL32Y106KCVZNWE_Tech_Article.pdf"
 			(at 237.49 30.48 0)
 			(effects
@@
 			)
 		)
-		(property "Product URL" "https://product.tdk.com/en/search/capacitor/ceramic/mlcc/info?part_no=C3225X7S2A475K200AB"
+		(property "Product URL" "https://product.samsungsem.com/mlcc/CL32Y106KCVZNW.do"
 			(at 0 0 0)
 			(effects
@@
 			)
 		)
-		(property "BOM Comments" "Local VM bypass. Nominal capacitance; effective capacitance and RMS ripple temperature require final PWM/layout validation. Generic STEP is visualization only; maximum component height 2.2 mm."
+		(property "BOM Comments" "Local VM bypass; same part as DC-link ceramic bank. Approximately 3.3 uF typical at 42 V before temperature, tolerance and aging. Validate RMS ripple heating. Generic STEP is visualization only; maximum component height 2.8 mm."
 			(at 0 0 0)
 			(effects
@@
 			)
 		)
-		(property "Manufacturer" "TDK"
+		(property "Manufacturer" "Samsung Electro-Mechanics"
 			(at 0 0 0)
 			(effects
@@
 			)
 		)
-		(property "MPN" "C3225X7S2A475K200AB"
+		(property "MPN" "CL32Y106KCVZNWE"
 			(at 0 0 0)
 			(effects
@@
 				)
 				(hide yes)
+			)
+		)
+		(property "LCSC" "C3840810"
+			(at 0 0 0)
+			(effects
+				(font
+					(size 1 1)
+				)
+				(hide yes)
