File: ShiroFOC/Manual_Layout_P3/06_Current_Temperature.kicad_sch (KiCad schematic)
At the start: 37 parts, among them U4 STSPIN32G4

Commit message: usb and pwr mux
Parts:
- added TP414, TP424, TP434: SCOPE GND, TestPoint:TestPoint_Pad_D1.0mm, symbol Manual:COMP_TP101
Connections:
- net GND: now also TP414.1, TP424.1, TP434.1

Commit message: CAN layout
Parts:
- C414: symbol Manual:COMP_C414 -> ShiroFOCLib:COMP_C414
- C424: symbol Manual:COMP_C424 -> ShiroFOCLib:COMP_C424
- C434: symbol Manual:COMP_C434 -> ShiroFOCLib:COMP_C434
- C711: symbol Manual:COMP_C711 -> ShiroFOCLib:COMP_C711
- C712: symbol Manual:COMP_C712 -> ShiroFOCLib:COMP_C712
- C713: symbol Manual:COMP_C713 -> ShiroFOCLib:COMP_C713
- R410: symbol Manual:COMP_R410 -> ShiroFOCLib:COMP_R410
- R417: symbol Manual:COMP_R417 -> ShiroFOCLib:COMP_R417
- R418: symbol Manual:COMP_R418 -> ShiroFOCLib:COMP_R418
- R419: symbol Manual:COMP_R419 -> ShiroFOCLib:COMP_R419
- R420: symbol Manual:COMP_R420 -> ShiroFOCLib:COMP_R420
- R427: symbol Manual:COMP_R427 -> ShiroFOCLib:COMP_R427
- R428: symbol Manual:COMP_R428 -> ShiroFOCLib:COMP_R428
- R429: symbol Manual:COMP_R429 -> ShiroFOCLib:COMP_R429
- R430: symbol Manual:COMP_R430 -> ShiroFOCLib:COMP_R430
- R437: symbol Manual:COMP_R437 -> ShiroFOCLib:COMP_R437
- R438: symbol Manual:COMP_R438 -> ShiroFOCLib:COMP_R438
- R439: symbol Manual:COMP_R439 -> ShiroFOCLib:COMP_R439
- R441: symbol Manual:COMP_R441 -> ShiroFOCLib:COMP_R441
- R442: symbol Manual:COMP_R442 -> ShiroFOCLib:COMP_R442
- R443: symbol Manual:COMP_R443 -> ShiroFOCLib:COMP_R443
- R701: symbol Manual:COMP_R701 -> ShiroFOCLib:COMP_R701
- R702: symbol Manual:COMP_R702 -> ShiroFOCLib:COMP_R702
- R703: symbol Manual:COMP_R703 -> ShiroFOCLib:COMP_R703
- R711: symbol Manual:COMP_R711 -> ShiroFOCLib:COMP_R711
- R712: symbol Manual:COMP_R712 -> ShiroFOCLib:COMP_R712
- R713: symbol Manual:COMP_R713 -> ShiroFOCLib:COMP_R713
- TH701: symbol Manual:COMP_TH701 -> ShiroFOCLib:COMP_TH701
- TH702: symbol Manual:COMP_TH702 -> ShiroFOCLib:COMP_TH702
- TH703: symbol Manual:COMP_TH703 -> ShiroFOCLib:COMP_TH703
- TP1018: symbol Manual:COMP_TP1018 -> ShiroFOCLib:COMP_TP1018
- TP1019: symbol Manual:COMP_TP1019 -> ShiroFOCLib:COMP_TP1019
- TP1020: symbol Manual:COMP_TP1020 -> ShiroFOCLib:COMP_TP1020
- TP414, TP424, TP434: symbol Manual:COMP_TP101 -> ShiroFOCLib:COMP_TP101
- TP701: symbol Manual:COMP_TP701 -> ShiroFOCLib:COMP_TP701
- TP702: symbol Manual:COMP_TP702 -> ShiroFOCLib:COMP_TP702
- TP703: symbol Manual:COMP_TP703 -> ShiroFOCLib:COMP_TP703
- U4: footprint Manual:QFN_IN32G4_STM -> ShiroFOCLib:QFN_IN32G4_STM; symbol Manual:STSPIN32G4_Functional -> ShiroFOCLib:STSPIN32G4_Functional
Changed lines of the file:
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@@
 	)
 	(symbol
-		(lib_id "Manual:COMP_TP1019")
+		(lib_id "ShiroFOCLib:COMP_TP1019")
 		(at 256.54 104.14 0)
 		(unit 1)
@@
 	)
 	(symbol
-		(lib_id "Manual:COMP_TP703")
+		(lib_id "ShiroFOCLib:COMP_TP703")
 		(at 363.22 219.71 0)
 		(unit 1)
@@
 	)
 	(symbol
-		(lib_id "Manual:COMP_R430")
+		(lib_id "ShiroFOCLib:COMP_R430")
 		(at 300.99 133.35 0)
 		(unit 1)
@@
 	)
 	(symbol
-		(lib_id "Manual:COMP_TP1020")
+		(lib_id "ShiroFOCLib:COMP_TP1020")
 		(at 387.35 104.14 0)
 		(unit 1)
@@
 	)
 	(symbol
-		(lib_id "Manual:COMP_TP101")
+		(lib_id "ShiroFOCLib:COMP_TP101")
 		(at 248.92 130.81 0)
 		(unit 1)
@@
 	)
 	(symbol
-		(lib_id "Manual:PWR_VREFplus")
+		(lib_id "ShiroFOCLib:PWR_VREFplus")
 		(at 27.94 133.35 0)
 		(unit 1)
@@
 	)
 	(symbol
-		(lib_id "Manual:PWR_GND")
+		(lib_id "ShiroFOCLib:PWR_GND")
 		(at 45.72 246.38 0)
 		(unit 1)
@@
 	)
 	(symbol
-		(lib_id "Manual:COMP_R438")
+		(lib_id "ShiroFOCLib:COMP_R438")
 		(at 308.61 97.79 0)
 		(unit 1)
@@
 	)
 	(symbol
-		(lib_id "Manual:PWR_3V3")
+		(lib_id "ShiroFOCLib:PWR_3V3")
 		(at 176.53 189.23 0)
 		(unit 1)
@@
 	)
 	(symbol
-		(lib_id "Manual:COMP_R419")
+		(lib_id "ShiroFOCLib:COMP_R419")
 		(at 92.71 66.04 0)
 		(unit 1)
@@
 	)
 	(symbol
-		(lib_id "Manual:COMP_TP1018")
+		(lib_id "ShiroFOCLib:COMP_TP1018")
 		(at 125.73 104.14 0)
 		(unit 1)
@@
 	)
 	(symbol
-		(lib_id "Manual:PWR_GND")
+		(lib_id "ShiroFOCLib:PWR_GND")
 		(at 307.34 246.38 0)
 		(unit 1)
@@
 	)
 	(symbol
-		(lib_id "Manual:PWR_GND")
+		(lib_id "ShiroFOCLib:PWR_GND")
 		(at 101.6 246.38 0)
 		(unit 1)
@@
 	)
 	(symbol
-		(lib_id "Manual:PWR_GND")
+		(lib_id "ShiroFOCLib:PWR_GND")
 		(at 176.53 246.38 0)
 		(unit 1)
@@
 	)
 	(symbol
-		(lib_id "Manual:COMP_R441")
+		(lib_id "ShiroFOCLib:COMP_R441")
 		(at 62.23 144.78 0)
 		(unit 1)
@@
 	)
 	(symbol
-		(lib_id "Manual:COMP_R712")
+		(lib_id "ShiroFOCLib:COMP_R712")
 		(at 208.28 219.71 0)
 		(unit 1)
@@
 	)
 	(symbol
-		(lib_id "Manual:PWR_VREFplus")
+		(lib_id "ShiroFOCLib:PWR_VREFplus")
 		(at 158.75 133.35 0)
 		(unit 1)
@@
 	)
 	(symbol
-		(lib_id "Manual:PWR_GND")
+		(lib_id "ShiroFOCLib:PWR_GND")
 		(at 232.41 246.38 0)
 		(unit 1)
@@
 	)
 	(symbol
-		(lib_id "Manual:COMP_R417")
+		(lib_id "ShiroFOCLib:COMP_R417")
 		(at 46.99 110.49 0)
 		(unit 1)
@@
 	)
 	(symbol
-		(lib_id "Manual:PWR_3V3")
+		(lib_id "ShiroFOCLib:PWR_3V3")
 		(at 45.72 189.23 0)
 		(unit 1)
@@
 	(symbol
 		(lib_name "STSPIN32G4_Functional_1")
-		(lib_id "Manual:STSPIN32G4_Functional")
+		(lib_id "ShiroFOCLib:STSPIN32G4_Functional")
 		(at 222.25 104.14 0)
 		(unit 5)
@@
 			)
 		)
-		(property "Footprint" "Manual:QFN_IN32G4_STM"
+		(property "Footprint" "ShiroFOCLib:QFN_IN32G4_STM"
 			(at 222.25 167.64 0)
 			(effects
@@
 	)
 	(symbol
-		(lib_id "Manual:COMP_R713")
+		(lib_id "ShiroFOCLib:COMP_R713")
 		(at 339.09 219.71 0)
 		(unit 1)
@@
 	)
 	(symbol
-		(lib_id "Manual:PWR_3V3")
+		(lib_id "ShiroFOCLib:PWR_3V3")
 		(at 307.34 189.23 0)
 		(unit 1)
@@
 	)
 	(symbol
-		(lib_id "Manual:COMP_R429")
+		(lib_id "ShiroFOCLib:COMP_R429")
 		(at 223.52 66.04 0)
 		(unit 1)
@@
 	)
 	(symbol
-		(lib_id "Manual:COMP_R427")
+		(lib_id "ShiroFOCLib:COMP_R427")
 		(at 177.8 110.49 0)
 		(unit 1)
@@
 	)
 	(symbol
-		(lib_id "Manual:COMP_TH703")
+		(lib_id "ShiroFOCLib:COMP_TH703")
 		(at 307.34 236.22 0)
 		(unit 1)
@@
 	)
 	(symbol
-		(lib_id "Manual:COMP_R418")
+		(lib_id "ShiroFOCLib:COMP_R418")
 		(at 46.99 97.79 0)
 		(unit 1)
@@
 	)
 	(symbol
-		(lib_id "Manual:COMP_TP101")
+		(lib_id "ShiroFOCLib:COMP_TP101")
 		(at 118.11 130.81 0)
 		(unit 1)
@@
 	)
 	(symbol
-		(lib_id "Manual:COMP_R428")
+		(lib_id "ShiroFOCLib:COMP_R428")
 		(at 177.8 97.79 0)
 		(unit 1)
@@
 	)
 	(symbol
-		(lib_id "Manual:PWR_GND")
+		(lib_id "ShiroFOCLib:PWR_GND")
 		(at 323.85 153.67 0)
 		(unit 1)
@@
 	)
 	(symbol
-		(lib_id "Manual:COMP_TH702")
+		(lib_id "ShiroFOCLib:COMP_TH702")
 		(at 176.53 236.22 0)
 		(unit 1)
@@
 	)
 	(symbol
-		(lib_id "Manual:COMP_R437")
+		(lib_id "ShiroFOCLib:COMP_R437")
 		(at 308.61 110.49 0)
 		(unit 1)
@@
 	)
 	(symbol
-		(lib_id "Manual:PWR_GND")
+		(lib_id "ShiroFOCLib:PWR_GND")
 		(at 363.22 246.38 0)
 		(unit 1)
@@
 	(symbol
 		(lib_name "STSPIN32G4_Functional_2")
-		(lib_id "Manual:STSPIN32G4_Functional")
+		(lib_id "ShiroFOCLib:STSPIN32G4_Functional")
 		(at 91.44 104.14 0)
 		(unit 4)
@@
 			)
 		)
-		(property "Footprint" "Manual:QFN_IN32G4_STM"
+		(property "Footprint" "ShiroFOCLib:QFN_IN32G4_STM"
 			(at 91.44 167.64 0)
 			(effects
@@
 	)
 	(symbol
-		(lib_id "Manual:COMP_TH701")
+		(lib_id "ShiroFOCLib:COMP_TH701")
 		(at 45.72 236.22 0)
 		(unit 1)
@@
 	)
 	(symbol
-		(lib_id "Manual:PWR_VREFplus")
+		(lib_id "ShiroFOCLib:PWR_VREFplus")
 		(at 289.56 133.35 0)
 		(unit 1)
@@
 	)
 	(symbol
-		(lib_id "Manual:COMP_R420")
+		(lib_id "ShiroFOCLib:COMP_R420")
 		(at 170.18 133.35 0)
 		(unit 1)
@@
 	)
 	(symbol
-		(lib_id "Manual:COMP_R439")
+		(lib_id "ShiroFOCLib:COMP_R439")
 		(at 354.33 66.04 0)
 		(unit 1)
@@
 	)
 	(symbol
-		(lib_id "Manual:PWR_GND")
+		(lib_id "ShiroFOCLib:PWR_GND")
 		(at 193.04 153.67 0)
 		(unit 1)
@@
 	)
 	(symbol
-		(lib_id "Manual:COMP_R443")
+		(lib_id "ShiroFOCLib:COMP_R443")
 		(at 323.85 144.78 0)
 		(unit 1)
@@
 	)
 	(symbol
-		(lib_id "Manual:COMP_R711")
+		(lib_id "ShiroFOCLib:COMP_R711")
 		(at 77.47 219.71 0)
 		(unit 1)
@@
 	)
 	(symbol
-		(lib_id "Manual:COMP_C711")
+		(lib_id "ShiroFOCLib:COMP_C711")
 		(at 101.6 236.22 0)
 		(unit 1)
@@
 	)
 	(symbol
-		(lib_id "Manual:COMP_R701")
+		(lib_id "ShiroFOCLib:COMP_R701")
 		(at 45.72 200.66 0)
 		(unit 1)
@@
 	)
 	(symbol
-		(lib_id "Manual:COMP_R702")
+		(lib_id "ShiroFOCLib:COMP_R702")
 		(at 176.53 200.66 0)
 		(unit 1)
@@
 	)
 	(symbol
-		(lib_id "Manual:COMP_TP701")
+		(lib_id "ShiroFOCLib:COMP_TP701")
 		(at 101.6 219.71 0)
 		(unit 1)
@@
 	)
 	(symbol
-		(lib_id "Manual:COMP_C713")
+		(lib_id "ShiroFOCLib:COMP_C713")
 		(at 363.22 236.22 0)
 		(unit 1)
@@
 	)
 	(symbol
-		(lib_id "Manual:PWR_GND")
+		(lib_id "ShiroFOCLib:PWR_GND")
 		(at 62.23 153.67 0)
 		(unit 1)
@@
 	)
 	(symbol
-		(lib_id "Manual:COMP_C712")
+		(lib_id "ShiroFOCLib:COMP_C712")
 		(at 232.41 236.22 0)
 		(unit 1)
@@
 	)
 	(symbol
-		(lib_id "Manual:COMP_C434")
+		(lib_id "ShiroFOCLib:COMP_C434")
 		(at 354.33 53.34 0)
 		(unit 1)
@@
 	)
 	(symbol
-		(lib_id "Manual:COMP_R703")
+		(lib_id "ShiroFOCLib:COMP_R703")
 		(at 307.34 200.66 0)
 		(unit 1)
@@
 	)
 	(symbol
-		(lib_id "Manual:COMP_C414")
+		(lib_id "ShiroFOCLib:COMP_C414")
 		(at 92.71 53.34 0)
 		(unit 1)
@@
 	)
 	(symbol
-		(lib_id "Manual:COMP_R410")
+		(lib_id "ShiroFOCLib:COMP_R410")
 		(at 39.37 133.35 0)
 		(unit 1)
@@
 	)
 	(symbol
-		(lib_id "Manual:COMP_R442")
+		(lib_id "ShiroFOCLib:COMP_R442")
 		(at 193.04 144.78 0)
 		(unit 1)
@@
 	)
 	(symbol
-		(lib_id "Manual:COMP_TP101")
+		(lib_id "ShiroFOCLib:COMP_TP101")
 		(at 379.73 130.81 0)
 		(unit 1)
@@
 	)
 	(symbol
-		(lib_id "Manual:STSPIN32G4_Functional")
+		(lib_id "ShiroFOCLib:STSPIN32G4_Functional")
 		(at 353.06 104.14 0)
 		(unit 6)
@@
 			)
 		)
-		(property "Footprint" "Manual:QFN_IN32G4_STM"
+		(property "Footprint" "ShiroFOCLib:QFN_IN32G4_STM"
 			(at 353.06 167.64 0)
 			(effects
@@
 	)
 	(symbol
-		(lib_id "Manual:COMP_TP702")
+		(lib_id "ShiroFOCLib:COMP_TP702")
 		(at 232.41 219.71 0)
 		(unit 1)
@@
 	)
 	(symbol
-		(lib_id "Manual:COMP_C424")
+		(lib_id "ShiroFOCLib:COMP_C424")
 		(at 223.52 53.34 0)
 		(unit 1)

Commit message: weekend progress
Parts:
- TP701: value NTC_PHASE_A -> NTC_PHASE_B; Test_Net NTC_PHASE_A -> NTC_PHASE_B
- TP702: value NTC_PHASE_B -> NTC_PHASE_A; Test_Net NTC_PHASE_B -> NTC_PHASE_A
Connections:
- net NTC_A_RAW: now also R702.2, R712.1, TH702.1; no longer R701.2, R711.1, TH701.1
- net NTC_B_RAW: now also R701.2, R711.1, TH701.1; no longer R702.2, R712.1, TH702.1
- net NTC_PHASE_A: now also C712.1, R712.2, TP702.1; no longer C711.1, R711.2, TP701.1
- net NTC_PHASE_B: now also C711.1, R711.2, TP701.1; no longer C712.1, R712.2, TP702.1
Changed lines of the file:
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@@
 		)
 	)
-	(text "NTC B - place beside phase V"
+	(text "NTC A - place beside phase U"
 		(exclude_from_sim no)
 		(at 148.59 177.8 0)
@@
 		)
 	)
-	(text "NTC A - place beside phase U"
+	(text "NTC B - place beside phase V"
 		(exclude_from_sim no)
 		(at 17.78 177.8 0)
@@
 		)
 	)
-	(label "NTC_B_RAW"
+	(label "NTC_A_RAW"
 		(at 176.53 219.71 0)
 		(effects
@@
 		)
 	)
-	(label "NTC_A_RAW"
+	(label "NTC_B_RAW"
 		(at 45.72 219.71 0)
 		(effects
@@
 		)
 	)
-	(global_label "NTC_PHASE_B"
+	(global_label "NTC_PHASE_A"
 		(shape bidirectional)
 		(at 254 219.71 0)
@@
 		)
 	)
-	(global_label "NTC_PHASE_A"
+	(global_label "NTC_PHASE_B"
 		(shape bidirectional)
 		(at 123.19 219.71 0)
@@
 			)
 		)
-		(property "Value" "NTC_PHASE_A"
+		(property "Value" "NTC_PHASE_B"
 			(at 104.14 217.17 0)
 			(effects
@@
 			)
 		)
-		(property "Description" "Test point: NTC_PHASE_A"
+		(property "Description" "Test point: NTC_PHASE_B"
 			(at 101.6 219.71 0)
 			(effects
@@
 			)
 		)
-		(property "Test_Net" "NTC_PHASE_A"
+		(property "Test_Net" "NTC_PHASE_B"
 			(at 104.14 219.71 0)
 			(effects
@@
 			)
 		)
-		(property "Value" "NTC_PHASE_B"
+		(property "Value" "NTC_PHASE_A"
 			(at 234.95 217.17 0)
 			(effects
@@
 			)
 		)
-		(property "Description" "Test point: NTC_PHASE_B"
+		(property "Description" "Test point: NTC_PHASE_A"
 			(at 232.41 219.71 0)
 			(effects
@@
 			)
 		)
-		(property "Test_Net" "NTC_PHASE_B"
+		(property "Test_Net" "NTC_PHASE_A"
 			(at 234.95 219.71 0)
 			(effects

Commit message: op amp traces draft
swapped phase U and W op amps
Parts:
- TP1018: value OPO_U1 -> OPO_W1; Test_Net OPO_U1 -> OPO_W1
- TP1020: value OPO_W1 -> OPO_U1; Test_Net OPO_W1 -> OPO_U1
Connections:
- net OPN_U1: now also C434.2, R438.2, R439.2, U4.25 (-); no longer C414.2, R418.2, R419.2, U4.16 (-)
- net OPN_W1: now also C414.2, R418.2, R419.2, U4.16 (-); no longer C434.2, R438.2, R439.2, U4.25 (-)
- net OPO_U1: now also C434.1, R439.1, TP1020.1, U4.24 (OUT); no longer C414.1, R419.1, TP1018.1, U4.15 (OUT)
- net OPO_W1: now also C414.1, R419.1, TP1018.1, U4.15 (OUT); no longer C434.1, R439.1, TP1020.1, U4.24 (OUT)
- net OPP_U1: now also R430.2, R437.2, R443.1, U4.23 (+); no longer R410.2, R417.2, R441.1, U4.14 (+)
- net OPP_W1: now also R410.2, R417.2, R441.1, U4.14 (+); no longer R430.2, R437.2, R443.1, U4.23 (+)
- net SHUNT_U_SENSE_N: now also R438.1; no longer R418.1
- net SHUNT_U_SENSE_P: now also R437.1; no longer R417.1
- net SHUNT_W_SENSE_N: now also R418.1; no longer R438.1
- net SHUNT_W_SENSE_P: now also R417.1; no longer R437.1
Other:
- note added: "PHASE U / OPAMP3"
- note added: "PHASE W / OPAMP1"
- note removed: "PHASE U / OPAMP1"
- note removed: "PHASE W / OPAMP3"
Changed lines of the file:
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@@
 		)
 	)
-	(text "PHASE U / OPAMP1"
+	(text "PHASE W / OPAMP1"
 		(exclude_from_sim no)
 		(at 17.78 41.91 0)
@@
 		)
 	)
-	(text "PHASE W / OPAMP3"
+	(text "PHASE U / OPAMP3"
 		(exclude_from_sim no)
 		(at 279.4 41.91 0)
@@
 		)
 	)
-	(label "OPN_U1"
+	(label "OPN_W1"
 		(at 57.15 97.79 0)
 		(effects
@@
 		)
 	)
-	(label "OPP_U1"
+	(label "OPP_W1"
 		(at 54.61 110.49 0)
 		(effects
@@
 		)
 	)
-	(label "OPN_W1"
+	(label "OPN_U1"
 		(at 318.77 97.79 0)
 		(effects
@@
 		)
 	)
-	(label "OPP_W1"
+	(label "OPP_U1"
 		(at 316.23 110.49 0)
 		(effects
@@
 		)
 	)
-	(global_label "SHUNT_U_SENSE_N"
+	(global_label "SHUNT_W_SENSE_N"
 		(shape bidirectional)
 		(at 34.29 97.79 180)
@@
 		)
 	)
-	(global_label "OPO_W1"
+	(global_label "OPO_U1"
 		(shape bidirectional)
 		(at 388.62 104.14 0)
@@
 		)
 	)
-	(global_label "SHUNT_W_SENSE_N"
+	(global_label "SHUNT_U_SENSE_N"
 		(shape bidirectional)
 		(at 295.91 97.79 180)
@@
 		)
 	)
-	(global_label "SHUNT_W_SENSE_P"
+	(global_label "SHUNT_U_SENSE_P"
 		(shape bidirectional)
 		(at 295.91 110.49 180)
@@
 		)
 	)
-	(global_label "OPO_U1"
+	(global_label "OPO_W1"
 		(shape bidirectional)
 		(at 127 104.14 0)
@@
 		)
 	)
-	(global_label "SHUNT_U_SENSE_P"
+	(global_label "SHUNT_W_SENSE_P"
 		(shape bidirectional)
 		(at 34.29 110.49 180)
@@
 			)
 		)
-		(property "Value" "OPO_W1"
+		(property "Value" "OPO_U1"
 			(at 389.89 101.6 0)
 			(effects
@@
 			)
 		)
-		(property "Description" "Test point: OPO_W1"
+		(property "Description" "Test point: OPO_U1"
 			(at 387.35 104.14 0)
 			(effects
@@
 			)
 		)
-		(property "Test_Net" "OPO_W1"
+		(property "Test_Net" "OPO_U1"
 			(at 389.89 104.14 0)
 			(effects
@@
 			)
 		)
-		(property "Value" "OPO_U1"
+		(property "Value" "OPO_W1"
 			(at 128.27 101.6 0)
 			(effects
@@
 			)
 		)
-		(property "Description" "Test point: OPO_U1"
+		(property "Description" "Test point: OPO_W1"
 			(at 125.73 104.14 0)
 			(effects
@@
 			)
 		)
-		(property "Test_Net" "OPO_U1"
+		(property "Test_Net" "OPO_W1"
 			(at 128.27 104.14 0)
 			(effects
