File: ShiroFOC/Manual_Layout_P3/09_Feedback_Selection.kicad_sch (KiCad schematic)
At the start: 26 parts, among them J601 EXT ENCODER / HALL, U602 TMUX1574PW, U603 74LVC3G17, U604 TPS2553DBVR

Commit message: CAN layout
Parts:
- C603, C605, C606, C607: symbol Manual:COMP_C603 -> ShiroFOCLib:COMP_C603
- C604: symbol Manual:COMP_C604 -> ShiroFOCLib:COMP_C604
- D601: value TPD3E001DRLR 3-line ESD -> TPD3E001DRYR; footprint Manual:TPD3E001_DRL5 -> ShiroFOCLib:TPD3E001_DRY6; symbol Manual:COMP_D601 -> ShiroFOCLib:COMP_D601; MPN TPD3E001DRLR -> TPD3E001DRYR; Manufacturer (none) -> Texas Instruments
- J601: symbol Manual:COMP_J601 -> ShiroFOCLib:COMP_J601
- R305: symbol Manual:COMP_R305 -> ShiroFOCLib:COMP_R305
- R306, R604, R615, R616, R617: symbol Manual:COMP_R306 -> ShiroFOCLib:COMP_R306
- R307: symbol Manual:COMP_R307 -> ShiroFOCLib:COMP_R307
- R605: symbol Manual:COMP_R605 -> ShiroFOCLib:COMP_R605
- R606: symbol Manual:COMP_R606 -> ShiroFOCLib:COMP_R606
- R607: symbol Manual:COMP_R607 -> ShiroFOCLib:COMP_R607
- R608: symbol Manual:COMP_R608 -> ShiroFOCLib:COMP_R608
- R609: symbol Manual:COMP_R609 -> ShiroFOCLib:COMP_R609
- R610: symbol Manual:COMP_R610 -> ShiroFOCLib:COMP_R610
- TP1015: symbol Manual:COMP_TP1015 -> ShiroFOCLib:COMP_TP1015
- TP1016: symbol Manual:COMP_TP1016 -> ShiroFOCLib:COMP_TP1016
- U602: footprint Manual:TMUX1574_PW16 -> ShiroFOCLib:TMUX1574_PW16; symbol Manual:COMP_U602 -> ShiroFOCLib:COMP_U602
- U604: symbol Manual:TPS2553_DBV -> ShiroFOCLib:TPS2553_DBV
Connections:
- net FB_ESD_RAIL: now also D601.6 (VCC); no longer D601.5 (VCC)
- net at J601.3, R605.1: now also D601.4 (IO3); no longer D601.1 (IO1)
- net at J601.5, R607.1: now also D601.1 (IO1); no longer D601.4 (IO3)
- no-connect marks 1 -> 2
Changed lines of the file:
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@@
 		(at 30.48 142.24)
 	)
+	(no_connect
+		(at 134.62 45.72)
+	)
 	(wire
 		(pts
@@
 	)
 	(symbol
-		(lib_id "Manual:COMP_U602")
+		(lib_id "ShiroFOCLib:COMP_U602")
 		(at 285.75 127 0)
 		(unit 1)
@@
 			)
 		)
-		(property "Footprint" "Manual:TMUX1574_PW16"
+		(property "Footprint" "ShiroFOCLib:TMUX1574_PW16"
 			(at 285.75 180.34 0)
 			(effects
@@
 	)
 	(symbol
-		(lib_id "Manual:PWR_3V3")
+		(lib_id "ShiroFOCLib:PWR_3V3")
 		(at 21.59 171.45 0)
 		(unit 1)
@@
 	)
 	(symbol
-		(lib_id "Manual:PWR_GND")
+		(lib_id "ShiroFOCLib:PWR_GND")
 		(at 165.1 251.46 0)
 		(unit 1)
@@
 	)
 	(symbol
-		(lib_id "Manual:COMP_R307")
+		(lib_id "ShiroFOCLib:COMP_R307")
 		(at 340.36 193.04 0)
 		(unit 1)
@@
 	)
 	(symbol
-		(lib_id "Manual:COMP_R609")
+		(lib_id "ShiroFOCLib:COMP_R609")
 		(at 184.15 119.38 0)
 		(unit 1)
@@
 	)
 	(symbol
-		(lib_id "Manual:TPS2553_DBV")
+		(lib_id "ShiroFOCLib:TPS2553_DBV")
 		(at 76.2 185.42 0)
 		(unit 1)
@@
 	)
 	(symbol
-		(lib_id "Manual:PWR_GND")
+		(lib_id "ShiroFOCLib:PWR_GND")
 		(at 157.48 205.74 0)
 		(unit 1)
@@
 	)
 	(symbol
-		(lib_id "Manual:COMP_R606")
+		(lib_id "ShiroFOCLib:COMP_R606")
 		(at 162.56 134.62 0)
 		(unit 1)
@@
 	)
 	(symbol
-		(lib_id "Manual:PWR_3V3")
+		(lib_id "ShiroFOCLib:PWR_3V3")
 		(at 198.12 226.06 0)
 		(unit 1)
@@
 	)
 	(symbol
-		(lib_id "Manual:PWR_3V3")
+		(lib_id "ShiroFOCLib:PWR_3V3")
 		(at 165.1 220.98 0)
 		(unit 1)
@@
 	)
 	(symbol
-		(lib_id "Manual:PWR_GND")
+		(lib_id "ShiroFOCLib:PWR_GND")
 		(at 76.2 205.74 0)
 		(unit 1)
@@
 	)
 	(symbol
-		(lib_id "Manual:PWR_GND")
+		(lib_id "ShiroFOCLib:PWR_GND")
 		(at 260.35 129.54 0)
 		(unit 1)
@@
 	)
 	(symbol
-		(lib_id "Manual:COMP_C603")
+		(lib_id "ShiroFOCLib:COMP_C603")
 		(at 339.09 227.33 0)
 		(unit 1)
@@
 	)
 	(symbol
-		(lib_id "Manual:PWR_GND")
+		(lib_id "ShiroFOCLib:PWR_GND")
 		(at 48.26 158.75 0)
 		(unit 1)
@@
 	)
 	(symbol
-		(lib_id "Manual:COMP_TP1015")
+		(lib_id "ShiroFOCLib:COMP_TP1015")
 		(at 330.2 92.71 0)
 		(unit 1)
@@
 	)
 	(symbol
-		(lib_id "Manual:PWR_GND")
+		(lib_id "ShiroFOCLib:PWR_GND")
 		(at 198.12 116.84 0)
 		(unit 1)
@@
 	)
 	(symbol
-		(lib_id "Manual:PWR_3V3")
+		(lib_id "ShiroFOCLib:PWR_3V3")
 		(at 114.3 162.56 0)
 		(unit 1)
@@
 	)
 	(symbol
-		(lib_id "Manual:PWR_3V3")
+		(lib_id "ShiroFOCLib:PWR_3V3")
 		(at 254 191.77 0)
 		(unit 1)
@@
 	)
 	(symbol
-		(lib_id "Manual:PWR_GND")
+		(lib_id "ShiroFOCLib:PWR_GND")
 		(at 40.64 205.74 0)
 		(unit 1)
@@
 	)
 	(symbol
-		(lib_id "Manual:PWR_3V3")
+		(lib_id "ShiroFOCLib:PWR_3V3")
 		(at 339.09 217.17 0)
 		(unit 1)
@@
 	)
 	(symbol
-		(lib_id "Manual:COMP_C603")
+		(lib_id "ShiroFOCLib:COMP_C603")
 		(at 157.48 196.85 0)
 		(unit 1)
@@
 	)
 	(symbol
-		(lib_id "Manual:COMP_J601")
+		(lib_id "ShiroFOCLib:COMP_J601")
 		(at 48.26 127 0)
 		(unit 1)
@@
 	)
 	(symbol
-		(lib_id "Manual:PWR_3V3")
+		(lib_id "ShiroFOCLib:PWR_3V3")
 		(at 298.45 193.04 0)
 		(unit 1)
@@
 	)
 	(symbol
-		(lib_id "Manual:PWR_GND")
+		(lib_id "ShiroFOCLib:PWR_GND")
 		(at 340.36 200.66 0)
 		(unit 1)
@@
 	)
 	(symbol
-		(lib_id "Manual:COMP_C603")
+		(lib_id "ShiroFOCLib:COMP_C603")
 		(at 198.12 236.22 0)
 		(unit 1)
@@
 	)
 	(symbol
-		(lib_id "Manual:PWR_GND")
+		(lib_id "ShiroFOCLib:PWR_GND")
 		(at 93.98 58.42 0)
 		(unit 1)
@@
 	)
 	(symbol
-		(lib_id "Manual:PWR_GND")
+		(lib_id "ShiroFOCLib:PWR_GND")
 		(at 260.35 167.64 0)
 		(unit 1)
@@
 	)
 	(symbol
-		(lib_id "Manual:PWR_GND")
+		(lib_id "ShiroFOCLib:PWR_GND")
 		(at 339.09 237.49 0)
 		(unit 1)
@@
 	)
 	(symbol
-		(lib_id "Manual:COMP_R608")
+		(lib_id "ShiroFOCLib:COMP_R608")
 		(at 184.15 81.28 0)
 		(unit 1)
@@
 	)
 	(symbol
-		(lib_id "Manual:PWR_GND")
+		(lib_id "ShiroFOCLib:PWR_GND")
 		(at 260.35 91.44 0)
 		(unit 1)
@@
 	)
 	(symbol
-		(lib_id "Manual:COMP_R306")
+		(lib_id "ShiroFOCLib:COMP_R306")
 		(at 241.3 227.33 0)
 		(unit 1)
@@
 	)
 	(symbol
-		(lib_id "Manual:COMP_D601")
+		(lib_id "ShiroFOCLib:COMP_D601")
 		(at 114.3 53.34 0)
 		(unit 1)
@@
 			)
 		)
-		(property "Value" "TPD3E001DRLR 3-line ESD"
+		(property "Value" "TPD3E001DRYR"
 			(at 114.3 47.625 0)
 			(effects
@@
 			)
 		)
-		(property "Footprint" "Manual:TPD3E001_DRL5"
+		(property "Footprint" "ShiroFOCLib:TPD3E001_DRY6"
 			(at 114.3 69.85 0)
 			(effects
@@
 			)
 		)
-		(property "MPN" "TPD3E001DRLR"
+		(property "MPN" "TPD3E001DRYR"
 			(at 114.3 69.85 0)
 			(effects
@@
 			)
 		)
+		(property "Manufacturer" "Texas Instruments"
+			(at 114.3 69.85 0)
+			(effects
+				(font
+					(size 1.27 1.27)
+				)
+				(hide yes)
+			)
+		)
 		(pin "3"
 		)
@@
 		(pin "4"
 		)
+		(pin "6"
+		)
 		(pin "5"
 		)
@@
 	)
 	(symbol
-		(lib_id "Manual:FLAG")
+		(lib_id "ShiroFOCLib:FLAG")
 		(at 50.8 180.34 0)
 		(unit 1)
@@
 	)
 	(symbol
-		(lib_id "Manual:PWR_GND")
+		(lib_id "ShiroFOCLib:PWR_GND")
 		(at 162.56 73.66 0)
 		(unit 1)
@@
 	)
 	(symbol
-		(lib_id "Manual:PWR_GND")
+		(lib_id "ShiroFOCLib:PWR_GND")
 		(at 298.45 254 0)
 		(unit 1)
@@
 	)
 	(symbol
-		(lib_id "Manual:PWR_GND")
+		(lib_id "ShiroFOCLib:PWR_GND")
 		(at 198.12 193.04 0)
 		(unit 1)
@@
 	)
 	(symbol
-		(lib_id "Manual:COMP_R306")
+		(lib_id "ShiroFOCLib:COMP_R306")
 		(at 198.12 147.32 0)
 		(unit 1)
@@
 	)
 	(symbol
-		(lib_id "Manual:PWR_5V_SYS")
+		(lib_id "ShiroFOCLib:PWR_5V_SYS")
 		(at 34.29 171.45 0)
 		(unit 1)
@@
 	)
 	(symbol
-		(lib_id "Manual:COMP_R306")
+		(lib_id "ShiroFOCLib:COMP_R306")
 		(at 198.12 185.42 0)
 		(unit 1)
@@
 	)
 	(symbol
-		(lib_id "Manual:COMP_R605")
+		(lib_id "ShiroFOCLib:COMP_R605")
 		(at 162.56 96.52 0)
 		(unit 1)
@@
 	)
 	(symbol
-		(lib_id "Manual:PWR_GND")
+		(lib_id "ShiroFOCLib:PWR_GND")
 		(at 198.12 246.38 0)
 		(unit 1)
@@
 	)
 	(symbol
-		(lib_id "Manual:COMP_TP1016")
+		(lib_id "ShiroFOCLib:COMP_TP1016")
 		(at 330.2 130.81 0)
 		(unit 1)
@@
 	)
 	(symbol
-		(lib_id "Manual:COMP_U602")
+		(lib_id "ShiroFOCLib:COMP_U602")
 		(at 77.47 236.22 0)
 		(unit 2)
@@
 			)
 		)
-		(property "Footprint" "Manual:TMUX1574_PW16"
+		(property "Footprint" "ShiroFOCLib:TMUX1574_PW16"
 			(at 77.47 248.92 0)
 			(effects
@@
 	)
 	(symbol
-		(lib_id "Manual:COMP_R306")
+		(lib_id "ShiroFOCLib:COMP_R306")
 		(at 198.12 109.22 0)
 		(unit 1)
@@
 	)
 	(symbol
-		(lib_id "Manual:PWR_GND")
+		(lib_id "ShiroFOCLib:PWR_GND")
 		(at 241.3 237.49 0)
 		(unit 1)
@@
 	)
 	(symbol
-		(lib_id "Manual:COMP_R306")
+		(lib_id "ShiroFOCLib:COMP_R306")
 		(at 114.3 172.72 0)
 		(unit 1)
@@
 	)
 	(symbol
-		(lib_id "Manual:COMP_R305")
+		(lib_id "ShiroFOCLib:COMP_R305")
 		(at 254 201.93 0)
 		(unit 1)
@@
 	)
 	(symbol
-		(lib_id "Manual:COMP_C604")
+		(lib_id "ShiroFOCLib:COMP_C604")
 		(at 162.56 63.5 0)
 		(unit 1)
@@
 	)
 	(symbol
-		(lib_id "Manual:COMP_R607")
+		(lib_id "ShiroFOCLib:COMP_R607")
 		(at 162.56 172.72 0)
 		(unit 1)
@@
 	)
 	(symbol
-		(lib_id "Manual:PWR_GND")
+		(lib_id "ShiroFOCLib:PWR_GND")
 		(at 198.12 154.94 0)
 		(unit 1)
@@
 	)
 	(symbol
-		(lib_id "Manual:COMP_R610")
+		(lib_id "ShiroFOCLib:COMP_R610")
 		(at 184.15 157.48 0)
 		(unit 1)
@@
 	)
 	(symbol
-		(lib_id "Manual:COMP_U602")
+		(lib_id "ShiroFOCLib:COMP_U602")
 		(at 298.45 223.52 0)
 		(unit 3)
@@
 			)
 		)
-		(property "Footprint" "Manual:TMUX1574_PW16"
+		(property "Footprint" "ShiroFOCLib:TMUX1574_PW16"
 			(at 298.45 246.38 0)
 			(effects
@@
 	)
 	(symbol
-		(lib_id "Manual:COMP_C603")
+		(lib_id "ShiroFOCLib:COMP_C603")
 		(at 40.64 196.85 0)
 		(unit 1)

Commit message: progress + p4
Parts:
- removed JP601: SENSOR SUPPLY, Jumper:SolderJumper-3_P1.3mm_Open_Pad1.0x1.5mm, symbol Jumper:Jumper_3_Open
- added R618: 49.9k 1%, Resistor_SMD:R_0402_1005Metric, symbol ShiroFOCLib:COMP_R306
- C606: value 4.7uF 16V X7R -> 4.7uF; Rating 4.7uF 16V X7R -> 4.7uF, 16V, X7R, 0603
- U604: BOM Comments Constant-current version, NOT -1 latch-off. EN and ILIM tie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 -> IN and EN on 5V_SYS; ILIM through R618=49.9k 1% to GND. OUT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; Procurement DBV SOT-23-6; footprint/3D association deferred to final CA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 -> TPS2553DBVR / SOT-23-6; constant-current version; Rating 2.5-6.5V; 75mA nominal limit with ILIM tied to IN; 50-100mA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 -> 520mA nominal shared limit; R618=49.9k 1%
Connections:
- net 5V_SYS: now also C606.1, U604.1 (IN), U604.3 (EN)
- net GND: now also J601.6, J601.MP (MOUNT), R618.2
- net at D601.2 (IO2), J601.4, R606.1: now also D601.5 (NC)
- net EXT_SENSOR_FAULT_N renamed EXT_POWER_FAULT_N
- removed net EXT_SUPPLY_SELECTED: C606.1, U604.1 (IN), U604.3 (EN), U604.5 (ILIM)
- new net: R618.1, U604.5 (ILIM)
- no-connect marks 2 -> 0
Other:
- note added: "INPUT OPTIONS Default: 3.3V / 5V push-pull; pull-ups DNP. Open-drain: fit R608-R610 (4.7k to protected 5V). Do not fit pull-ups for externally driven push-pull. 100k pull-downs define disconnected inputs. Single-ended only; common ground required."
- note added: "Joint feedback supply: fixed, protected 5V shared with J502 fan. J601.1 = 5V output; J601.2/6 = GND. No power input. For a 5V Hall/ABI encoder; no voltage selector. Sensor + pull-ups target <=25mA; shared accessory target <=300mA."
- note added: "U604: R618=49.9k 1% =>520mA nominal shared limit. EXT_VCC feeds J601 sensor + J502 fan + U503 PWM buffer. EXT_POWER_FAULT_N -> PC13; shared branch fault. Stop torque on fault or external-feedback loss; verify fan startup margin."
- note removed: "External sensor power is protected by U604 below. JP601: solder ONE pair:1-2=3V3,2-3=5V. Open for self-powered sensor; leave J601.1 unconnected. Normal sensor + pull-up load budget:25mA."
- note removed: "INPUT OPTIONS Default: 3.3V / 5V push-pull; pull-ups DNP. Open-drain: fit R608-R610 (4.7k). Pull-ups follow selected sensor supply. Do not fit for externally driven push-pull. 100k pull-downs define disconnected inputs. Single-ended only; common ground required."
- note removed: "U604: ILIM tied to IN =>75mA nominal (50-100mA). EN tied to IN: hardware protection, automatic recovery. FAULT_N -> PC13; firmware stops if external feedback is in use."
- moved on the sheet: C606, R305, TP1015, TP1016

Commit message: Routing started
Connections:
- net FEEDBACK_A_H1: now also U602.7 (D2); no longer U602.4 (D1)
- net FEEDBACK_B_H2: now also U602.4 (D1); no longer U602.7 (D2)
- net at U602.3 (S1B): now also U603.5; no longer U603.7
- net at U602.6 (S2B): now also U603.7; no longer U603.5

Commit message: weekend progress
Parts:
- J601: footprint Connector_JST:JST_GH_BM06B-GHS-TBT_1x06-1MP_P1.25mm_Vertical -> Connector_JST:JST_GH_SM06B-GHS-TB_1x06-1MP_P1.25mm_Horizontal; MPN BM06B-GHS-TBT -> SM06B-GHS-TB
Changed lines of the file:
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@@
 			)
 		)
-		(property "Footprint" "Connector_JST:JST_GH_BM06B-GHS-TBT_1x06-1MP_P1.25mm_Vertical"
+		(property "Footprint" "Connector_JST:JST_GH_SM06B-GHS-TB_1x06-1MP_P1.25mm_Horizontal"
 			(at 48.26 151.13 0)
 			(effects
@@
 			)
 		)
-		(property "MPN" "BM06B-GHS-TBT"
+		(property "MPN" "SM06B-GHS-TB"
 			(at 48.26 151.13 0)
 			(effects

Commit message: mosfet stages and opamps revamped
Connections:
- net FEEDBACK_A_H1: now also U602.9 (D3); no longer U602.7 (D2)
- net FEEDBACK_B_H2: now also U602.7 (D2); no longer U602.4 (D1)
- net FEEDBACK_I_H3: now also U602.4 (D1); no longer U602.9 (D3)
Other:
- moved on the sheet: TP1015, TP1016
Changed lines of the file:
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@@
 	)
 	(junction
-		(at 343.535 130.81)
-		(diameter 0)
-		(color 0 0 0 0)
-	)
-	(junction
 		(at 114.3 127)
 		(diameter 0)
@@
 	(wire
 		(pts
-			(xy 340.36 168.91) (xy 340.36 187.96)
+			(xy 340.36 181.61) (xy 340.36 187.96)
 		)
 		(stroke
@@
 		)
 	)
-	(global_label "FEEDBACK_A_H1"
+	(global_label "FEEDBACK_B_H2"
 		(shape bidirectional)
 		(at 368.3 92.71 0)
@@
 		)
 	)
-	(global_label "FEEDBACK_B_H2"
+	(global_label "FEEDBACK_I_H3"
 		(shape bidirectional)
 		(at 368.3 130.81 0)
@@
 		)
 	)
-	(global_label "FEEDBACK_I_H3"
+	(global_label "FEEDBACK_A_H1"
 		(shape bidirectional)
 		(at 368.3 168.91 0)
@@
 	(symbol
 		(lib_id "ShiroFOCLib:COMP_TP1015")
-		(at 343.535 92.71 0)
+		(at 340.36 168.91 0)
 		(mirror y)
 		(unit 1)
@@
 		(dnp no)
 		(property "Reference" "TP1015"
-			(at 340.995 87.63 0)
+			(at 337.82 163.83 0)
 			(effects
 				(font
@@
 		)
 		(property "Value" "FEEDBACK_A_H1"
-			(at 340.995 90.17 0)
+			(at 337.82 166.37 0)
 			(effects
 				(font
@@
 		)
 		(property "Footprint" "TestPoint:TestPoint_Pad_D1.0mm"
-			(at 340.995 92.71 0)
+			(at 337.82 168.91 0)
 			(effects
 				(font
@@
 		)
 		(property "Datasheet" ""
-			(at 340.995 92.71 0)
+			(at 337.82 168.91 0)
 			(effects
 				(font
@@
 		)
 		(property "Description" "Test point: FEEDBACK_A_H1"
-			(at 343.535 92.71 0)
+			(at 340.36 168.91 0)
 			(effects
 				(font
@@
 		)
 		(property "Assembly" "FIT"
-			(at 340.995 92.71 0)
+			(at 337.82 168.91 0)
 			(effects
 				(font
@@
 		)
 		(property "MPN" "PCB feature"
-			(at 340.995 92.71 0)
+			(at 337.82 168.91 0)
 			(effects
 				(font
@@
 		)
 		(property "Rating" "PCB test pad"
-			(at 340.995 92.71 0)
+			(at 337.82 168.91 0)
 			(effects
 				(font
@@
 		)
 		(property "Test_Net" "FEEDBACK_A_H1"
-			(at 340.995 92.71 0)
+			(at 337.82 168.91 0)
 			(effects
 				(font
@@
 	(symbol
 		(lib_id "ShiroFOCLib:COMP_TP1016")
-		(at 343.535 130.81 0)
+		(at 343.535 92.71 0)
 		(mirror y)
 		(unit 1)
@@
 		(dnp no)
 		(property "Reference" "TP1016"
-			(at 340.995 125.73 0)
+			(at 340.995 87.63 0)
 			(effects
 				(font
@@
 		)
 		(property "Value" "FEEDBACK_B_H2"
-			(at 340.995 128.27 0)
+			(at 340.995 90.17 0)
 			(effects
 				(font
@@
 		)
 		(property "Footprint" "TestPoint:TestPoint_Pad_D1.0mm"
-			(at 340.995 130.81 0)
+			(at 340.995 92.71 0)
 			(effects
 				(font
@@
 		)
 		(property "Datasheet" ""
-			(at 340.995 130.81 0)
+			(at 340.995 92.71 0)
 			(effects
 				(font
@@
 		)
 		(property "Description" "Test point: FEEDBACK_B_H2"
-			(at 343.535 130.81 0)
+			(at 343.535 92.71 0)
 			(effects
 				(font
@@
 		)
 		(property "Assembly" "FIT"
-			(at 340.995 130.81 0)
+			(at 340.995 92.71 0)
 			(effects
 				(font
@@
 		)
 		(property "MPN" "PCB feature"
-			(at 340.995 130.81 0)
+			(at 340.995 92.71 0)
 			(effects
 				(font
@@
 		)
 		(property "Rating" "PCB test pad"
-			(at 340.995 130.81 0)
+			(at 340.995 92.71 0)
 			(effects
 				(font
@@
 		)
 		(property "Test_Net" "FEEDBACK_B_H2"
-			(at 340.995 130.81 0)
+			(at 340.995 92.71 0)
 			(effects
 				(font
@@
 		)
 	)
+(global_label "FEEDBACK_I_H3" (shape bidirectional) (at 340.36 181.61 0)
+ (effects (font (size 1.016 1.016)) (justify left))
+ (property "Intersheetrefs" "${INTERSHEET_REFS}" (at 340.36 181.61 0) (effects (font (size 1.27 1.27)) (hide yes))))
 )
